File: Power_KiCAD_Project/Pcie_Connection.sch (KiCad schematic (older format))
At the start: 4 parts

Commit message: Changes to bus
bus was changed
Parts:
- removed J? (x4): PCIE-036-02-X-D-EMS2, Connector_PCBEdge:BUS_PCI_Express_Mini, symbol PCIE-036-02-X-D-EMS2:PCIE-036-02-X-D-EMS2
- added J? (x4): DB37_Female_MountingHoles, symbol Connector:DB37_Female_MountingHoles
Changed lines of the file:
@@
 $EndDescr
 $Comp
-L PCIE-036-02-X-D-EMS2:PCIE-036-02-X-D-EMS2 J?
-U 1 1 61841470
-P 4450 2750
-F 0 "J?" H 4450 3917 50  0000 C CNN
-F 1 "PCIE-036-02-X-D-EMS2" H 4450 3826 50  0000 C CNN
-F 2 "Connector_PCBEdge:BUS_PCI_Express_Mini" H 4450 2750 50  0001 L BNN
-F 3 "" H 4450 2750 50  0001 L BNN
-F 4 "3.715mm" H 4450 2750 50  0001 L BNN "MAXIMUM_PACKAGE_HEIGHT"
-F 5 "C" H 4450 2750 50  0001 L BNN "PARTREV"
-F 6 "Manufacturer Recommendations" H 4450 2750 50  0001 L BNN "STANDARD"
-F 7 "Samtec" H 4450 2750 50  0001 L BNN "MANUFACTURER"
-	1    4450 2750
+L Connector:DB37_Female_MountingHoles J?
+U 1 1 619B5F96
+P 4950 3150
+F 0 "J?" H 5130 3152 50  0000 L CNN
+F 1 "DB37_Female_MountingHoles" H 5130 3061 50  0000 L CNN
+F 2 "" H 4950 3150 50  0001 C CNN
+F 3 " ~" H 4950 3150 50  0001 C CNN
+	1    4950 3150
 	1    0    0    -1
 $EndComp
 $Comp
-L PCIE-036-02-X-D-EMS2:PCIE-036-02-X-D-EMS2 J?
-U 1 1 61848AB9
-P 5950 2750
-F 0 "J?" H 5950 3917 50  0000 C CNN
-F 1 "PCIE-036-02-X-D-EMS2" H 5950 3826 50  0000 C CNN
-F 2 "Connector_PCBEdge:BUS_PCI_Express_Mini" H 5950 2750 50  0001 L BNN
-F 3 "" H 5950 2750 50  0001 L BNN
-F 4 "3.715mm" H 5950 2750 50  0001 L BNN "MAXIMUM_PACKAGE_HEIGHT"
-F 5 "C" H 5950 2750 50  0001 L BNN "PARTREV"
-F 6 "Manufacturer Recommendations" H 5950 2750 50  0001 L BNN "STANDARD"
-F 7 "Samtec" H 5950 2750 50  0001 L BNN "MANUFACTURER"
-	1    5950 2750
+L Connector:DB37_Female_MountingHoles J?
+U 1 1 619B8741
+P 6750 3150
+F 0 "J?" H 6930 3152 50  0000 L CNN
+F 1 "DB37_Female_MountingHoles" H 6930 3061 50  0000 L CNN
+F 2 "" H 6750 3150 50  0001 C CNN
+F 3 " ~" H 6750 3150 50  0001 C CNN
+	1    6750 3150
 	1    0    0    -1
 $EndComp
 $Comp
-L PCIE-036-02-X-D-EMS2:PCIE-036-02-X-D-EMS2 J?
-U 1 1 61849C68
-P 7500 2750
-F 0 "J?" H 7500 3917 50  0000 C CNN
-F 1 "PCIE-036-02-X-D-EMS2" H 7500 3826 50  0000 C CNN
-F 2 "Connector_PCBEdge:BUS_PCI_Express_Mini" H 7500 2750 50  0001 L BNN
-F 3 "" H 7500 2750 50  0001 L BNN
-F 4 "3.715mm" H 7500 2750 50  0001 L BNN "MAXIMUM_PACKAGE_HEIGHT"
-F 5 "C" H 7500 2750 50  0001 L BNN "PARTREV"
-F 6 "Manufacturer Recommendations" H 7500 2750 50  0001 L BNN "STANDARD"
-F 7 "Samtec" H 7500 2750 50  0001 L BNN "MANUFACTURER"
-	1    7500 2750
+L Connector:DB37_Female_MountingHoles J?
+U 1 1 619BDF74
+P 8550 3200
+F 0 "J?" H 8730 3202 50  0000 L CNN
+F 1 "DB37_Female_MountingHoles" H 8730 3111 50  0000 L CNN
+F 2 "" H 8550 3200 50  0001 C CNN
+F 3 " ~" H 8550 3200 50  0001 C CNN
+	1    8550 3200
 	1    0    0    -1
 $EndComp
 $Comp
-L PCIE-036-02-X-D-EMS2:PCIE-036-02-X-D-EMS2 J?
-U 1 1 6184AAC3
-P 9000 2750
-F 0 "J?" H 9000 3917 50  0000 C CNN
-F 1 "PCIE-036-02-X-D-EMS2" H 9000 3826 50  0000 C CNN
-F 2 "Connector_PCBEdge:BUS_PCI_Express_Mini" H 9000 2750 50  0001 L BNN
-F 3 "" H 9000 2750 50  0001 L BNN
-F 4 "3.715mm" H 9000 2750 50  0001 L BNN "MAXIMUM_PACKAGE_HEIGHT"
-F 5 "C" H 9000 2750 50  0001 L BNN "PARTREV"
-F 6 "Manufacturer Recommendations" H 9000 2750 50  0001 L BNN "STANDARD"
-F 7 "Samtec" H 9000 2750 50  0001 L BNN "MANUFACTURER"
-	1    9000 2750
+L Connector:DB37_Female_MountingHoles J?
+U 1 1 619C0BB4
+P 3050 3150
+F 0 "J?" H 3230 3152 50  0000 L CNN
+F 1 "DB37_Female_MountingHoles" H 3230 3061 50  0000 L CNN
+F 2 "" H 3050 3150 50  0001 C CNN
+F 3 " ~" H 3050 3150 50  0001 C CNN
+	1    3050 3150
 	1    0    0    -1
 $EndComp
