File: Power_KiCAD_Project/TEMPSENSOR_MCP9808.sch (KiCad schematic (older format))
At the start: 2 parts

Commit message: Changes to bus
bus was changed
Parts:
- removed C?: 100nF, symbol Device:C
- added C2: 100nF, symbol Device:C
- gave numbers to parts that had none: 1
Connections:
- net +3V3: now also C2.1
- net GND: now also C2.2
Changed lines of the file:
@@
 $Descr A4 11693 8268
 encoding utf-8
-Sheet 2 6
+Sheet 2 11
 Title "MCP9608 Temperature Sensor"
 Date "2021-10-05"
@@
 $Comp
 L power:GND #PWR?
-U 1 1 6160E311
+U 1 1 61A8C2E0
 P 3250 3650
-AR Path="/6160E311" Ref="#PWR?"  Part="1"
-AR Path="/615C1FB4/6160E311" Ref="#PWR?"  Part="1"
-AR Path="/61B1B3BC/6160E311" Ref="#PWR?"  Part="1"
-AR Path="/61B35621/6160E311" Ref="#PWR?"  Part="1"
-F 0 "#PWR?" H 3250 3400 50  0001 C CNN
+AR Path="/61A8C2E0" Ref="#PWR?"  Part="1"
+AR Path="/615C1FB4/61A8C2E0" Ref="#PWR?"  Part="1"
+AR Path="/61B1B3BC/61A8C2E0" Ref="#PWR0103"  Part="1"
+AR Path="/61B35621/61A8C2E0" Ref="#PWR?"  Part="1"
+F 0 "#PWR0103" H 3250 3400 50  0001 C CNN
 F 1 "GND" H 3255 3477 50  0000 C CNN
 F 2 "" H 3250 3650 50  0001 C CNN
@@
 $Comp
 L power:+3.3V #PWR?
-U 1 1 6160E323
+U 1 1 61A8C2E1
 P 3700 2450
-AR Path="/6160E323" Ref="#PWR?"  Part="1"
-AR Path="/615C1FB4/6160E323" Ref="#PWR?"  Part="1"
-AR Path="/61B1B3BC/6160E323" Ref="#PWR?"  Part="1"
-AR Path="/61B35621/6160E323" Ref="#PWR?"  Part="1"
-F 0 "#PWR?" H 3700 2300 50  0001 C CNN
+AR Path="/61A8C2E1" Ref="#PWR?"  Part="1"
+AR Path="/615C1FB4/61A8C2E1" Ref="#PWR?"  Part="1"
+AR Path="/61B1B3BC/61A8C2E1" Ref="#PWR0104"  Part="1"
+AR Path="/61B35621/61A8C2E1" Ref="#PWR?"  Part="1"
+F 0 "#PWR0104" H 3700 2300 50  0001 C CNN
 F 1 "+3.3V" H 3715 2623 50  0000 C CNN
 F 2 "" H 3700 2450 50  0001 C CNN
@@
 $Comp
 L Device:C C?
-U 1 1 6160E331
+U 1 1 61A8C2E2
 P 4250 3100
-AR Path="/6160E331" Ref="C?"  Part="1"
-AR Path="/615C1FB4/6160E331" Ref="C?"  Part="1"
-AR Path="/61B1B3BC/6160E331" Ref="C?"  Part="1"
-AR Path="/61B35621/6160E331" Ref="C?"  Part="1"
-F 0 "C?" H 4365 3146 50  0000 L CNN
+AR Path="/61A8C2E2" Ref="C?"  Part="1"
+AR Path="/615C1FB4/61A8C2E2" Ref="C?"  Part="1"
+AR Path="/61B1B3BC/61A8C2E2" Ref="C2"  Part="1"
+AR Path="/61B35621/61A8C2E2" Ref="C?"  Part="1"
+F 0 "C2" H 4365 3146 50  0000 L CNN
 F 1 "100nF" H 4365 3055 50  0000 L CNN
 F 2 "" H 4288 2950 50  0001 C CNN
@@
 AR Path="/6160E30B" Ref="U?"  Part="1"
 AR Path="/615C1FB4/6160E30B" Ref="U?"  Part="1"
-AR Path="/61B1B3BC/6160E30B" Ref="U?"  Part="1"
+AR Path="/61B1B3BC/6160E30B" Ref="U1"  Part="1"
 AR Path="/61B35621/6160E30B" Ref="U?"  Part="1"
-F 0 "U?" H 3200 3800 50  0000 L CNN
+F 0 "U1" H 3200 3800 50  0000 L CNN
 F 1 "MCP9808_MSOP" H 2950 3700 50  0000 L CNN
 F 2 "Package_SO:MSOP-8_3x3mm_P0.65mm" H 3250 3050 50  0001 C CNN
@@
 AR Path="/618848DE" Ref="#PWR?"  Part="1"
 AR Path="/615C1FB4/618848DE" Ref="#PWR?"  Part="1"
-AR Path="/61B1B3BC/618848DE" Ref="#PWR?"  Part="1"
+AR Path="/61B1B3BC/618848DE" Ref="#PWR0105"  Part="1"
 AR Path="/61B35621/618848DE" Ref="#PWR?"  Part="1"
-F 0 "#PWR?" H 4250 3000 50  0001 C CNN
+F 0 "#PWR0105" H 4250 3000 50  0001 C CNN
 F 1 "GND" H 4255 3077 50  0000 C CNN
 F 2 "" H 4250 3250 50  0001 C CNN

Commit message: added components
added a few components and the correct numbers
Parts:
- C1: renamed from C2; footprint (none) -> Capacitor_SMD:C_0603_1608Metric
Connections:
- net GND renamed ground
Changed lines of the file:
@@
 $EndDescr
-$Comp
-L power:GND #PWR?
-U 1 1 61A8C2E0
-P 3250 3650
-AR Path="/61A8C2E0" Ref="#PWR?"  Part="1"
-AR Path="/615C1FB4/61A8C2E0" Ref="#PWR?"  Part="1"
-AR Path="/61B1B3BC/61A8C2E0" Ref="#PWR0103"  Part="1"
-AR Path="/61B35621/61A8C2E0" Ref="#PWR?"  Part="1"
-F 0 "#PWR0103" H 3250 3400 50  0001 C CNN
-F 1 "GND" H 3255 3477 50  0000 C CNN
-F 2 "" H 3250 3650 50  0001 C CNN
-F 3 "" H 3250 3650 50  0001 C CNN
-	1    3250 3650
-	1    0    0    -1
-$EndComp
 $Comp
 L power:+3.3V #PWR?
@@
 AR Path="/61A8C2E1" Ref="#PWR?"  Part="1"
 AR Path="/615C1FB4/61A8C2E1" Ref="#PWR?"  Part="1"
-AR Path="/61B1B3BC/61A8C2E1" Ref="#PWR0104"  Part="1"
+AR Path="/61B1B3BC/61A8C2E1" Ref="#PWR04"  Part="1"
 AR Path="/61B35621/61A8C2E1" Ref="#PWR?"  Part="1"
-F 0 "#PWR0104" H 3700 2300 50  0001 C CNN
+F 0 "#PWR04" H 3700 2300 50  0001 C CNN
 F 1 "+3.3V" H 3715 2623 50  0000 C CNN
 F 2 "" H 3700 2450 50  0001 C CNN
@@
 AR Path="/61A8C2E2" Ref="C?"  Part="1"
 AR Path="/615C1FB4/61A8C2E2" Ref="C?"  Part="1"
-AR Path="/61B1B3BC/61A8C2E2" Ref="C2"  Part="1"
+AR Path="/61B1B3BC/61A8C2E2" Ref="C1"  Part="1"
 AR Path="/61B35621/61A8C2E2" Ref="C?"  Part="1"
-F 0 "C2" H 4365 3146 50  0000 L CNN
+F 0 "C1" H 4365 3146 50  0000 L CNN
 F 1 "100nF" H 4365 3055 50  0000 L CNN
-F 2 "" H 4288 2950 50  0001 C CNN
+F 2 "Capacitor_SMD:C_0603_1608Metric" H 4288 2950 50  0001 C CNN
 F 3 "~" H 4250 3100 50  0001 C CNN
 	1    4250 3100
@@
 	3700 2500 4250 2500
 Connection ~ 3700 2500
-$Comp
-L power:GND #PWR?
-U 1 1 618848DE
-P 4250 3250
-AR Path="/618848DE" Ref="#PWR?"  Part="1"
-AR Path="/615C1FB4/618848DE" Ref="#PWR?"  Part="1"
-AR Path="/61B1B3BC/618848DE" Ref="#PWR0105"  Part="1"
-AR Path="/61B35621/618848DE" Ref="#PWR?"  Part="1"
-F 0 "#PWR0105" H 4250 3000 50  0001 C CNN
-F 1 "GND" H 4255 3077 50  0000 C CNN
-F 2 "" H 4250 3250 50  0001 C CNN
-F 3 "" H 4250 3250 50  0001 C CNN
-	1    4250 3250
-	1    0    0    -1
-$EndComp
 Text HLabel 3650 3050 2    50   Input ~ 0
 ALERT
@@
 Wire Wire Line
 	4250 2500 4250 2950
+Text HLabel 3250 3650 3    50   Input ~ 0
+ground
+Text HLabel 4250 3250 3    50   Input ~ 0
+ground
 $EndSCHEMATC
