File: Power_KiCAD_Project/LiPo_Pack_Monitor.sch (KiCad schematic (older format))
At the start: 36 parts

Commit message: Changed labels from global to local
Changed lines of the file:
@@
 $EndDescr
-$Comp
-L Battery_Management:BQ76920PW U?
-U 1 1 615F6CE9
-P 6750 3300
-F 0 "U?" H 6750 4450 50  0000 C CNN
-F 1 "BQ76920PW" H 6750 4350 50  0000 C CNN
-F 2 "Package_SO:TSSOP-20_4.4x6.5mm_P0.65mm" H 7650 2550 50  0001 C CNN
-F 3 "http://www.ti.com/lit/ds/symlink/bq76920.pdf" H 7450 3850 50  0001 C CNN
-F 4 "LiPo Pack Monitor" H 6750 4250 50  0000 C CNN "Description"
-	1    6750 3300
-	-1   0    0    -1
-$EndComp
 $Comp
 L Device:R R?
@@
 Wire Wire Line
 	6500 5250 6500 5350
-Text GLabel 6250 3100 0    50   Input ~ 0
-VC5
-Text GLabel 6250 3200 0    50   Input ~ 0
-VC4
-Text GLabel 6250 3300 0    50   Input ~ 0
-VC3
-Text GLabel 6250 3400 0    50   Input ~ 0
-VC2
-Text GLabel 6250 3500 0    50   Input ~ 0
-VC1
-Text GLabel 6250 3600 0    50   Input ~ 0
-VC0
-Text GLabel 4400 2900 2    50   Input ~ 0
-VC5
-Text GLabel 4400 3300 2    50   Input ~ 0
-VC4
-Text GLabel 4400 3700 2    50   Input ~ 0
-VC3
-Text GLabel 4400 4500 2    50   Input ~ 0
-VC1
-Text GLabel 4400 5100 2    50   Input ~ 0
-VC0
-Text GLabel 4400 4100 2    50   Input ~ 0
-VC2
 Wire Wire Line
 	4300 3300 4400 3300
@@
 Connection ~ 4300 5100
 Wire Wire Line
-	6750 2450 6750 2500
-Wire Wire Line
 	4400 2900 4300 2900
 Connection ~ 4300 2900
-$Comp
-L power:GND #PWR?
-U 1 1 615F6DAB
-P 6750 4100
-F 0 "#PWR?" H 6750 3850 50  0001 C CNN
-F 1 "GND" H 6755 3927 50  0000 C CNN
-F 2 "" H 6750 4100 50  0001 C CNN
-F 3 "" H 6750 4100 50  0001 C CNN
-	1    6750 4100
-	1    0    0    -1
-$EndComp
-Text GLabel 6250 3800 0    50   Input ~ 0
-SRP
-Text GLabel 6250 3900 0    50   Input ~ 0
-SRN
-Text GLabel 5100 4900 0    50   Input ~ 0
-SRP
-Text GLabel 6000 4900 2    50   Input ~ 0
-SRN
 Wire Wire Line
 	6000 4900 5950 4900
@@
 Wire Wire Line
 	5150 4900 5100 4900
-Text GLabel 7250 3400 2    50   Input ~ 0
-TS1
-Text GLabel 5100 4350 0    50   Input ~ 0
-TS1
 $Comp
 L Device:R R?
@@
 	1    0    0    -1
 $EndComp
-Text GLabel 6400 4350 2    50   Input ~ 0
-VC1
-$Comp
-L Switch:SW_Push SW?
-U 1 1 615F6DD2
-P 6100 4350
-F 0 "SW?" H 6100 4635 50  0000 C CNN
-F 1 "Reboot" H 6100 4544 50  0000 C CNN
-F 2 "" H 6100 4550 50  0001 C CNN
-F 3 "~" H 6100 4550 50  0001 C CNN
-	1    6100 4350
-	1    0    0    -1
-$EndComp
 Wire Wire Line
 	5800 4350 5900 4350
-Wire Wire Line
-	6300 4350 6400 4350
 $Comp
 L Device:Q_NMOS_GDS Q?
@@
 Wire Wire Line
 	5650 5250 5950 5250
-Text GLabel 6250 2900 0    50   Input ~ 0
-BAT
 $Comp
 L Device:R R?
@@
 Connection ~ 8350 4350
 Wire Wire Line
-	7850 4350 7350 4350
-Wire Wire Line
-	7350 4350 7350 3900
-Wire Wire Line
-	7350 3900 7250 3900
-Wire Wire Line
 	7350 4850 7350 4450
 Wire Wire Line
 	7350 4450 7500 4450
-Wire Wire Line
-	7500 4450 7500 3800
-Wire Wire Line
-	7500 3800 7250 3800
 Connection ~ 7350 4850
 $Comp
@@
 	1    0    0    -1
 $EndComp
-Text GLabel 7250 3000 2    50   Input ~ 0
-BATT_ALERT
 $Comp
 L Device:C_Small C?
@@
 	5700 2800 5700 2700
 Wire Wire Line
-	5700 2700 6250 2700
-Wire Wire Line
 	7850 2750 7850 2450
 $Comp
@@
 Wire Wire Line
 	8250 2500 8250 2450
-Wire Wire Line
-	8250 2450 7850 2450
 Connection ~ 7850 2450
 Wire Wire Line
 	8250 3000 8250 2900
-Text GLabel 8350 2900 2    50   Input ~ 0
-BAT
 Wire Wire Line
 	8350 2900 8250 2900
@@
 Wire Wire Line
 	7700 3650 7700 3600
-Wire Wire Line
-	7700 3600 7250 3600
 $Comp
 L power:+3.3V #PWR?
@@
 $EndComp
 Connection ~ 5700 2700
-Text GLabel 7250 2700 2    50   Input ~ 0
-I2C1_SDA
-Text GLabel 7250 2800 2    50   Input ~ 0
-I2C1_SCL
 Wire Wire Line
 	5150 5700 5400 5700
@@
 $EndComp
 Connection ~ 5150 5700
-Text Notes 2500 2050 0    100  ~ 0
-LiPo Pack Monitor
 Connection ~ 3050 5100
 Wire Wire Line
@@
 Wire Notes Line
 	2500 5950 2500 2100
-Wire Notes Line
-	2500 2100 9500 2100
 Wire Notes Line
 	2500 5950 9500 5950
@@
 +
 Wire Wire Line
-	6750 2450 7850 2450
-Wire Wire Line
 	4300 2800 4300 2900
 Wire Wire Line
@@
 Text HLabel 2950 5250 0    50   Input ~ 0
 PACK-
+Wire Notes Line
+	2500 2100 9500 2100
+Text Notes 2500 2050 0    100  ~ 0
+LiPo Pack Monitor
+Wire Wire Line
+	8250 2450 7850 2450
+Wire Wire Line
+	7850 4350 7350 4350
+Wire Wire Line
+	6300 4350 6400 4350
+$Comp
+L Battery_Management:BQ76920PW U?
+U 1 1 615F6CE9
+P 6750 3300
+F 0 "U?" H 6750 4450 50  0000 C CNN
+F 1 "BQ76920PW" H 6750 4350 50  0000 C CNN
+F 2 "Package_SO:TSSOP-20_4.4x6.5mm_P0.65mm" H 7650 2550 50  0001 C CNN
+F 3 "http://www.ti.com/lit/ds/symlink/bq76920.pdf" H 7450 3850 50  0001 C CNN
+F 4 "LiPo Pack Monitor" H 6750 4250 50  0000 C CNN "Description"
+	1    6750 3300
+	-1   0    0    -1
+$EndComp
+Wire Wire Line
+	7700 3600 7250 3600
+Wire Wire Line
+	7500 3800 7250 3800
+Wire Wire Line
+	7350 3900 7250 3900
+Text Label 6250 3100 2    50   ~ 0
+VC5
+Wire Wire Line
+	6750 2450 7850 2450
+Wire Wire Line
+	5700 2700 6250 2700
+Wire Wire Line
+	7500 4450 7500 3800
+Wire Wire Line
+	7350 4350 7350 3900
+$Comp
+L Switch:SW_Push SW?
+U 1 1 615F6DD2
+P 6100 4350
+F 0 "SW?" H 6100 4635 50  0000 C CNN
+F 1 "Reboot" H 6100 4544 50  0000 C CNN
+F 2 "" H 6100 4550 50  0001 C CNN
+F 3 "~" H 6100 4550 50  0001 C CNN
+	1    6100 4350
+	1    0    0    -1
+$EndComp
+$Comp
+L power:GND #PWR?
+U 1 1 615F6DAB
+P 6750 4100
+F 0 "#PWR?" H 6750 3850 50  0001 C CNN
+F 1 "GND" H 6755 3927 50  0000 C CNN
+F 2 "" H 6750 4100 50  0001 C CNN
+F 3 "" H 6750 4100 50  0001 C CNN
+	1    6750 4100
+	1    0    0    -1
+$EndComp
+Wire Wire Line
+	6750 2450 6750 2500
+Text Label 6250 3200 2    50   ~ 0
+VC4
+Text Label 6250 3300 2    50   ~ 0
+VC3
+Text Label 6250 3400 2    50   ~ 0
+VC2
+Text Label 6250 3500 2    50   ~ 0
+VC1
+Text Label 6250 3600 2    50   ~ 0
+VC0
+Text Label 6250 3800 2    50   ~ 0
+SRP
+Text Label 6250 3900 2    50   ~ 0
+SRN
+Text Label 6250 2900 2    50   ~ 0
+BAT
+Text Label 7550 3200 0    50   ~ 0
+l
+Text Label 7250 2700 0    50   ~ 0
+I2C1_SDA
+Text Label 7250 2800 0    50   ~ 0
+I2C1_SCL
+Text Label 7250 3000 0    50   ~ 0
+BATT_ALERT
+Text Label 7250 3400 0    50   ~ 0
+TS1
+Text Label 8350 2900 0    50   ~ 0
+BAT
+Text Label 6000 4900 0    50   ~ 0
+SRN
+Text Label 6400 4350 0    50   ~ 0
+VC1
+Text Label 5100 4350 2    50   ~ 0
+TS1
+Text Label 5100 4900 2    50   ~ 0
+SRP
+Text Label 4400 5100 0    50   ~ 0
+VC0
+Text Label 4400 4500 0    50   ~ 0
+VC1
+Text Label 4400 4100 0    50   ~ 0
+VC2
+Text Label 4400 3700 0    50   ~ 0
+VC3
+Text Label 4400 3300 0    50   ~ 0
+VC4
+Text Label 4400 2900 0    50   ~ 0
+VC5
 $EndSCHEMATC

Commit message: Changes to bus
bus was changed
Parts:
- gave numbers to parts that had none: 36
Connections:
- net GND: no longer Q1.3 (S), R13.2
- net PACK+: now also C14.2, R14.1, U3.9 (REGSRC)
- net at R10.1, R12.2: now also Q1.3 (S), R13.2
- net PACK-: now reaches Q3.2 (D), R16.2
- net I2C1_SCL renamed I2C_SCL
- net I2C1_SDA renamed I2C_SDA

Commit message: added components
added a few components and the correct numbers
Parts:
- removed D2: D, symbol Device:D
- removed Q1, Q3: Q_NMOS_GDS, symbol Device:Q_NMOS_GDS
- removed Q2: Q_PMOS_SDG, symbol Device:Q_PMOS_SDG
- added D2: 1N4148W-7-F, SamacSys_Parts:SOD3716X145N, symbol SamacSys_Parts:1N4148W-7-F
- added Q1, Q3: CSD17501Q5A, SamacSys_Parts:Q5A, symbol SamacSys_Parts:CSD17501Q5A
- added Q2: BSS84PH6327XTSA2, SamacSys_Parts:SOT95P240X110-3N, symbol SamacSys_Parts:BSS84PH6327XTSA2
- C10: renamed from C11; footprint (none) -> Capacitor_SMD:C_0603_1608Metric
- C11: renamed from C12; footprint (none) -> Capacitor_SMD:C_0603_1608Metric
- C12: renamed from C13; footprint (none) -> Capacitor_SMD:C_0603_1608Metric
- C13: renamed from C1; footprint (none) -> Capacitor_SMD:C_0603_1608Metric
- C14: footprint (none) -> Capacitor_SMD:C_0603_1608Metric
- C15: value Cf -> 10μF; footprint (none) -> Capacitor_SMD:C_0603_1608Metric
- C3: renamed from C4; value Cc -> 1μF; footprint (none) -> Capacitor_SMD:C_0603_1608Metric
- C4: renamed from C5; value Cc -> 1μF; footprint (none) -> Capacitor_SMD:C_0603_1608Metric
- C5: renamed from C6; value Cc -> 1μF; footprint (none) -> Capacitor_SMD:C_0603_1608Metric
- C6: renamed from C7; value Cc -> 1μF; footprint (none) -> Capacitor_SMD:C_0603_1608Metric
- C7: renamed from C8; value Cc -> 1μF; footprint (none) -> Capacitor_SMD:C_0603_1608Metric
- C8: renamed from C9; value Cc -> 1μF; footprint (none) -> Capacitor_SMD:C_0603_1608Metric
- C9: renamed from C10; footprint (none) -> Capacitor_SMD:C_0603_1608Metric
- D1: footprint (none) -> LED_SMD:LED_0603_1608Metric
- R1, R2, R3, R4, R5, R6: value Rc -> 100Ω; footprint (none) -> Resistor_SMD:R_0603_1608Metric
- R10: value Rsns -> .001Ω; footprint (none) -> Resistor_SMD:R_0603_1608Metric
- R11, R12, R13, R15, R16, R7, R8, R9: footprint (none) -> Resistor_SMD:R_0603_1608Metric
- R14: value Rf -> 100Ω; footprint (none) -> Resistor_SMD:R_0603_1608Metric
- SW1: footprint (none) -> Button_Switch_SMD:SW_Push_1P1T_NO_6x6mm_H9.5mm
Connections:
- net GND: now also Q2.1
- net PACK-: now also Q3.1 (S_1), Q3.2 (S_2), Q3.3 (S_3)
- net at R13.1, U3.1 (DSG): now also Q1.4 (G)
- net at U3.2 (CHG): now also Q2.3
- net at R10.1, R12.2, R13.2: now also Q1.1 (S_1), Q1.2 (S_2), Q1.3 (S_3)
- net at R15.1, R16.1: now also D2.1, Q3.4 (G)
- net at R15.2: now also D2.2, Q2.2
- new net: Q1.5 (D_1), Q1.6 (D_2), Q1.7 (D_3), Q1.8 (D_4), Q3.5 (D_1), Q3.6 (D_2), Q3.7 (D_3), Q3.8 (D_4)

Commit message: pcb finished
pcb is done. 3am kicad be like
Parts:
- removed R9: 10kΩ, Resistor_SMD:R_0603_1608Metric, symbol Device:R_Variable
- added VR1: T93YA103KT20, SamacSys_Parts:T93YA5K10, symbol SamacSys_Parts:T93YA103KT20
- renumbered R11 to R10, R12 to R11, R13 to R12, R14 to R13, R15 to R14, R16 to R15, R10 to R9
Connections:
- net GND: now also VR1.2 (B), VR1.3 (C)
- net TS1: now also VR1.1 (A)
- net +3V3: no longer names the net of C11.2, D1.2 (A), U3.8 (REGOUT)
Changed lines of the file:
@@
 $Descr A4 11693 8268
 encoding utf-8
-Sheet 4 12
+Sheet 7 7
 Title ""
 Date "2021-10-05"
@@
 $EndComp
 $Comp
-L Device:R R12
+L Device:R R11
 U 1 1 615F6D72
 P 5950 5500
-F 0 "R12" H 6020 5546 50  0000 L CNN
+F 0 "R11" H 6020 5546 50  0000 L CNN
 F 1 "100Ω" H 6020 5455 50  0000 L CNN
 F 2 "Resistor_SMD:R_0603_1608Metric" V 5880 5500 50  0001 C CNN
@@
 	5150 5700 5150 5650
 $Comp
-L Device:R R10
+L Device:R R9
 U 1 1 615F6D7F
 P 5550 5700
-F 0 "R10" V 5343 5700 50  0000 C CNN
+F 0 "R9" V 5343 5700 50  0000 C CNN
 F 1 ".001Ω" V 5434 5700 50  0000 C CNN
 F 2 "Resistor_SMD:R_0603_1608Metric" V 5480 5700 50  0001 C CNN
@@
 	4700 5250 4700 5350
 $Comp
-L power:GND #PWR013
+L power:GND #PWR012
 U 1 1 615F6D8E
 P 6500 5350
-F 0 "#PWR013" H 6500 5100 50  0001 C CNN
+F 0 "#PWR012" H 6500 5100 50  0001 C CNN
 F 1 "GND" H 6505 5177 50  0000 C CNN
 F 2 "" H 6500 5350 50  0001 C CNN
@@
 	5150 4900 5100 4900
 $Comp
-L Device:R R11
+L Device:R R10
 U 1 1 615F6DBB
 P 5650 4350
-F 0 "R11" V 5857 4350 50  0000 C CNN
+F 0 "R10" V 5857 4350 50  0000 C CNN
 F 1 "10kΩ" V 5766 4350 50  0000 C CNN
 F 2 "Resistor_SMD:R_0603_1608Metric" V 5580 4350 50  0001 C CNN
@@
 	0    -1   -1   0
 $EndComp
-Wire Wire Line
-	5100 4350 5350 4350
-$Comp
-L Device:R_Variable R9
-U 1 1 615F6DC2
-P 5350 4700
-F 0 "R9" H 5478 4746 50  0000 L CNN
-F 1 "10kΩ" H 5478 4655 50  0000 L CNN
-F 2 "Resistor_SMD:R_0603_1608Metric" V 5280 4700 50  0001 C CNN
-F 3 "~" H 5350 4700 50  0001 C CNN
-	1    5350 4700
-	1    0    0    -1
-$EndComp
-Wire Wire Line
-	5350 4550 5350 4350
 Connection ~ 5350 4350
 Wire Wire Line
@@
 	5650 5250 5950 5250
 $Comp
-L Device:R R13
+L Device:R R12
 U 1 1 615F6DEA
 P 6950 5050
-F 0 "R13" H 7020 5096 50  0000 L CNN
+F 0 "R12" H 7020 5096 50  0000 L CNN
 F 1 "1MΩ" H 7020 5005 50  0000 L CNN
 F 2 "Resistor_SMD:R_0603_1608Metric" V 6880 5050 50  0001 C CNN
@@
 	6950 5200 6950 5250
 $Comp
-L Device:R R16
+L Device:R R15
 U 1 1 615F6DF5
 P 9250 5050
-F 0 "R16" H 9320 5096 50  0000 L CNN
+F 0 "R15" H 9320 5096 50  0000 L CNN
 F 1 "1MΩ" H 9320 5005 50  0000 L CNN
 F 2 "Resistor_SMD:R_0603_1608Metric" V 9180 5050 50  0001 C CNN
@@
 	9250 4900 8850 4900
 $Comp
-L Device:R R15
+L Device:R R14
 U 1 1 615F6E05
 P 8600 4350
-F 0 "R15" V 8393 4350 50  0000 C CNN
+F 0 "R14" V 8393 4350 50  0000 C CNN
 F 1 "1MΩ" V 8484 4350 50  0000 C CNN
 F 2 "Resistor_SMD:R_0603_1608Metric" V 8530 4350 50  0001 C CNN
@@
 Connection ~ 7350 4850
 $Comp
-L power:GND #PWR017
+L power:GND #PWR016
 U 1 1 615F6E25
 P 8050 4650
-F 0 "#PWR017" H 8050 4400 50  0001 C CNN
+F 0 "#PWR016" H 8050 4400 50  0001 C CNN
 F 1 "GND" H 8050 4500 50  0000 C CNN
 F 2 "" H 8050 4650 50  0001 C CNN
@@
 $EndComp
 $Comp
-L power:GND #PWR016
+L power:GND #PWR015
 U 1 1 615F6E32
 P 7850 2950
-F 0 "#PWR016" H 7850 2700 50  0001 C CNN
+F 0 "#PWR015" H 7850 2700 50  0001 C CNN
 F 1 "GND" H 7855 2777 50  0000 C CNN
 F 2 "" H 7850 2950 50  0001 C CNN
@@
 $EndComp
 $Comp
-L power:GND #PWR015
+L power:GND #PWR014
 U 1 1 615F6E3E
 P 7700 3850
-F 0 "#PWR015" H 7700 3600 50  0001 C CNN
+F 0 "#PWR014" H 7700 3600 50  0001 C CNN
 F 1 "GND" H 7705 3677 50  0000 C CNN
 F 2 "" H 7700 3850 50  0001 C CNN
@@
 $EndComp
 $Comp
-L power:GND #PWR018
+L power:GND #PWR017
 U 1 1 615F6E4A
 P 8250 3200
-F 0 "#PWR018" H 8250 2950 50  0001 C CNN
+F 0 "#PWR017" H 8250 2950 50  0001 C CNN
 F 1 "GND" H 8255 3027 50  0000 C CNN
 F 2 "" H 8250 3200 50  0001 C CNN
@@
 $EndComp
 $Comp
-L power:GND #PWR012
+L power:GND #PWR011
 U 1 1 615F6E56
 P 5700 3000
-F 0 "#PWR012" H 5700 2750 50  0001 C CNN
+F 0 "#PWR011" H 5700 2750 50  0001 C CNN
 F 1 "GND" H 5705 2827 50  0000 C CNN
 F 2 "" H 5700 3000 50  0001 C CNN
@@
 	7850 2750 7850 2450
 $Comp
-L Device:R R14
+L Device:R R13
 U 1 1 615F6E5F
 P 8250 2650
-F 0 "R14" H 8180 2696 50  0000 R CNN
+F 0 "R13" H 8180 2696 50  0000 R CNN
 F 1 "100Ω" H 8180 2605 50  0000 R CNN
 F 2 "Resistor_SMD:R_0603_1608Metric" V 8180 2650 50  0001 C CNN
@@
 Wire Wire Line
 	7700 3650 7700 3600
-$Comp
-L power:+3.3V #PWR011
-U 1 1 615F6E6F
-P 5700 2700
-F 0 "#PWR011" H 5700 2550 50  0001 C CNN
-F 1 "+3.3V" H 5715 2873 50  0000 C CNN
-F 2 "" H 5700 2700 50  0001 C CNN
-F 3 "" H 5700 2700 50  0001 C CNN
-	1    5700 2700
-	1    0    0    -1
-$EndComp
 Connection ~ 5700 2700
 Wire Wire Line
@@
 Wire Wire Line
 	2950 3700 3650 3700
-Wire Wire Line
-	2950 3300 3650 3300
 Wire Notes Line
 	3050 2950 3400 2950
@@
 Wire Wire Line
 	6300 4350 6400 4350
-$Comp
-L Battery_Management:BQ76920PW U3
-U 1 1 615F6CE9
-P 6750 3300
-F 0 "U3" H 6750 4450 50  0000 C CNN
-F 1 "BQ76920PW" H 6750 4350 50  0000 C CNN
-F 2 "Package_SO:TSSOP-20_4.4x6.5mm_P0.65mm" H 7650 2550 50  0001 C CNN
-F 3 "http://www.ti.com/lit/ds/symlink/bq76920.pdf" H 7450 3850 50  0001 C CNN
-F 4 "LiPo Pack Monitor" H 6750 4250 50  0000 C CNN "Description"
-	1    6750 3300
-	-1   0    0    -1
-$EndComp
 Wire Wire Line
 	7700 3600 7250 3600
@@
 $EndComp
 $Comp
-L power:GND #PWR014
+L power:GND #PWR013
 U 1 1 615F6DAB
 P 6750 4100
-F 0 "#PWR014" H 6750 3850 50  0001 C CNN
+F 0 "#PWR013" H 6750 3850 50  0001 C CNN
 F 1 "GND" H 6755 3927 50  0000 C CNN
 F 2 "" H 6750 4100 50  0001 C CNN
@@
 Text Label 6250 2900 2    50   ~ 0
 BAT
-Text Label 7550 3200 0    50   ~ 0
-l
-Text Label 7250 3000 0    50   ~ 0
-BATT_ALERT
 Text Label 7250 3400 0    50   ~ 0
 TS1
@@
 Text Label 6400 4350 0    50   ~ 0
 VC1
-Text Label 5100 4350 2    50   ~ 0
+Text Label 5350 4200 1    50   ~ 0
 TS1
 Text Label 5100 4900 2    50   ~ 0
@@
 Text Label 7250 2800 0    50   ~ 0
 I2C_SCL
-Wire Wire Line
-	3650 2900 3050 2900
 Connection ~ 3050 2900
 $Comp
@@
 	0    1    1    0
 $EndComp
+$Comp
+L SamacSys_Parts:T93YA103KT20 VR1
+U 1 1 61CE0AE1
+P 5350 4700
+F 0 "VR1" H 5642 4235 50  0000 C CNN
+F 1 "T93YA103KT20" H 5642 4326 50  0000 C CNN
+F 2 "SamacSys_Parts:T93YA5K10" H 6000 4800 50  0001 L CNN
+F 3 "https://www.vishay.com/docs/51026/t93.pdf" H 6000 4700 50  0001 L CNN
+F 4 "10k, Through Hole Trimmer Potentiometer 0.5W Top Adjust Vishay, T93" H 6000 4600 50  0001 L CNN "Description"
+F 5 "9" H 6000 4500 50  0001 L CNN "Height"
+F 6 "72-T93YA-10K" H 6000 4400 50  0001 L CNN "Mouser Part Number"
+F 7 "https://www.mouser.co.uk/ProductDetail/Vishay-Sfernice/T93YA103KT20?qs=h4f6qdGYbthXcbdd7vDO0Q%3D%3D" H 6000 4300 50  0001 L CNN "Mouser Price/Stock"
+F 8 "Vishay" H 6000 4200 50  0001 L CNN "Manufacturer_Name"
+F 9 "T93YA103KT20" H 6000 4100 50  0001 L CNN "Manufacturer_Part_Number"
+	1    5350 4700
+	-1   0    0    1
+$EndComp
+Wire Wire Line
+	5350 4500 5350 4350
+Wire Wire Line
+	5350 4700 5350 4850
+Wire Wire Line
+	5350 4600 5350 4700
+Connection ~ 5350 4700
+Wire Wire Line
+	5350 4350 5350 4200
+Text Label 7250 3000 0    50   ~ 0
+BATT_ALERT
+Text Label 7550 3200 0    50   ~ 0
+l
+Wire Wire Line
+	2950 3300 3650 3300
+Wire Wire Line
+	3650 2900 3050 2900
+$Comp
+L Battery_Management:BQ76920PW U3
+U 1 1 615F6CE9
+P 6750 3300
+F 0 "U3" H 6750 4450 50  0000 C CNN
+F 1 "BQ76920PW" H 6750 4350 50  0000 C CNN
+F 2 "Package_SO:TSSOP-20_4.4x6.5mm_P0.65mm" H 7650 2550 50  0001 C CNN
+F 3 "http://www.ti.com/lit/ds/symlink/bq76920.pdf" H 7450 3850 50  0001 C CNN
+F 4 "LiPo Pack Monitor" H 6750 4250 50  0000 C CNN "Description"
+	1    6750 3300
+	-1   0    0    -1
+$EndComp
 $EndSCHEMATC
