File: Hardware/Power_KiCAD_Project.sch (KiCad schematic (older format))
At the start: 7 parts, among them J1 XT60-M, J2 XT60-M, J3 XT60-M, J4 XT60-M, J5 XT60-M, J6 PJ-102AH, J7 XT60-M

Commit message: Replaced passive component footprints with handsolder variants
I think the component sheet for the MCU STM32L152VET6Q is incorrect. Will investigate.
Changed lines of the file:
@@
 Wire Wire Line
 	3350 4200 3350 6550
-NoConn ~ 2800 2900
 $Comp
 L Power_KiCAD_Project-rescue:XT60-M-XT60-M J7
@@
 F10 "Switch" I L 3700 6200 50
 $EndSheet
+NoConn ~ 3400 3400
 Wire Bus Line
 	3050 2000 3050 2600
