File: Hardware/Power_KiCAD_Project.kicad_sch (KiCad schematic)
At the start: 7 parts, among them J1 Barrel_Jack_MountingPin, J2 XT60 Cell 5, J3 XT60 Cell 4, J4 XT60 Cell 3, J5 XT60 Cell 2, J6 XT60 Cell 1, J7 XT60 To External Switch

Commit message: Progress 1 to small board
Changed components around,deleted xt60s
Parts:
- removed J3: XT60 Cell 4, RDT_Custom_Footprints:AMASS_XT60-M, symbol Power_KiCAD_Project-rescue:XT60-M-XT60-M-Power_KiCAD_Project-rescue
- removed J5: XT60 Cell 2, RDT_Custom_Footprints:AMASS_XT60-M, symbol Power_KiCAD_Project-rescue:XT60-M-XT60-M-Power_KiCAD_Project-rescue
Connections:
- net PACK_M2 is gone; now on net PACK_M1: J4.1 (-)
- net PACK_M4 is gone; now on net PACK_M3: J2.1 (-)
Changed lines of the file:
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@@
+    (stroke (width 0) (type default) (color 0 0 0 0))
+  )
+  (wire (pts (xy 133.35 168.91) (xy 133.35 173.99))
     (stroke (width 0) (type default) (color 0 0 0 0))
   )
@@
     (stroke (width 0) (type default) (color 0 0 0 0))
   )
-  (wire (pts (xy 133.35 173.99) (xy 124.46 173.99))
+  (wire (pts (xy 124.46 173.99) (xy 133.35 173.99))
+    (stroke (width 0) (type default) (color 0 0 0 0))
+  )
+  (wire (pts (xy 133.35 146.05) (xy 133.35 151.13))
     (stroke (width 0) (type default) (color 0 0 0 0))
   )
@@
     (pin "3")
   )
-  (symbol (lib_id "Power_KiCAD_Project-rescue:XT60-M-XT60-M-Power_KiCAD_Project-rescue") (at 140.97 171.45 0) (mirror x) (unit 1)
-    (in_bom yes) (on_board yes)
-    (property "Reference" "J5" (id 0) (at 144.272 172.6184 0)
-      (effects (font (size 1.27 1.27)) (justify left))
-    )
-    (property "Value" "XT60 Cell 2" (id 1) (at 144.272 170.307 0)
-      (effects (font (size 1.27 1.27)) (justify left))
-    )
-    (property "Footprint" "RDT_Custom_Footprints:AMASS_XT60-M" (id 2) (at 140.97 171.45 0)
-      (effects (font (size 1.27 1.27)) (justify left bottom) hide)
-    )
-    (property "Datasheet" "" (id 3) (at 140.97 171.45 0)
-      (effects (font (size 1.27 1.27)) (justify left bottom) hide)
-    )
-    (property "MP" "XT60-M" (id 4) (at 140.97 171.45 0)
-      (effects (font (size 1.27 1.27)) (justify left bottom) hide)
-    )
-    (property "Price" "None" (id 5) (at 140.97 171.45 0)
-      (effects (font (size 1.27 1.27)) (justify left bottom) hide)
-    )
-    (property "Package" "Package" (id 6) (at 140.97 171.45 0)
-      (effects (font (size 1.27 1.27)) (justify left bottom) hide)
-    )
-    (property "MF" "AMASS" (id 7) (at 140.97 171.45 0)
-      (effects (font (size 1.27 1.27)) (justify left bottom) hide)
-    )
-    (property "Availability" "Not in stock" (id 8) (at 140.97 171.45 0)
-      (effects (font (size 1.27 1.27)) (justify left bottom) hide)
-    )
-    (property "Description" "Plug; DC supply; XT60; male; PIN: 2; for cable; soldered; 30A; 500V" (id 9) (at 140.97 171.45 0)
-      (effects (font (size 1.27 1.27)) (justify left bottom) hide)
-    )
-    (pin "1")
-    (pin "2")
-  )
   (symbol (lib_id "Power_KiCAD_Project-rescue:XT60-M-XT60-M-Power_KiCAD_Project-rescue") (at 140.97 160.02 0) (mirror x) (unit 1)
     (in_bom yes) (on_board yes)
@@
     )
     (property "Description" "Plug; DC supply; XT60; male; PIN: 2; for cable; soldered; 30A; 500V" (id 9) (at 140.97 160.02 0)
-      (effects (font (size 1.27 1.27)) (justify left bottom) hide)
-    )
-    (pin "1")
-    (pin "2")
-  )
-  (symbol (lib_id "Power_KiCAD_Project-rescue:XT60-M-XT60-M-Power_KiCAD_Project-rescue") (at 140.97 148.59 0) (mirror x) (unit 1)
-    (in_bom yes) (on_board yes)
-    (property "Reference" "J3" (id 0) (at 144.272 149.7584 0)
-      (effects (font (size 1.27 1.27)) (justify left))
-    )
-    (property "Value" "XT60 Cell 4" (id 1) (at 144.272 147.447 0)
-      (effects (font (size 1.27 1.27)) (justify left))
-    )
-    (property "Footprint" "RDT_Custom_Footprints:AMASS_XT60-M" (id 2) (at 140.97 148.59 0)
-      (effects (font (size 1.27 1.27)) (justify left bottom) hide)
-    )
-    (property "Datasheet" "" (id 3) (at 140.97 148.59 0)
-      (effects (font (size 1.27 1.27)) (justify left bottom) hide)
-    )
-    (property "MP" "XT60-M" (id 4) (at 140.97 148.59 0)
-      (effects (font (size 1.27 1.27)) (justify left bottom) hide)
-    )
-    (property "Price" "None" (id 5) (at 140.97 148.59 0)
-      (effects (font (size 1.27 1.27)) (justify left bottom) hide)
-    )
-    (property "Package" "Package" (id 6) (at 140.97 148.59 0)
-      (effects (font (size 1.27 1.27)) (justify left bottom) hide)
-    )
-    (property "MF" "AMASS" (id 7) (at 140.97 148.59 0)
-      (effects (font (size 1.27 1.27)) (justify left bottom) hide)
-    )
-    (property "Availability" "Not in stock" (id 8) (at 140.97 148.59 0)
-      (effects (font (size 1.27 1.27)) (justify left bottom) hide)
-    )
-    (property "Description" "Plug; DC supply; XT60; male; PIN: 2; for cable; soldered; 30A; 500V" (id 9) (at 140.97 148.59 0)
       (effects (font (size 1.27 1.27)) (justify left bottom) hide)
     )
@@
       (reference "C11") (unit 1) (value "1μF") (footprint "Capacitor_SMD:C_1206_3216Metric_Pad1.42x1.75mm_HandSolder")
     )
-    (path "/00000000-0000-0000-0000-0000615ed460/00000000-0000-0000-0000-0000615f6d1d"
-      (reference "C12") (unit 1) (value "1μF") (footprint "Capacitor_SMD:C_1206_3216Metric_Pad1.42x1.75mm_HandSolder")
-    )
     (path "/00000000-0000-0000-0000-0000615ed460/00000000-0000-0000-0000-0000615f6d23"
       (reference "C13") (unit 1) (value "1μF") (footprint "Capacitor_SMD:C_1206_3216Metric_Pad1.42x1.75mm_HandSolder")
     )
-    (path "/00000000-0000-0000-0000-0000615ed460/00000000-0000-0000-0000-0000615f6d29"
-      (reference "C14") (unit 1) (value "1μF") (footprint "Capacitor_SMD:C_1206_3216Metric_Pad1.42x1.75mm_HandSolder")
-    )
     (path "/00000000-0000-0000-0000-0000615ed460/00000000-0000-0000-0000-0000615f6d3a"
       (reference "C15") (unit 1) (value "1μF") (footprint "Capacitor_SMD:C_1206_3216Metric_Pad1.42x1.75mm_HandSolder")
@@
       (reference "J2") (unit 1) (value "XT60 Cell 5") (footprint "RDT_Custom_Footprints:AMASS_XT60-M")
     )
-    (path "/00000000-0000-0000-0000-000061c25141"
-      (reference "J3") (unit 1) (value "XT60 Cell 4") (footprint "RDT_Custom_Footprints:AMASS_XT60-M")
-    )
     (path "/00000000-0000-0000-0000-000061c24ca6"
       (reference "J4") (unit 1) (value "XT60 Cell 3") (footprint "RDT_Custom_Footprints:AMASS_XT60-M")
     )
-    (path "/00000000-0000-0000-0000-000061c24684"
-      (reference "J5") (unit 1) (value "XT60 Cell 2") (footprint "RDT_Custom_Footprints:AMASS_XT60-M")
-    )
     (path "/00000000-0000-0000-0000-000061c66d12"
