File: Hardware/COMPONENT_SHEETS/LiPo_Pack_Monitor.sch (KiCad schematic (older format))
At the start: 36 parts

Commit message: FIxed board
issues with the board after the merge have been fixed
Parts:
- R10: renamed from R?; footprint RESC7146X175N -> RDT_Custom_Footprints:RESC7146X175N
- gave numbers to parts that had none: 35
Connections:
- wire segments 128 -> 129

Commit message: Replaced passive component footprints with handsolder variants
I think the component sheet for the MCU STM32L152VET6Q is incorrect. Will investigate.
Parts:
- C17, C18, C19, C20, C21, C22, C23, C24, C25, C26, C27, C28, C29: footprint Capacitor_SMD:C_0603_1608Metric -> Capacitor_SMD:C_0603_1608Metric_Pad1.08x0.95mm_HandSolder
- D5: footprint LED_SMD:LED_0603_1608Metric -> LED_SMD:LED_0603_1608Metric_Pad1.05x0.95mm_HandSolder
- R11, R12, R13, R14, R15, R16, R17, R3, R4, R5, R6, R7, R8, R9: footprint Resistor_SMD:R_0603_1608Metric -> Resistor_SMD:R_0603_1608Metric_Pad1.05x0.95mm_HandSolder
Changed lines of the file:
@@
 F 0 "R3" V 4007 2900 50  0000 C CNN
 F 1 "100Ω" V 3916 2900 50  0000 C CNN
-F 2 "Resistor_SMD:R_0603_1608Metric" V 3730 2900 50  0001 C CNN
+F 2 "Resistor_SMD:R_0603_1608Metric_Pad1.05x0.95mm_HandSolder" V 3730 2900 50  0001 C CNN
 F 3 "~" H 3800 2900 50  0001 C CNN
 	1    3800 2900
@@
 F 0 "R4" V 4007 3300 50  0000 C CNN
 F 1 "100Ω" V 3916 3300 50  0000 C CNN
-F 2 "Resistor_SMD:R_0603_1608Metric" V 3730 3300 50  0001 C CNN
+F 2 "Resistor_SMD:R_0603_1608Metric_Pad1.05x0.95mm_HandSolder" V 3730 3300 50  0001 C CNN
 F 3 "~" H 3800 3300 50  0001 C CNN
 	1    3800 3300
@@
 F 0 "R5" V 4007 3700 50  0000 C CNN
 F 1 "100Ω" V 3916 3700 50  0000 C CNN
-F 2 "Resistor_SMD:R_0603_1608Metric" V 3730 3700 50  0001 C CNN
+F 2 "Resistor_SMD:R_0603_1608Metric_Pad1.05x0.95mm_HandSolder" V 3730 3700 50  0001 C CNN
 F 3 "~" H 3800 3700 50  0001 C CNN
 	1    3800 3700
@@
 F 0 "R6" V 4007 4100 50  0000 C CNN
 F 1 "100Ω" V 3916 4100 50  0000 C CNN
-F 2 "Resistor_SMD:R_0603_1608Metric" V 3730 4100 50  0001 C CNN
+F 2 "Resistor_SMD:R_0603_1608Metric_Pad1.05x0.95mm_HandSolder" V 3730 4100 50  0001 C CNN
 F 3 "~" H 3800 4100 50  0001 C CNN
 	1    3800 4100
@@
 F 0 "R7" V 4007 4500 50  0000 C CNN
 F 1 "100Ω" V 3916 4500 50  0000 C CNN
-F 2 "Resistor_SMD:R_0603_1608Metric" V 3730 4500 50  0001 C CNN
+F 2 "Resistor_SMD:R_0603_1608Metric_Pad1.05x0.95mm_HandSolder" V 3730 4500 50  0001 C CNN
 F 3 "~" H 3800 4500 50  0001 C CNN
 	1    3800 4500
@@
 F 0 "R8" V 4007 5100 50  0000 C CNN
 F 1 "100Ω" V 3916 5100 50  0000 C CNN
-F 2 "Resistor_SMD:R_0603_1608Metric" V 3730 5100 50  0001 C CNN
+F 2 "Resistor_SMD:R_0603_1608Metric_Pad1.05x0.95mm_HandSolder" V 3730 5100 50  0001 C CNN
 F 3 "~" H 3800 5100 50  0001 C CNN
 	1    3800 5100
@@
 F 0 "C17" H 4392 3146 50  0000 L CNN
 F 1 "1μF" H 4392 3055 50  0000 L CNN
-F 2 "Capacitor_SMD:C_0603_1608Metric" H 4300 3100 50  0001 C CNN
+F 2 "Capacitor_SMD:C_0603_1608Metric_Pad1.08x0.95mm_HandSolder" H 4300 3100 50  0001 C CNN
 F 3 "~" H 4300 3100 50  0001 C CNN
 	1    4300 3100
@@
 F 0 "C18" H 4392 3546 50  0000 L CNN
 F 1 "1μF" H 4392 3455 50  0000 L CNN
-F 2 "Capacitor_SMD:C_0603_1608Metric" H 4300 3500 50  0001 C CNN
+F 2 "Capacitor_SMD:C_0603_1608Metric_Pad1.08x0.95mm_HandSolder" H 4300 3500 50  0001 C CNN
 F 3 "~" H 4300 3500 50  0001 C CNN
 	1    4300 3500
@@
 F 0 "C19" H 4392 3946 50  0000 L CNN
 F 1 "1μF" H 4392 3855 50  0000 L CNN
-F 2 "Capacitor_SMD:C_0603_1608Metric" H 4300 3900 50  0001 C CNN
+F 2 "Capacitor_SMD:C_0603_1608Metric_Pad1.08x0.95mm_HandSolder" H 4300 3900 50  0001 C CNN
 F 3 "~" H 4300 3900 50  0001 C CNN
 	1    4300 3900
@@
 F 0 "C20" H 4392 4346 50  0000 L CNN
 F 1 "1μF" H 4392 4255 50  0000 L CNN
-F 2 "Capacitor_SMD:C_0603_1608Metric" H 4300 4300 50  0001 C CNN
+F 2 "Capacitor_SMD:C_0603_1608Metric_Pad1.08x0.95mm_HandSolder" H 4300 4300 50  0001 C CNN
 F 3 "~" H 4300 4300 50  0001 C CNN
 	1    4300 4300
@@
 F 0 "C21" H 4392 4696 50  0000 L CNN
 F 1 "1μF" H 4392 4605 50  0000 L CNN
-F 2 "Capacitor_SMD:C_0603_1608Metric" H 4300 4650 50  0001 C CNN
+F 2 "Capacitor_SMD:C_0603_1608Metric_Pad1.08x0.95mm_HandSolder" H 4300 4650 50  0001 C CNN
 F 3 "~" H 4300 4650 50  0001 C CNN
 	1    4300 4650
@@
 F 0 "C22" H 4392 4996 50  0000 L CNN
 F 1 "1μF" H 4392 4905 50  0000 L CNN
-F 2 "Capacitor_SMD:C_0603_1608Metric" H 4300 4950 50  0001 C CNN
+F 2 "Capacitor_SMD:C_0603_1608Metric_Pad1.08x0.95mm_HandSolder" H 4300 4950 50  0001 C CNN
 F 3 "~" H 4300 4950 50  0001 C CNN
 	1    4300 4950
@@
 F 0 "C23" V 4671 5250 50  0000 C CNN
 F 1 "0.1μF" V 4762 5250 50  0000 C CNN
-F 2 "Capacitor_SMD:C_0603_1608Metric" H 4900 5250 50  0001 C CNN
+F 2 "Capacitor_SMD:C_0603_1608Metric_Pad1.08x0.95mm_HandSolder" H 4900 5250 50  0001 C CNN
 F 3 "~" H 4900 5250 50  0001 C CNN
 	1    4900 5250
@@
 F 0 "C24" V 5321 5250 50  0000 C CNN
 F 1 "0.1μF" V 5412 5250 50  0000 C CNN
-F 2 "Capacitor_SMD:C_0603_1608Metric" H 5550 5250 50  0001 C CNN
+F 2 "Capacitor_SMD:C_0603_1608Metric_Pad1.08x0.95mm_HandSolder" H 5550 5250 50  0001 C CNN
 F 3 "~" H 5550 5250 50  0001 C CNN
 	1    5550 5250
@@
 F 0 "C26" V 6071 5250 50  0000 C CNN
 F 1 "0.1μF" V 6162 5250 50  0000 C CNN
-F 2 "Capacitor_SMD:C_0603_1608Metric" H 6300 5250 50  0001 C CNN
+F 2 "Capacitor_SMD:C_0603_1608Metric_Pad1.08x0.95mm_HandSolder" H 6300 5250 50  0001 C CNN
 F 3 "~" H 6300 5250 50  0001 C CNN
 	1    6300 5250
@@
 F 0 "R9" H 5080 5546 50  0000 R CNN
 F 1 "100Ω" H 5080 5455 50  0000 R CNN
-F 2 "Resistor_SMD:R_0603_1608Metric" V 5080 5500 50  0001 C CNN
+F 2 "Resistor_SMD:R_0603_1608Metric_Pad1.05x0.95mm_HandSolder" V 5080 5500 50  0001 C CNN
 F 3 "~" H 5150 5500 50  0001 C CNN
 	1    5150 5500
@@
 F 0 "R13" H 6020 5546 50  0000 L CNN
 F 1 "100Ω" H 6020 5455 50  0000 L CNN
-F 2 "Resistor_SMD:R_0603_1608Metric" V 5880 5500 50  0001 C CNN
+F 2 "Resistor_SMD:R_0603_1608Metric_Pad1.05x0.95mm_HandSolder" V 5880 5500 50  0001 C CNN
 F 3 "~" H 5950 5500 50  0001 C CNN
 	1    5950 5500
@@
 F 0 "R12" V 5857 4350 50  0000 C CNN
 F 1 "10kΩ" V 5766 4350 50  0000 C CNN
-F 2 "Resistor_SMD:R_0603_1608Metric" V 5580 4350 50  0001 C CNN
+F 2 "Resistor_SMD:R_0603_1608Metric_Pad1.05x0.95mm_HandSolder" V 5580 4350 50  0001 C CNN
 F 3 "~" H 5650 4350 50  0001 C CNN
 	1    5650 4350
@@
 F 0 "R14" H 7020 5096 50  0000 L CNN
 F 1 "1MΩ" H 7020 5005 50  0000 L CNN
-F 2 "Resistor_SMD:R_0603_1608Metric" V 6880 5050 50  0001 C CNN
+F 2 "Resistor_SMD:R_0603_1608Metric_Pad1.05x0.95mm_HandSolder" V 6880 5050 50  0001 C CNN
 F 3 "~" H 6950 5050 50  0001 C CNN
 	1    6950 5050
@@
 F 0 "R16" V 8393 4350 50  0000 C CNN
 F 1 "1MΩ" V 8484 4350 50  0000 C CNN
-F 2 "Resistor_SMD:R_0603_1608Metric" V 8530 4350 50  0001 C CNN
+F 2 "Resistor_SMD:R_0603_1608Metric_Pad1.05x0.95mm_HandSolder" V 8530 4350 50  0001 C CNN
 F 3 "~" H 8600 4350 50  0001 C CNN
 	1    8600 4350
@@
 F 0 "C28" H 7758 2804 50  0000 R CNN
 F 1 "1μF" H 7758 2895 50  0000 R CNN
-F 2 "Capacitor_SMD:C_0603_1608Metric" H 7850 2850 50  0001 C CNN
+F 2 "Capacitor_SMD:C_0603_1608Metric_Pad1.08x0.95mm_HandSolder" H 7850 2850 50  0001 C CNN
 F 3 "~" H 7850 2850 50  0001 C CNN
 	1    7850 2850
@@
 F 0 "C27" H 7608 3704 50  0000 R CNN
 F 1 "1μF" H 7608 3795 50  0000 R CNN
-F 2 "Capacitor_SMD:C_0603_1608Metric" H 7700 3750 50  0001 C CNN
+F 2 "Capacitor_SMD:C_0603_1608Metric_Pad1.08x0.95mm_HandSolder" H 7700 3750 50  0001 C CNN
 F 3 "~" H 7700 3750 50  0001 C CNN
 	1    7700 3750
@@
 F 0 "C29" H 8158 3054 50  0000 R CNN
 F 1 "10μF" H 8158 3145 50  0000 R CNN
-F 2 "Capacitor_SMD:C_0603_1608Metric" H 8250 3100 50  0001 C CNN
+F 2 "Capacitor_SMD:C_0603_1608Metric_Pad1.08x0.95mm_HandSolder" H 8250 3100 50  0001 C CNN
 F 3 "~" H 8250 3100 50  0001 C CNN
 	1    8250 3100
@@
 F 0 "C25" H 5608 2854 50  0000 R CNN
 F 1 "4.7μF" H 5608 2945 50  0000 R CNN
-F 2 "Capacitor_SMD:C_0603_1608Metric" H 5700 2900 50  0001 C CNN
+F 2 "Capacitor_SMD:C_0603_1608Metric_Pad1.08x0.95mm_HandSolder" H 5700 2900 50  0001 C CNN
 F 3 "~" H 5700 2900 50  0001 C CNN
 	1    5700 2900
@@
 F 0 "R15" H 8180 2696 50  0000 R CNN
 F 1 "100Ω" H 8180 2605 50  0000 R CNN
-F 2 "Resistor_SMD:R_0603_1608Metric" V 8180 2650 50  0001 C CNN
+F 2 "Resistor_SMD:R_0603_1608Metric_Pad1.05x0.95mm_HandSolder" V 8180 2650 50  0001 C CNN
 F 3 "~" H 8250 2650 50  0001 C CNN
 	1    8250 2650
@@
 F 0 "R11" H 5370 3496 50  0000 L CNN
 F 1 "1k5Ω" H 5370 3405 50  0000 L CNN
-F 2 "Resistor_SMD:R_0603_1608Metric" V 5230 3450 50  0001 C CNN
+F 2 "Resistor_SMD:R_0603_1608Metric_Pad1.05x0.95mm_HandSolder" V 5230 3450 50  0001 C CNN
 F 3 "~" H 5300 3450 50  0001 C CNN
 	1    5300 3450
@@
 F 0 "R17" H 9320 5096 50  0000 L CNN
 F 1 "1MΩ" H 9320 5005 50  0000 L CNN
-F 2 "Resistor_SMD:R_0603_1608Metric" V 9180 5050 50  0001 C CNN
+F 2 "Resistor_SMD:R_0603_1608Metric_Pad1.05x0.95mm_HandSolder" V 9180 5050 50  0001 C CNN
 F 3 "~" H 9250 5050 50  0001 C CNN
 	1    9250 5050
@@
 F 0 "D5" V 5339 2882 50  0000 R CNN
 F 1 "LED" V 5248 2882 50  0000 R CNN
-F 2 "LED_SMD:LED_0603_1608Metric" H 5300 3000 50  0001 C CNN
+F 2 "LED_SMD:LED_0603_1608Metric_Pad1.05x0.95mm_HandSolder" H 5300 3000 50  0001 C CNN
 F 3 "~" H 5300 3000 50  0001 C CNN
 	1    5300 3000
