File: Hardware/COMPONENT_SHEETS/LiPo_Pack_Monitor.sch (KiCad schematic (older format))
At the start: 36 parts, among them Q1 BSS84PH6327XTSA2, SW1 Reboot, U5 BQ76920PW, U6 PSMN2R6-40YS, U7 PSMN2R6-40YS

Commit message: Rearranged LiPo Monitor component sheet
 - Added XT60 connector for external switch connection
 - Updated a few component symbols to be the default ones
 - Replaced label "ground" with the GNDREF symbol
 - LiPo Pack Monitor I2C and Alert Lines still need to be added
Parts:
- removed D6: 1N4148W-7-F, SamacSys_Parts:SOD3716X145N, symbol Power_KiCAD_Project-rescue:1N4148W-7-F-SamacSys_Parts
- removed Q1: BSS84PH6327XTSA2, SamacSys_Parts:SOT95P240X110-3N, symbol Power_KiCAD_Project-rescue:BSS84PH6327XTSA2-SamacSys_Parts
- removed R10: WSHP28185L000FEA, RDT_Custom_Footprints:RESC7146X175N, symbol Power_KiCAD_Project-rescue:WSHP28185L000FEA-SamacSys_Parts
- removed U6, U7: PSMN2R6-40YS, TO127P600X120-5N:TO127P600X120-5N, symbol Power_KiCAD_Project-rescue:PSMN2R6-40YS-1-747301-6
- removed VR1: T93YA103KT20, SamacSys_Parts:T93YA5K10, symbol Power_KiCAD_Project-rescue:T93YA103KT20-SamacSys_Parts
- added D6: 1N4148W-7-F, Diode_SMD:D_SOD-123, symbol Device:D
- added J13: XT60 To External Switch, XT60-M:AMASS_XT60-M, symbol Power_KiCAD_Project-rescue:XT60-M-XT60-M
- added Q1, Q3: PSMN2R6-40YS, Package_TO_SOT_SMD:LFPAK33, symbol Transistor_FET:BUK7M9R9-60EX
- added Q2: BSS84PH6327XTSA2, Package_TO_SOT_SMD:SOT-23, symbol Device:Q_PMOS_GSD
- added R11: 5mΩ 10W, RDT_Custom_Footprints:RESC7146X175N, symbol Device:R
- added RV1: 10Ω to 2.2MΩ, symbol Device:R_POT_TRIM
- renumbered C25 to C24, C24 to C25, C28 to C27, C27 to C28, R9 to R10, R13 to R12, R14 to R13, R15 to R14, R16 to R15, R12 to R16, R11 to R9
Connections:
- net labels added: GNDREF
- net labels removed: BAT, GND, SRN, SRP, Switch, TS1, l
- wire segments 129 -> 119
- no-connect marks 0 -> 1
Other:
- note removed: "LiPo Pack Monitor"
- note removed: "Simplified Schematic given from BQ76920 datasheet."
- moved on the sheet: C17, C18, C19, C20, C21, C22, C23, C24, C25, C26, C27, C28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

Commit message: Updated component footprints, moved to RDT_Custom_Footprints library
Parts:
- C17, C18, C19, C20, C21, C22, C23, C24, C25, C26, C27, C28, C29: footprint Capacitor_SMD:C_0603_1608Metric -> Capacitor_SMD:C_0603_1608Metric_Pad1.08x0.95mm_HandSolder
- J13: footprint XT60-M:AMASS_XT60-M -> RDT_Custom_Footprints:AMASS_XT60-M
- R10, R12, R13, R14, R15, R16, R17, R3, R4, R5, R6, R7, R8, R9: footprint Resistor_SMD:R_0603_1608Metric -> Resistor_SMD:R_0603_1608Metric_Pad1.05x0.95mm_HandSolder
- RV1: footprint (none) -> RDT_Custom_Footprints:T93YA5K10
Changed lines of the file:
@@
 $Descr A4 11693 8268
 encoding utf-8
-Sheet 6 7
+Sheet 5 7
 Title "LiPo Pack Monitor"
 Date "2021-12-20"
@@
 F 0 "R3" V 2457 2700 50  0000 C CNN
 F 1 "100Ω" V 2366 2700 50  0000 C CNN
-F 2 "Resistor_SMD:R_0603_1608Metric" V 2180 2700 50  0001 C CNN
+F 2 "Resistor_SMD:R_0603_1608Metric_Pad1.05x0.95mm_HandSolder" V 2180 2700 50  0001 C CNN
 F 3 "~" H 2250 2700 50  0001 C CNN
 	1    2250 2700
@@
 F 0 "R4" V 2457 3100 50  0000 C CNN
 F 1 "100Ω" V 2366 3100 50  0000 C CNN
-F 2 "Resistor_SMD:R_0603_1608Metric" V 2180 3100 50  0001 C CNN
+F 2 "Resistor_SMD:R_0603_1608Metric_Pad1.05x0.95mm_HandSolder" V 2180 3100 50  0001 C CNN
 F 3 "~" H 2250 3100 50  0001 C CNN
 	1    2250 3100
@@
 F 0 "R5" V 2457 3500 50  0000 C CNN
 F 1 "100Ω" V 2366 3500 50  0000 C CNN
-F 2 "Resistor_SMD:R_0603_1608Metric" V 2180 3500 50  0001 C CNN
+F 2 "Resistor_SMD:R_0603_1608Metric_Pad1.05x0.95mm_HandSolder" V 2180 3500 50  0001 C CNN
 F 3 "~" H 2250 3500 50  0001 C CNN
 	1    2250 3500
@@
 F 0 "R6" V 2457 3900 50  0000 C CNN
 F 1 "100Ω" V 2366 3900 50  0000 C CNN
-F 2 "Resistor_SMD:R_0603_1608Metric" V 2180 3900 50  0001 C CNN
+F 2 "Resistor_SMD:R_0603_1608Metric_Pad1.05x0.95mm_HandSolder" V 2180 3900 50  0001 C CNN
 F 3 "~" H 2250 3900 50  0001 C CNN
 	1    2250 3900
@@
 F 0 "R7" V 2457 4300 50  0000 C CNN
 F 1 "100Ω" V 2366 4300 50  0000 C CNN
-F 2 "Resistor_SMD:R_0603_1608Metric" V 2180 4300 50  0001 C CNN
+F 2 "Resistor_SMD:R_0603_1608Metric_Pad1.05x0.95mm_HandSolder" V 2180 4300 50  0001 C CNN
 F 3 "~" H 2250 4300 50  0001 C CNN
 	1    2250 4300
@@
 F 0 "R8" V 2457 4900 50  0000 C CNN
 F 1 "100Ω" V 2366 4900 50  0000 C CNN
-F 2 "Resistor_SMD:R_0603_1608Metric" V 2180 4900 50  0001 C CNN
+F 2 "Resistor_SMD:R_0603_1608Metric_Pad1.05x0.95mm_HandSolder" V 2180 4900 50  0001 C CNN
 F 3 "~" H 2250 4900 50  0001 C CNN
 	1    2250 4900
@@
 F 0 "C17" H 3042 2946 50  0000 L CNN
 F 1 "1μF" H 3042 2855 50  0000 L CNN
-F 2 "Capacitor_SMD:C_0603_1608Metric" H 2950 2900 50  0001 C CNN
+F 2 "Capacitor_SMD:C_0603_1608Metric_Pad1.08x0.95mm_HandSolder" H 2950 2900 50  0001 C CNN
 F 3 "~" H 2950 2900 50  0001 C CNN
 	1    2950 2900
@@
 F 0 "C18" H 3042 3346 50  0000 L CNN
 F 1 "1μF" H 3042 3255 50  0000 L CNN
-F 2 "Capacitor_SMD:C_0603_1608Metric" H 2950 3300 50  0001 C CNN
+F 2 "Capacitor_SMD:C_0603_1608Metric_Pad1.08x0.95mm_HandSolder" H 2950 3300 50  0001 C CNN
 F 3 "~" H 2950 3300 50  0001 C CNN
 	1    2950 3300
@@
 F 0 "C19" H 3042 3746 50  0000 L CNN
 F 1 "1μF" H 3042 3655 50  0000 L CNN
-F 2 "Capacitor_SMD:C_0603_1608Metric" H 2950 3700 50  0001 C CNN
+F 2 "Capacitor_SMD:C_0603_1608Metric_Pad1.08x0.95mm_HandSolder" H 2950 3700 50  0001 C CNN
 F 3 "~" H 2950 3700 50  0001 C CNN
 	1    2950 3700
@@
 F 0 "C20" H 3042 4146 50  0000 L CNN
 F 1 "1μF" H 3042 4055 50  0000 L CNN
-F 2 "Capacitor_SMD:C_0603_1608Metric" H 2950 4100 50  0001 C CNN
+F 2 "Capacitor_SMD:C_0603_1608Metric_Pad1.08x0.95mm_HandSolder" H 2950 4100 50  0001 C CNN
 F 3 "~" H 2950 4100 50  0001 C CNN
 	1    2950 4100
@@
 F 0 "C21" H 3042 4496 50  0000 L CNN
 F 1 "1μF" H 3042 4405 50  0000 L CNN
-F 2 "Capacitor_SMD:C_0603_1608Metric" H 2950 4450 50  0001 C CNN
+F 2 "Capacitor_SMD:C_0603_1608Metric_Pad1.08x0.95mm_HandSolder" H 2950 4450 50  0001 C CNN
 F 3 "~" H 2950 4450 50  0001 C CNN
 	1    2950 4450
@@
 F 0 "C22" H 3042 4796 50  0000 L CNN
 F 1 "1μF" H 3042 4705 50  0000 L CNN
-F 2 "Capacitor_SMD:C_0603_1608Metric" H 2950 4750 50  0001 C CNN
+F 2 "Capacitor_SMD:C_0603_1608Metric_Pad1.08x0.95mm_HandSolder" H 2950 4750 50  0001 C CNN
 F 3 "~" H 2950 4750 50  0001 C CNN
 	1    2950 4750
@@
 F 0 "C23" V 4471 5250 50  0000 C CNN
 F 1 "0.1μF" V 4562 5250 50  0000 C CNN
-F 2 "Capacitor_SMD:C_0603_1608Metric" H 4700 5250 50  0001 C CNN
+F 2 "Capacitor_SMD:C_0603_1608Metric_Pad1.08x0.95mm_HandSolder" H 4700 5250 50  0001 C CNN
 F 3 "~" H 4700 5250 50  0001 C CNN
 	1    4700 5250
@@
 F 0 "C25" V 5121 5250 50  0000 C CNN
 F 1 "0.1μF" V 5212 5250 50  0000 C CNN
-F 2 "Capacitor_SMD:C_0603_1608Metric" H 5350 5250 50  0001 C CNN
+F 2 "Capacitor_SMD:C_0603_1608Metric_Pad1.08x0.95mm_HandSolder" H 5350 5250 50  0001 C CNN
 F 3 "~" H 5350 5250 50  0001 C CNN
 	1    5350 5250
@@
 F 0 "C26" V 5871 5250 50  0000 C CNN
 F 1 "0.1μF" V 5962 5250 50  0000 C CNN
-F 2 "Capacitor_SMD:C_0603_1608Metric" H 6100 5250 50  0001 C CNN
+F 2 "Capacitor_SMD:C_0603_1608Metric_Pad1.08x0.95mm_HandSolder" H 6100 5250 50  0001 C CNN
 F 3 "~" H 6100 5250 50  0001 C CNN
 	1    6100 5250
@@
 F 0 "R10" H 4880 5546 50  0000 R CNN
 F 1 "100Ω" H 4880 5455 50  0000 R CNN
-F 2 "Resistor_SMD:R_0603_1608Metric" V 4880 5500 50  0001 C CNN
+F 2 "Resistor_SMD:R_0603_1608Metric_Pad1.05x0.95mm_HandSolder" V 4880 5500 50  0001 C CNN
 F 3 "~" H 4950 5500 50  0001 C CNN
 	1    4950 5500
@@
 F 0 "R12" H 5820 5546 50  0000 L CNN
 F 1 "100Ω" H 5820 5455 50  0000 L CNN
-F 2 "Resistor_SMD:R_0603_1608Metric" V 5680 5500 50  0001 C CNN
+F 2 "Resistor_SMD:R_0603_1608Metric_Pad1.05x0.95mm_HandSolder" V 5680 5500 50  0001 C CNN
 F 3 "~" H 5750 5500 50  0001 C CNN
 	1    5750 5500
@@
 F 0 "R16" V 9257 3400 50  0000 C CNN
 F 1 "10kΩ" V 9166 3400 50  0000 C CNN
-F 2 "Resistor_SMD:R_0603_1608Metric" V 8980 3400 50  0001 C CNN
+F 2 "Resistor_SMD:R_0603_1608Metric_Pad1.05x0.95mm_HandSolder" V 8980 3400 50  0001 C CNN
 F 3 "~" H 9050 3400 50  0001 C CNN
 	1    9050 3400
@@
 F 0 "R13" H 7470 5596 50  0000 L CNN
 F 1 "1MΩ" H 7470 5505 50  0000 L CNN
-F 2 "Resistor_SMD:R_0603_1608Metric" V 7330 5550 50  0001 C CNN
+F 2 "Resistor_SMD:R_0603_1608Metric_Pad1.05x0.95mm_HandSolder" V 7330 5550 50  0001 C CNN
 F 3 "~" H 7400 5550 50  0001 C CNN
 	1    7400 5550
@@
 F 0 "R15" V 8743 4900 50  0000 C CNN
 F 1 "1MΩ" V 8834 4900 50  0000 C CNN
-F 2 "Resistor_SMD:R_0603_1608Metric" V 8880 4900 50  0001 C CNN
+F 2 "Resistor_SMD:R_0603_1608Metric_Pad1.05x0.95mm_HandSolder" V 8880 4900 50  0001 C CNN
 F 3 "~" H 8950 4900 50  0001 C CNN
 	1    8950 4900
@@
 F 0 "C28" H 8058 3604 50  0000 R CNN
 F 1 "1μF" H 8058 3695 50  0000 R CNN
-F 2 "Capacitor_SMD:C_0603_1608Metric" H 8150 3650 50  0001 C CNN
+F 2 "Capacitor_SMD:C_0603_1608Metric_Pad1.08x0.95mm_HandSolder" H 8150 3650 50  0001 C CNN
 F 3 "~" H 8150 3650 50  0001 C CNN
 	1    8150 3650
@@
 F 0 "C24" H 4308 2654 50  0000 R CNN
 F 1 "4.7μF" H 4308 2745 50  0000 R CNN
-F 2 "Capacitor_SMD:C_0603_1608Metric" H 4400 2700 50  0001 C CNN
+F 2 "Capacitor_SMD:C_0603_1608Metric_Pad1.08x0.95mm_HandSolder" H 4400 2700 50  0001 C CNN
 F 3 "~" H 4400 2700 50  0001 C CNN
 	1    4400 2700
@@
 F 0 "R9" H 4070 3296 50  0000 L CNN
 F 1 "1k5Ω" H 4070 3205 50  0000 L CNN
-F 2 "Resistor_SMD:R_0603_1608Metric" V 3930 3250 50  0001 C CNN
+F 2 "Resistor_SMD:R_0603_1608Metric_Pad1.05x0.95mm_HandSolder" V 3930 3250 50  0001 C CNN
 F 3 "~" H 4000 3250 50  0001 C CNN
 	1    4000 3250
@@
 F 0 "R17" H 9620 5596 50  0000 L CNN
 F 1 "1MΩ" H 9620 5505 50  0000 L CNN
-F 2 "Resistor_SMD:R_0603_1608Metric" V 9480 5550 50  0001 C CNN
+F 2 "Resistor_SMD:R_0603_1608Metric_Pad1.05x0.95mm_HandSolder" V 9480 5550 50  0001 C CNN
 F 3 "~" H 9550 5550 50  0001 C CNN
 	1    9550 5550
@@
 F 0 "RV1" H 8680 3741 50  0000 R CNN
 F 1 "10Ω to 2.2MΩ" H 8680 3650 50  0000 R CNN
-F 2 "" H 8750 3650 50  0001 C CNN
+F 2 "RDT_Custom_Footprints:T93YA5K10" H 8750 3650 50  0001 C CNN
 F 3 "~" H 8750 3650 50  0001 C CNN
 F 4 "Nominal 10kΩ" H 8680 3559 50  0000 R CNN "Other"
@@
 F 0 "C27" H 7808 1954 50  0000 R CNN
 F 1 "1μF" H 7808 2045 50  0000 R CNN
-F 2 "Capacitor_SMD:C_0603_1608Metric" H 7900 2000 50  0001 C CNN
+F 2 "Capacitor_SMD:C_0603_1608Metric_Pad1.08x0.95mm_HandSolder" H 7900 2000 50  0001 C CNN
 F 3 "~" H 7900 2000 50  0001 C CNN
 	1    7900 2000
@@
 F 0 "C29" H 5158 2854 50  0000 R CNN
 F 1 "10μF" H 5158 2945 50  0000 R CNN
-F 2 "Capacitor_SMD:C_0603_1608Metric" H 5250 2900 50  0001 C CNN
+F 2 "Capacitor_SMD:C_0603_1608Metric_Pad1.08x0.95mm_HandSolder" H 5250 2900 50  0001 C CNN
 F 3 "~" H 5250 2900 50  0001 C CNN
 	1    5250 2900
@@
 F 0 "R14" H 5180 2096 50  0000 R CNN
 F 1 "100Ω" H 5180 2005 50  0000 R CNN
-F 2 "Resistor_SMD:R_0603_1608Metric" V 5180 2050 50  0001 C CNN
+F 2 "Resistor_SMD:R_0603_1608Metric_Pad1.05x0.95mm_HandSolder" V 5180 2050 50  0001 C CNN
 F 3 "~" H 5250 2050 50  0001 C CNN
 	1    5250 2050
@@
 F 0 "J13" V 3000 5600 50  0000 L CNN
 F 1 "XT60 To External Switch" V 3150 4900 50  0000 L CNN
-F 2 "XT60-M:AMASS_XT60-M" H 3000 5400 50  0001 L BNN
+F 2 "RDT_Custom_Footprints:AMASS_XT60-M" H 3000 5400 50  0001 L BNN
 F 3 "" H 3000 5400 50  0001 L BNN
 F 4 "XT60-M" H 3000 5400 50  0001 L BNN "MP"

Commit message: Reset annotations, changed SPST switch footprint
Parts:
- SW1: footprint Button_Switch_SMD:SW_Push_1P1T_NO_6x6mm_H9.5mm -> Button_Switch_SMD:SW_SPST_PTS645
- renumbered C17 to C11, C18 to C12, C19 to C13, C20 to C14, C21 to C15, C22 to C16, C24 to C17, C23 to C18, C29 to C19, C25 to C20, C26 to C21, C27 to C22, C28 to C23, D5 to D3, D6 to D4, J13 to J7, R3 to R1, R11 to R10, R12 to R11, R13 to R12, R15 to R13, R16 to R14, R17 to R15, R4 to R2, R5 to R3, R6 to R4, R7 to R5, R8 to R6, R9 to R7, R10 to R8, R14 to R9

Commit message: Routed 3v3 and 5v buck converters
Switched to working on my laptop so some of the component references might be messed up for a bit
Parts:
- J7: symbol Power_KiCAD_Project-rescue:XT60-M-XT60-M -> Power_KiCAD_Project-rescue:XT60-M-XT60-M-Power_KiCAD_Project-rescue
Changed lines of the file:
@@
 	4400 2500 5850 2500
 $Comp
-L Power_KiCAD_Project-rescue:XT60-M-XT60-M J?
+L Power_KiCAD_Project-rescue:XT60-M-XT60-M-Power_KiCAD_Project-rescue J?
 U 1 1 61C225DB
 P 3000 5400

Commit message: Moved external switch connector to pack+, added missing no connection flags
This change renders the current PCB layout defunct, next commits will be redesigns of the layout.
Parts:
- removed J7: XT60 To External Switch, RDT_Custom_Footprints:AMASS_XT60-M, symbol Power_KiCAD_Project-rescue:XT60-M-XT60-M-Power_KiCAD_Project-rescue
Connections:
- wire segments 119 -> 116
Changed lines of the file:
@@
 Wire Wire Line
 	4400 2500 5850 2500
-$Comp
-L Power_KiCAD_Project-rescue:XT60-M-XT60-M-Power_KiCAD_Project-rescue J?
-U 1 1 61C225DB
-P 3000 5400
-AR Path="/61C225DB" Ref="J?"  Part="1"
-AR Path="/615ED460/61C225DB" Ref="J7"  Part="1"
-F 0 "J7" V 3000 5600 50  0000 L CNN
-F 1 "XT60 To External Switch" V 3150 4900 50  0000 L CNN
-F 2 "RDT_Custom_Footprints:AMASS_XT60-M" H 3000 5400 50  0001 L BNN
-F 3 "" H 3000 5400 50  0001 L BNN
-F 4 "XT60-M" H 3000 5400 50  0001 L BNN "MP"
-F 5 "None" H 3000 5400 50  0001 L BNN "Price"
-F 6 "Package" H 3000 5400 50  0001 L BNN "Package"
-F 7 "AMASS" H 3000 5400 50  0001 L BNN "MF"
-F 8 "Not in stock" H 3000 5400 50  0001 L BNN "Availability"
-F 9 "Plug; DC supply; XT60; male; PIN: 2; for cable; soldered; 30A; 500V" H 3000 5400 50  0001 L BNN "Description"
-	1    3000 5400
-	0    -1   -1   0
-$EndComp
 Wire Bus Line
 	4750 3700 4750 3250
@@
 Wire Bus Line
 	3450 3700 4750 3700
-Wire Wire Line
-	2900 5750 2900 5700
-Wire Wire Line
-	3100 5700 3100 5750
 Connection ~ 4950 5750
 Wire Wire Line
@@
 Wire Wire Line
 	5650 3600 5650 4700
-Wire Wire Line
-	3100 5750 4950 5750
 Wire Wire Line
 	1500 1750 5250 1750
@@
 	1700 4900 2100 4900
 Wire Wire Line
-	2900 5750 1700 5750
-Wire Wire Line
 	1700 4900 1700 5750
 $Comp
@@
 	1700 5850 1700 5750
 Connection ~ 1700 5750
+Wire Wire Line
+	1700 5750 4950 5750
 Wire Bus Line
 	3450 2800 3450 3700

Commit message: Routed GNDREF side of board
Correcting keepout silkscreen added 3mm to top and bottom, much appreciated!
Parts:
- C11, C12, C13, C14, C15, C16, C19, C22, C23: footprint Capacitor_SMD:C_0603_1608Metric_Pad1.08x0.95mm_HandSolder -> Capacitor_SMD:C_1206_3216Metric_Pad1.42x1.75mm_HandSolder
- C18, C20, C21: footprint Capacitor_SMD:C_0603_1608Metric_Pad1.08x0.95mm_HandSolder -> Resistor_SMD:R_0603_1608Metric_Pad1.05x0.95mm_HandSolder
- R1, R2, R3, R4, R5, R6, R9: footprint Resistor_SMD:R_0603_1608Metric_Pad1.05x0.95mm_HandSolder -> Resistor_SMD:R_1206_3216Metric_Pad1.42x1.75mm_HandSolder
Changed lines of the file:
@@
 $Descr A4 11693 8268
 encoding utf-8
-Sheet 5 7
+Sheet 4 7
 Title "LiPo Pack Monitor"
 Date "2021-12-20"
@@
 F 0 "R1" V 2457 2700 50  0000 C CNN
 F 1 "100Ω" V 2366 2700 50  0000 C CNN
-F 2 "Resistor_SMD:R_0603_1608Metric_Pad1.05x0.95mm_HandSolder" V 2180 2700 50  0001 C CNN
+F 2 "Resistor_SMD:R_1206_3216Metric_Pad1.42x1.75mm_HandSolder" V 2180 2700 50  0001 C CNN
 F 3 "~" H 2250 2700 50  0001 C CNN
 	1    2250 2700
@@
 F 0 "R2" V 2457 3100 50  0000 C CNN
 F 1 "100Ω" V 2366 3100 50  0000 C CNN
-F 2 "Resistor_SMD:R_0603_1608Metric_Pad1.05x0.95mm_HandSolder" V 2180 3100 50  0001 C CNN
+F 2 "Resistor_SMD:R_1206_3216Metric_Pad1.42x1.75mm_HandSolder" V 2180 3100 50  0001 C CNN
 F 3 "~" H 2250 3100 50  0001 C CNN
 	1    2250 3100
@@
 F 0 "R3" V 2457 3500 50  0000 C CNN
 F 1 "100Ω" V 2366 3500 50  0000 C CNN
-F 2 "Resistor_SMD:R_0603_1608Metric_Pad1.05x0.95mm_HandSolder" V 2180 3500 50  0001 C CNN
+F 2 "Resistor_SMD:R_1206_3216Metric_Pad1.42x1.75mm_HandSolder" V 2180 3500 50  0001 C CNN
 F 3 "~" H 2250 3500 50  0001 C CNN
 	1    2250 3500
@@
 F 0 "R4" V 2457 3900 50  0000 C CNN
 F 1 "100Ω" V 2366 3900 50  0000 C CNN
-F 2 "Resistor_SMD:R_0603_1608Metric_Pad1.05x0.95mm_HandSolder" V 2180 3900 50  0001 C CNN
+F 2 "Resistor_SMD:R_1206_3216Metric_Pad1.42x1.75mm_HandSolder" V 2180 3900 50  0001 C CNN
 F 3 "~" H 2250 3900 50  0001 C CNN
 	1    2250 3900
@@
 F 0 "R5" V 2457 4300 50  0000 C CNN
 F 1 "100Ω" V 2366 4300 50  0000 C CNN
-F 2 "Resistor_SMD:R_0603_1608Metric_Pad1.05x0.95mm_HandSolder" V 2180 4300 50  0001 C CNN
+F 2 "Resistor_SMD:R_1206_3216Metric_Pad1.42x1.75mm_HandSolder" V 2180 4300 50  0001 C CNN
 F 3 "~" H 2250 4300 50  0001 C CNN
 	1    2250 4300
@@
 F 0 "R6" V 2457 4900 50  0000 C CNN
 F 1 "100Ω" V 2366 4900 50  0000 C CNN
-F 2 "Resistor_SMD:R_0603_1608Metric_Pad1.05x0.95mm_HandSolder" V 2180 4900 50  0001 C CNN
+F 2 "Resistor_SMD:R_1206_3216Metric_Pad1.42x1.75mm_HandSolder" V 2180 4900 50  0001 C CNN
 F 3 "~" H 2250 4900 50  0001 C CNN
 	1    2250 4900
@@
 F 0 "C11" H 3042 2946 50  0000 L CNN
 F 1 "1μF" H 3042 2855 50  0000 L CNN
-F 2 "Capacitor_SMD:C_0603_1608Metric_Pad1.08x0.95mm_HandSolder" H 2950 2900 50  0001 C CNN
+F 2 "Capacitor_SMD:C_1206_3216Metric_Pad1.42x1.75mm_HandSolder" H 2950 2900 50  0001 C CNN
 F 3 "~" H 2950 2900 50  0001 C CNN
 	1    2950 2900
@@
 F 0 "C12" H 3042 3346 50  0000 L CNN
 F 1 "1μF" H 3042 3255 50  0000 L CNN
-F 2 "Capacitor_SMD:C_0603_1608Metric_Pad1.08x0.95mm_HandSolder" H 2950 3300 50  0001 C CNN
+F 2 "Capacitor_SMD:C_1206_3216Metric_Pad1.42x1.75mm_HandSolder" H 2950 3300 50  0001 C CNN
 F 3 "~" H 2950 3300 50  0001 C CNN
 	1    2950 3300
@@
 F 0 "C13" H 3042 3746 50  0000 L CNN
 F 1 "1μF" H 3042 3655 50  0000 L CNN
-F 2 "Capacitor_SMD:C_0603_1608Metric_Pad1.08x0.95mm_HandSolder" H 2950 3700 50  0001 C CNN
+F 2 "Capacitor_SMD:C_1206_3216Metric_Pad1.42x1.75mm_HandSolder" H 2950 3700 50  0001 C CNN
 F 3 "~" H 2950 3700 50  0001 C CNN
 	1    2950 3700
@@
 F 0 "C14" H 3042 4146 50  0000 L CNN
 F 1 "1μF" H 3042 4055 50  0000 L CNN
-F 2 "Capacitor_SMD:C_0603_1608Metric_Pad1.08x0.95mm_HandSolder" H 2950 4100 50  0001 C CNN
+F 2 "Capacitor_SMD:C_1206_3216Metric_Pad1.42x1.75mm_HandSolder" H 2950 4100 50  0001 C CNN
 F 3 "~" H 2950 4100 50  0001 C CNN
 	1    2950 4100
@@
 F 0 "C15" H 3042 4496 50  0000 L CNN
 F 1 "1μF" H 3042 4405 50  0000 L CNN
-F 2 "Capacitor_SMD:C_0603_1608Metric_Pad1.08x0.95mm_HandSolder" H 2950 4450 50  0001 C CNN
+F 2 "Capacitor_SMD:C_1206_3216Metric_Pad1.42x1.75mm_HandSolder" H 2950 4450 50  0001 C CNN
 F 3 "~" H 2950 4450 50  0001 C CNN
 	1    2950 4450
@@
 F 0 "C16" H 3042 4796 50  0000 L CNN
 F 1 "1μF" H 3042 4705 50  0000 L CNN
-F 2 "Capacitor_SMD:C_0603_1608Metric_Pad1.08x0.95mm_HandSolder" H 2950 4750 50  0001 C CNN
+F 2 "Capacitor_SMD:C_1206_3216Metric_Pad1.42x1.75mm_HandSolder" H 2950 4750 50  0001 C CNN
 F 3 "~" H 2950 4750 50  0001 C CNN
 	1    2950 4750
@@
 F 0 "C18" V 4471 5250 50  0000 C CNN
 F 1 "0.1μF" V 4562 5250 50  0000 C CNN
-F 2 "Capacitor_SMD:C_0603_1608Metric_Pad1.08x0.95mm_HandSolder" H 4700 5250 50  0001 C CNN
+F 2 "Resistor_SMD:R_0603_1608Metric_Pad1.05x0.95mm_HandSolder" H 4700 5250 50  0001 C CNN
 F 3 "~" H 4700 5250 50  0001 C CNN
 	1    4700 5250
@@
 F 0 "C20" V 5121 5250 50  0000 C CNN
 F 1 "0.1μF" V 5212 5250 50  0000 C CNN
-F 2 "Capacitor_SMD:C_0603_1608Metric_Pad1.08x0.95mm_HandSolder" H 5350 5250 50  0001 C CNN
+F 2 "Resistor_SMD:R_0603_1608Metric_Pad1.05x0.95mm_HandSolder" H 5350 5250 50  0001 C CNN
 F 3 "~" H 5350 5250 50  0001 C CNN
 	1    5350 5250
@@
 F 0 "C21" V 5871 5250 50  0000 C CNN
 F 1 "0.1μF" V 5962 5250 50  0000 C CNN
-F 2 "Capacitor_SMD:C_0603_1608Metric_Pad1.08x0.95mm_HandSolder" H 6100 5250 50  0001 C CNN
+F 2 "Resistor_SMD:R_0603_1608Metric_Pad1.05x0.95mm_HandSolder" H 6100 5250 50  0001 C CNN
 F 3 "~" H 6100 5250 50  0001 C CNN
 	1    6100 5250
@@
 F 0 "C23" H 8058 3604 50  0000 R CNN
 F 1 "1μF" H 8058 3695 50  0000 R CNN
-F 2 "Capacitor_SMD:C_0603_1608Metric_Pad1.08x0.95mm_HandSolder" H 8150 3650 50  0001 C CNN
+F 2 "Capacitor_SMD:C_1206_3216Metric_Pad1.42x1.75mm_HandSolder" H 8150 3650 50  0001 C CNN
 F 3 "~" H 8150 3650 50  0001 C CNN
 	1    8150 3650
@@
 F 0 "C22" H 7808 1954 50  0000 R CNN
 F 1 "1μF" H 7808 2045 50  0000 R CNN
-F 2 "Capacitor_SMD:C_0603_1608Metric_Pad1.08x0.95mm_HandSolder" H 7900 2000 50  0001 C CNN
+F 2 "Capacitor_SMD:C_1206_3216Metric_Pad1.42x1.75mm_HandSolder" H 7900 2000 50  0001 C CNN
 F 3 "~" H 7900 2000 50  0001 C CNN
 	1    7900 2000
@@
 F 0 "C19" H 5158 2854 50  0000 R CNN
 F 1 "10μF" H 5158 2945 50  0000 R CNN
-F 2 "Capacitor_SMD:C_0603_1608Metric_Pad1.08x0.95mm_HandSolder" H 5250 2900 50  0001 C CNN
+F 2 "Capacitor_SMD:C_1206_3216Metric_Pad1.42x1.75mm_HandSolder" H 5250 2900 50  0001 C CNN
 F 3 "~" H 5250 2900 50  0001 C CNN
 	1    5250 2900
@@
 F 0 "R9" H 5180 2096 50  0000 R CNN
 F 1 "100Ω" H 5180 2005 50  0000 R CNN
-F 2 "Resistor_SMD:R_0603_1608Metric_Pad1.05x0.95mm_HandSolder" V 5180 2050 50  0001 C CNN
+F 2 "Resistor_SMD:R_1206_3216Metric_Pad1.42x1.75mm_HandSolder" V 5180 2050 50  0001 C CNN
 F 3 "~" H 5250 2050 50  0001 C CNN
 	1    5250 2050

Commit message: Routed all connections and placed all components
MCU crystal still needs a ground peninsula
Parts:
- C23: footprint Capacitor_SMD:C_1206_3216Metric_Pad1.42x1.75mm_HandSolder -> Capacitor_SMD:C_0603_1608Metric_Pad1.08x0.95mm_HandSolder
Changed lines of the file:
@@
 F 0 "C23" H 8058 3604 50  0000 R CNN
 F 1 "1μF" H 8058 3695 50  0000 R CNN
-F 2 "Capacitor_SMD:C_1206_3216Metric_Pad1.42x1.75mm_HandSolder" H 8150 3650 50  0001 C CNN
+F 2 "Capacitor_SMD:C_0603_1608Metric_Pad1.08x0.95mm_HandSolder" H 8150 3650 50  0001 C CNN
 F 3 "~" H 8150 3650 50  0001 C CNN
 	1    8150 3650
