File: Hardware/COMPONENT_SHEETS/MCU_STM32L562VET6Q.sch (KiCad schematic (older format))
At the start: 11 parts, among them Y1 Crystal

Commit message: FIxed board
issues with the board after the merge have been fixed
Parts:
- gave numbers to parts that had none: 1
- renumbered C3 to C2, C4 to C3, C5 to C4, C6 to C5, C7 to C6
Changed lines of the file:
@@
 P 1700 4050
 AR Path="/61614678" Ref="C?"  Part="1"
-AR Path="/6160DF75/61614678" Ref="C3"  Part="1"
-F 0 "C3" H 1608 4004 50  0000 R CNN
+AR Path="/6160DF75/61614678" Ref="C2"  Part="1"
+F 0 "C2" H 1608 4004 50  0000 R CNN
 F 1 "1uF" H 1608 4095 50  0000 R CNN
 F 2 "Capacitor_SMD:C_0603_1608Metric" H 1700 4050 50  0001 C CNN
@@
 P 2100 4050
 AR Path="/6161467E" Ref="C?"  Part="1"
-AR Path="/6160DF75/6161467E" Ref="C4"  Part="1"
-F 0 "C4" H 2008 4004 50  0000 R CNN
+AR Path="/6160DF75/6161467E" Ref="C3"  Part="1"
+F 0 "C3" H 2008 4004 50  0000 R CNN
 F 1 "100nF" H 2008 4095 50  0000 R CNN
 F 2 "Capacitor_SMD:C_0603_1608Metric" H 2100 4050 50  0001 C CNN
@@
 P 2500 4050
 AR Path="/61614684" Ref="C?"  Part="1"
-AR Path="/6160DF75/61614684" Ref="C5"  Part="1"
-F 0 "C5" H 2408 4004 50  0000 R CNN
+AR Path="/6160DF75/61614684" Ref="C4"  Part="1"
+F 0 "C4" H 2408 4004 50  0000 R CNN
 F 1 "100nF" H 2408 4095 50  0000 R CNN
 F 2 "Capacitor_SMD:C_0603_1608Metric" H 2500 4050 50  0001 C CNN
@@
 P 1700 3800
 AR Path="/61614698" Ref="#PWR?"  Part="1"
-AR Path="/6160DF75/61614698" Ref="#PWR06"  Part="1"
-F 0 "#PWR06" H 1700 3650 50  0001 C CNN
+AR Path="/6160DF75/61614698" Ref="#PWR05"  Part="1"
+F 0 "#PWR05" H 1700 3650 50  0001 C CNN
 F 1 "+3.3V" H 1715 3973 50  0000 C CNN
 F 2 "" H 1700 3800 50  0001 C CNN
@@
 P 6850 2550
 AR Path="/6161463B" Ref="#PWR?"  Part="1"
-AR Path="/6160DF75/6161463B" Ref="#PWR07"  Part="1"
-F 0 "#PWR07" H 6850 2400 50  0001 C CNN
+AR Path="/6160DF75/6161463B" Ref="#PWR06"  Part="1"
+F 0 "#PWR06" H 6850 2400 50  0001 C CNN
 F 1 "+3.3V" H 6865 2723 50  0000 C CNN
 F 2 "" H 6850 2550 50  0001 C CNN
@@
 P 6050 6600
 AR Path="/61614648" Ref="C?"  Part="1"
-AR Path="/6160DF75/61614648" Ref="C7"  Part="1"
-F 0 "C7" H 5958 6554 50  0000 R CNN
+AR Path="/6160DF75/61614648" Ref="C6"  Part="1"
+F 0 "C6" H 5958 6554 50  0000 R CNN
 F 1 "30pF" H 5958 6645 50  0000 R CNN
 F 2 "Capacitor_SMD:C_0603_1608Metric" H 6050 6600 50  0001 C CNN
@@
 P 5450 6600
 AR Path="/6161464E" Ref="C?"  Part="1"
-AR Path="/6160DF75/6161464E" Ref="C6"  Part="1"
-F 0 "C6" H 5358 6554 50  0000 R CNN
+AR Path="/6160DF75/6161464E" Ref="C5"  Part="1"
+F 0 "C5" H 5358 6554 50  0000 R CNN
 F 1 "30pF" H 5358 6645 50  0000 R CNN
 F 2 "Capacitor_SMD:C_0603_1608Metric" H 5450 6600 50  0001 C CNN
@@
 	5450 6000 5450 6350
 $Comp
-L Power_KiCAD_Project-rescue:STM32L562VET6Q-SamacSys_Parts IC?
+L Power_KiCAD_Project-rescue:STM32L562VET6Q-SamacSys_Parts IC1
 U 1 1 61BFCBF3
 P 3850 2550
-F 0 "IC?" H 5350 1400 50  0000 L CNN
+F 0 "IC1" H 5350 1400 50  0000 L CNN
 F 1 "STM32L562VET6Q" H 5100 1300 50  0000 L CNN
 F 2 "SamacSys_Parts:QFP50P1600X1600X160-100N" H 6700 3250 50  0001 L CNN

Commit message: Replaced passive component footprints with handsolder variants
I think the component sheet for the MCU STM32L152VET6Q is incorrect. Will investigate.
Parts:
- C2, C3, C4, C5, C6: footprint Capacitor_SMD:C_0603_1608Metric -> Capacitor_SMD:C_0603_1608Metric_Pad1.08x0.95mm_HandSolder
- D1, D2: footprint LED_SMD:LED_0603_1608Metric -> LED_SMD:LED_0603_1608Metric_Pad1.05x0.95mm_HandSolder
- R1, R2: footprint Resistor_SMD:R_0603_1608Metric -> Resistor_SMD:R_0603_1608Metric_Pad1.05x0.95mm_HandSolder
Changed lines of the file:
@@
 F 0 "C2" H 1608 4004 50  0000 R CNN
 F 1 "1uF" H 1608 4095 50  0000 R CNN
-F 2 "Capacitor_SMD:C_0603_1608Metric" H 1700 4050 50  0001 C CNN
+F 2 "Capacitor_SMD:C_0603_1608Metric_Pad1.08x0.95mm_HandSolder" H 1700 4050 50  0001 C CNN
 F 3 "~" H 1700 4050 50  0001 C CNN
 	1    1700 4050
@@
 F 0 "C3" H 2008 4004 50  0000 R CNN
 F 1 "100nF" H 2008 4095 50  0000 R CNN
-F 2 "Capacitor_SMD:C_0603_1608Metric" H 2100 4050 50  0001 C CNN
+F 2 "Capacitor_SMD:C_0603_1608Metric_Pad1.08x0.95mm_HandSolder" H 2100 4050 50  0001 C CNN
 F 3 "~" H 2100 4050 50  0001 C CNN
 	1    2100 4050
@@
 F 0 "C4" H 2408 4004 50  0000 R CNN
 F 1 "100nF" H 2408 4095 50  0000 R CNN
-F 2 "Capacitor_SMD:C_0603_1608Metric" H 2500 4050 50  0001 C CNN
+F 2 "Capacitor_SMD:C_0603_1608Metric_Pad1.08x0.95mm_HandSolder" H 2500 4050 50  0001 C CNN
 F 3 "~" H 2500 4050 50  0001 C CNN
 	1    2500 4050
@@
 F 0 "R2" H 7920 3096 50  0000 L CNN
 F 1 "1k5Ω" H 7920 3005 50  0000 L CNN
-F 2 "Resistor_SMD:R_0603_1608Metric" V 7780 3050 50  0001 C CNN
+F 2 "Resistor_SMD:R_0603_1608Metric_Pad1.05x0.95mm_HandSolder" V 7780 3050 50  0001 C CNN
 F 3 "~" H 7850 3050 50  0001 C CNN
 	1    7850 3050
@@
 F 0 "D2" V 7889 3332 50  0000 R CNN
 F 1 "RED" V 7798 3332 50  0000 R CNN
-F 2 "LED_SMD:LED_0603_1608Metric" H 7850 3450 50  0001 C CNN
+F 2 "LED_SMD:LED_0603_1608Metric_Pad1.05x0.95mm_HandSolder" H 7850 3450 50  0001 C CNN
 F 3 "~" H 7850 3450 50  0001 C CNN
 	1    7850 3450
@@
 F 0 "D1" V 7539 3332 50  0000 R CNN
 F 1 "GREEN" V 7448 3332 50  0000 R CNN
-F 2 "LED_SMD:LED_0603_1608Metric" H 7500 3450 50  0001 C CNN
+F 2 "LED_SMD:LED_0603_1608Metric_Pad1.05x0.95mm_HandSolder" H 7500 3450 50  0001 C CNN
 F 3 "~" H 7500 3450 50  0001 C CNN
 	1    7500 3450
@@
 F 0 "R1" H 7570 3096 50  0000 L CNN
 F 1 "1k5Ω" H 7570 3005 50  0000 L CNN
-F 2 "Resistor_SMD:R_0603_1608Metric" V 7430 3050 50  0001 C CNN
+F 2 "Resistor_SMD:R_0603_1608Metric_Pad1.05x0.95mm_HandSolder" V 7430 3050 50  0001 C CNN
 F 3 "~" H 7500 3050 50  0001 C CNN
 	1    7500 3050
@@
 F 0 "C6" H 5958 6554 50  0000 R CNN
 F 1 "30pF" H 5958 6645 50  0000 R CNN
-F 2 "Capacitor_SMD:C_0603_1608Metric" H 6050 6600 50  0001 C CNN
+F 2 "Capacitor_SMD:C_0603_1608Metric_Pad1.08x0.95mm_HandSolder" H 6050 6600 50  0001 C CNN
 F 3 "~" H 6050 6600 50  0001 C CNN
 	1    6050 6600
@@
 F 0 "C5" H 5358 6554 50  0000 R CNN
 F 1 "30pF" H 5358 6645 50  0000 R CNN
-F 2 "Capacitor_SMD:C_0603_1608Metric" H 5450 6600 50  0001 C CNN
+F 2 "Capacitor_SMD:C_0603_1608Metric_Pad1.08x0.95mm_HandSolder" H 5450 6600 50  0001 C CNN
 F 3 "~" H 5450 6600 50  0001 C CNN
 	1    5450 6600
