File: Hardware/COMPONENT_SHEETS/TEMPSENSOR_MCP9808.sch (KiCad schematic (older format))
At the start: 2 parts, among them U2 MCP9808_MSOP

Commit message: FIxed board
issues with the board after the merge have been fixed
Parts:
- renumbered C2 to C7
Changed lines of the file:
@@
 $Descr A4 11693 8268
 encoding utf-8
-Sheet 2 7
+Sheet 4 7
 Title "MCP9608 Temperature Sensor"
 Date "2021-12-06"
@@
 AR Path="/6160E323" Ref="#PWR?"  Part="1"
 AR Path="/615C1FB4/6160E323" Ref="#PWR?"  Part="1"
-AR Path="/61B1B3BC/6160E323" Ref="#PWR?"  Part="1"
-AR Path="/61B35621/6160E323" Ref="#PWR05"  Part="1"
-F 0 "#PWR05" H 3700 2300 50  0001 C CNN
+AR Path="/61B1B3BC/6160E323" Ref="#PWR07"  Part="1"
+AR Path="/61B35621/6160E323" Ref="#PWR04"  Part="1"
+F 0 "#PWR07" H 3700 2300 50  0001 C CNN
 F 1 "+3.3V" H 3715 2623 50  0000 C CNN
 F 2 "" H 3700 2450 50  0001 C CNN
@@
 AR Path="/6160E331" Ref="C?"  Part="1"
 AR Path="/615C1FB4/6160E331" Ref="C?"  Part="1"
-AR Path="/61B1B3BC/6160E331" Ref="C?"  Part="1"
-AR Path="/61B35621/6160E331" Ref="C2"  Part="1"
-F 0 "C2" H 4365 3146 50  0000 L CNN
+AR Path="/61B1B3BC/6160E331" Ref="C7"  Part="1"
+AR Path="/61B35621/6160E331" Ref="C1"  Part="1"
+F 0 "C7" H 4365 3146 50  0000 L CNN
 F 1 "100nF" H 4365 3055 50  0000 L CNN
 F 2 "Capacitor_SMD:C_0603_1608Metric" H 4288 2950 50  0001 C CNN
@@
 AR Path="/61A8C2DF" Ref="U?"  Part="1"
 AR Path="/615C1FB4/61A8C2DF" Ref="U?"  Part="1"
-AR Path="/61B1B3BC/61A8C2DF" Ref="U?"  Part="1"
-AR Path="/61B35621/61A8C2DF" Ref="U2"  Part="1"
+AR Path="/61B1B3BC/61A8C2DF" Ref="U2"  Part="1"
+AR Path="/61B35621/61A8C2DF" Ref="U1"  Part="1"
 F 0 "U2" H 3200 3800 50  0000 L CNN
 F 1 "MCP9808_MSOP" H 2950 3700 50  0000 L CNN

Commit message: Replaced passive component footprints with handsolder variants
I think the component sheet for the MCU STM32L152VET6Q is incorrect. Will investigate.
Parts:
- C7: footprint Capacitor_SMD:C_0603_1608Metric -> Capacitor_SMD:C_0603_1608Metric_Pad1.08x0.95mm_HandSolder
Changed lines of the file:
@@
 $Descr A4 11693 8268
 encoding utf-8
-Sheet 4 7
+Sheet 2 7
 Title "MCP9608 Temperature Sensor"
 Date "2021-12-06"
@@
 AR Path="/61B1B3BC/6160E331" Ref="C7"  Part="1"
 AR Path="/61B35621/6160E331" Ref="C1"  Part="1"
-F 0 "C7" H 4365 3146 50  0000 L CNN
+F 0 "C1" H 4365 3146 50  0000 L CNN
 F 1 "100nF" H 4365 3055 50  0000 L CNN
-F 2 "Capacitor_SMD:C_0603_1608Metric" H 4288 2950 50  0001 C CNN
+F 2 "Capacitor_SMD:C_0603_1608Metric_Pad1.08x0.95mm_HandSolder" H 4288 2950 50  0001 C CNN
 F 3 "~" H 4250 3100 50  0001 C CNN
 	1    4250 3100
@@
 AR Path="/61B1B3BC/61A8C2DF" Ref="U2"  Part="1"
 AR Path="/61B35621/61A8C2DF" Ref="U1"  Part="1"
-F 0 "U2" H 3200 3800 50  0000 L CNN
+F 0 "U1" H 3200 3800 50  0000 L CNN
 F 1 "MCP9808_MSOP" H 2950 3700 50  0000 L CNN
 F 2 "Package_SO:MSOP-8_3x3mm_P0.65mm" H 3250 3050 50  0001 C CNN
