File: Hardware/COMPONENT_SHEETS/TEMPSENSOR_MCP9808.sch (KiCad schematic (older format))
At the start: 2 parts, among them U2 MCP9808_MSOP

Commit message: Routed I2C lines between temp sensors, lipo monitor, and mcu
Changed lines of the file:
@@
 $Descr A4 11693 8268
 encoding utf-8
-Sheet 3 7
+Sheet 2 7
 Title "MCP9608 Temperature Sensor"
 Date "2021-12-20"
@@
 AR Path="/61B1B3BC/6160E331" Ref="C2"  Part="1"
 AR Path="/61B35621/6160E331" Ref="C1"  Part="1"
-F 0 "C2" H 4365 3146 50  0000 L CNN
+F 0 "C1" H 4365 3146 50  0000 L CNN
 F 1 "100nF" H 4365 3055 50  0000 L CNN
 F 2 "Capacitor_SMD:C_0603_1608Metric_Pad1.08x0.95mm_HandSolder" H 4288 2950 50  0001 C CNN
@@
 AR Path="/61B1B3BC/61A8C2DF" Ref="U2"  Part="1"
 AR Path="/61B35621/61A8C2DF" Ref="U1"  Part="1"
-F 0 "U2" H 3200 3800 50  0000 L CNN
+F 0 "U1" H 3200 3800 50  0000 L CNN
 F 1 "MCP9808_MSOP" H 2950 3700 50  0000 L CNN
 F 2 "Package_SO:MSOP-8_3x3mm_P0.65mm" H 3250 3050 50  0001 C CNN

Commit message: More adjustments of internal planes
Changed lines of the file:
@@
 $Descr A4 11693 8268
 encoding utf-8
-Sheet 7 7
+Sheet 2 7
 Title "MCP9608 Temperature Sensor"
 Date "2021-12-20"
@@
 AR Path="/61B1B3BC/6160E323" Ref="#PWR011"  Part="1"
 AR Path="/61B35621/6160E323" Ref="#PWR08"  Part="1"
-F 0 "#PWR08" H 3700 2300 50  0001 C CNN
+F 0 "#PWR011" H 3700 2300 50  0001 C CNN
 F 1 "+3.3V" H 3715 2623 50  0000 C CNN
 F 2 "" H 3700 2450 50  0001 C CNN
@@
 AR Path="/61B1B3BC/6160E331" Ref="C2"  Part="1"
 AR Path="/61B35621/6160E331" Ref="C1"  Part="1"
-F 0 "C1" H 4365 3146 50  0000 L CNN
+F 0 "C2" H 4365 3146 50  0000 L CNN
 F 1 "100nF" H 4365 3055 50  0000 L CNN
 F 2 "Capacitor_SMD:C_0603_1608Metric_Pad1.08x0.95mm_HandSolder" H 4288 2950 50  0001 C CNN
@@
 AR Path="/61B1B3BC/61A8C2DF" Ref="U2"  Part="1"
 AR Path="/61B35621/61A8C2DF" Ref="U1"  Part="1"
-F 0 "U1" H 3200 3800 50  0000 L CNN
+F 0 "U2" H 3200 3800 50  0000 L CNN
 F 1 "MCP9808_MSOP" H 2950 3700 50  0000 L CNN
 F 2 "Package_SO:MSOP-8_3x3mm_P0.65mm" H 3250 3050 50  0001 C CNN
@@
 AR Path="/61B1B3BC/61CCAD29" Ref="#PWR012"  Part="1"
 AR Path="/61B35621/61CCAD29" Ref="#PWR09"  Part="1"
-F 0 "#PWR09" H 4250 3000 50  0001 C CNN
+F 0 "#PWR012" H 4250 3000 50  0001 C CNN
 F 1 "GND" H 4255 3077 50  0000 C CNN
 F 2 "" H 4250 3250 50  0001 C CNN
@@
 AR Path="/61B1B3BC/61CCAD97" Ref="#PWR010"  Part="1"
 AR Path="/61B35621/61CCAD97" Ref="#PWR07"  Part="1"
-F 0 "#PWR07" H 3250 3400 50  0001 C CNN
+F 0 "#PWR010" H 3250 3400 50  0001 C CNN
 F 1 "GND" H 3255 3477 50  0000 C CNN
 F 2 "" H 3250 3650 50  0001 C CNN

Commit message: Routed all connections and placed all components
MCU crystal still needs a ground peninsula
Changed lines of the file:
@@
 $Descr A4 11693 8268
 encoding utf-8
-Sheet 2 7
+Sheet 7 7
 Title "MCP9608 Temperature Sensor"
 Date "2021-12-20"
@@
 AR Path="/61B1B3BC/6160E323" Ref="#PWR011"  Part="1"
 AR Path="/61B35621/6160E323" Ref="#PWR08"  Part="1"
-F 0 "#PWR011" H 3700 2300 50  0001 C CNN
+F 0 "#PWR08" H 3700 2300 50  0001 C CNN
 F 1 "+3.3V" H 3715 2623 50  0000 C CNN
 F 2 "" H 3700 2450 50  0001 C CNN
@@
 AR Path="/61B1B3BC/6160E331" Ref="C2"  Part="1"
 AR Path="/61B35621/6160E331" Ref="C1"  Part="1"
-F 0 "C2" H 4365 3146 50  0000 L CNN
+F 0 "C1" H 4365 3146 50  0000 L CNN
 F 1 "100nF" H 4365 3055 50  0000 L CNN
 F 2 "Capacitor_SMD:C_0603_1608Metric_Pad1.08x0.95mm_HandSolder" H 4288 2950 50  0001 C CNN
@@
 AR Path="/61B1B3BC/61A8C2DF" Ref="U2"  Part="1"
 AR Path="/61B35621/61A8C2DF" Ref="U1"  Part="1"
-F 0 "U2" H 3200 3800 50  0000 L CNN
+F 0 "U1" H 3200 3800 50  0000 L CNN
 F 1 "MCP9808_MSOP" H 2950 3700 50  0000 L CNN
 F 2 "Package_SO:MSOP-8_3x3mm_P0.65mm" H 3250 3050 50  0001 C CNN
@@
 AR Path="/61B1B3BC/61CCAD29" Ref="#PWR012"  Part="1"
 AR Path="/61B35621/61CCAD29" Ref="#PWR09"  Part="1"
-F 0 "#PWR012" H 4250 3000 50  0001 C CNN
+F 0 "#PWR09" H 4250 3000 50  0001 C CNN
 F 1 "GND" H 4255 3077 50  0000 C CNN
 F 2 "" H 4250 3250 50  0001 C CNN
@@
 AR Path="/61B1B3BC/61CCAD97" Ref="#PWR010"  Part="1"
 AR Path="/61B35621/61CCAD97" Ref="#PWR07"  Part="1"
-F 0 "#PWR010" H 3250 3400 50  0001 C CNN
+F 0 "#PWR07" H 3250 3400 50  0001 C CNN
 F 1 "GND" H 3255 3477 50  0000 C CNN
 F 2 "" H 3250 3650 50  0001 C CNN
