File: Hardware/COMPONENT_SHEETS/DSUB-slot.sch (KiCad schematic (older format))
At the start: 2 parts, among them J8 L717SDC37P1ACH4F

Commit message: Replaced passive component footprints with handsolder variants
I think the component sheet for the MCU STM32L152VET6Q is incorrect. Will investigate.
Parts:
- C8: footprint Capacitor_SMD:C_0603_1608Metric -> Capacitor_SMD:C_0603_1608Metric_Pad1.08x0.95mm_HandSolder
Changed lines of the file:
@@
 F 0 "C8" H 5292 2446 50  0000 L CNN
 F 1 "100nF" H 5292 2355 50  0000 L CNN
-F 2 "Capacitor_SMD:C_0603_1608Metric" H 5200 2400 50  0001 C CNN
+F 2 "Capacitor_SMD:C_0603_1608Metric_Pad1.08x0.95mm_HandSolder" H 5200 2400 50  0001 C CNN
 F 3 "~" H 5200 2400 50  0001 C CNN
 	1    5200 2400

Commit message: Component sheets added
Component sheets were added from the telemetry board to match across all boards
Parts:
- C29: renamed from C8; footprint Capacitor_SMD:C_0603_1608Metric_Pad1.08x0.95mm_HandSolder -> Capacitor_SMD:C_0603_1608Metric
- J7: renamed from J8; symbol Power_KiCAD_Project-rescue:L717SDC37P1ACH4F-SamacSys_Parts -> SamacSys_Parts:L717SDC37P1ACH4F
Changed lines of the file:
@@
 $Descr A4 11693 8268
 encoding utf-8
-Sheet 5 7
+Sheet 6 7
 Title ""
-Date "2021-12-06"
+Date ""
 Rev ""
-Comp "Missouri S&T Rocket Design Team '21 (Jacob King)"
+Comp ""
 Comment1 ""
 Comment2 ""
@@
 AR Path="/61A55586" Ref="C?"  Part="1"
 AR Path="/61A437B5/61A55586" Ref="C?"  Part="1"
-AR Path="/61D3585E/61A55586" Ref="C8"  Part="1"
-F 0 "C8" H 5292 2446 50  0000 L CNN
+AR Path="/61D3585E/61A55586" Ref="C29"  Part="1"
+F 0 "C29" H 5292 2446 50  0000 L CNN
 F 1 "100nF" H 5292 2355 50  0000 L CNN
-F 2 "Capacitor_SMD:C_0603_1608Metric_Pad1.08x0.95mm_HandSolder" H 5200 2400 50  0001 C CNN
+F 2 "Capacitor_SMD:C_0603_1608Metric" H 5200 2400 50  0001 C CNN
 F 3 "~" H 5200 2400 50  0001 C CNN
 	1    5200 2400
@@
 	5300 2400 5700 2400
 $Comp
-L power:+3.3V #PWR010
+L power:+3.3V #PWR022
 U 1 1 61A4A3FB
 P 6700 2000
-F 0 "#PWR010" H 6700 1850 50  0001 C CNN
+F 0 "#PWR022" H 6700 1850 50  0001 C CNN
 F 1 "+3.3V" V 6715 2128 50  0000 L CNN
 F 2 "" H 6700 2000 50  0001 C CNN
@@
 $EndComp
 $Comp
-L power:+5V #PWR08
+L power:+5V #PWR020
 U 1 1 61A491E6
 P 5700 1900
-F 0 "#PWR08" H 5700 1750 50  0001 C CNN
+F 0 "#PWR020" H 5700 1750 50  0001 C CNN
 F 1 "+5V" V 5715 2028 50  0000 L CNN
 F 2 "" H 5700 1900 50  0001 C CNN
@@
 $EndComp
 $Comp
-L power:+3.3V #PWR011
+L power:+3.3V #PWR023
 U 1 1 61A4AB5D
 P 6700 3600
-F 0 "#PWR011" H 6700 3450 50  0001 C CNN
+F 0 "#PWR023" H 6700 3450 50  0001 C CNN
 F 1 "+3.3V" V 6715 3728 50  0000 L CNN
 F 2 "" H 6700 3600 50  0001 C CNN
@@
 $EndComp
 $Comp
-L Power_KiCAD_Project-rescue:L717SDC37P1ACH4F-SamacSys_Parts J8
+L SamacSys_Parts:L717SDC37P1ACH4F J7
 U 1 1 61D5E9EE
 P 6200 1600
-F 0 "J8" V 6019 1600 50  0000 C CNN
+F 0 "J7" V 6019 1600 50  0000 C CNN
 F 1 "L717SDC37P1ACH4F" V 6110 1600 50  0000 C CNN
 F 2 "SamacSys_Parts:L717SDC37P1ACH4F" H 8450 1900 50  0001 L CNN
@@
 	6850 3700 6700 3700
 $Comp
-L power:+5V #PWR09
+L power:+5V #PWR021
 U 1 1 61A49AB4
 P 5700 3600
-F 0 "#PWR09" H 5700 3450 50  0001 C CNN
+F 0 "#PWR021" H 5700 3450 50  0001 C CNN
 F 1 "+5V" V 5715 3728 50  0000 L CNN
 F 2 "" H 5700 3600 50  0001 C CNN
