File: Hardware/COMPONENT_SHEETS/DSUB-slot.sch (KiCad schematic (older format))
At the start: 2 parts

Commit message: FIxed board
issues with the board after the merge have been fixed
Parts:
- gave numbers to parts that had none: 1
- renumbered C16 to C8
Changed lines of the file:
@@
 AR Path="/61A55586" Ref="C?"  Part="1"
 AR Path="/61A437B5/61A55586" Ref="C?"  Part="1"
-AR Path="/61D3585E/61A55586" Ref="C16"  Part="1"
-F 0 "C16" H 5292 2446 50  0000 L CNN
+AR Path="/61D3585E/61A55586" Ref="C8"  Part="1"
+F 0 "C8" H 5292 2446 50  0000 L CNN
 F 1 "100nF" H 5292 2355 50  0000 L CNN
 F 2 "Capacitor_SMD:C_0603_1608Metric" H 5200 2400 50  0001 C CNN
@@
 	5300 2400 5700 2400
 $Comp
-L power:+3.3V #PWR?
+L power:+3.3V #PWR010
 U 1 1 61A4A3FB
 P 6700 2000
-F 0 "#PWR?" H 6700 1850 50  0001 C CNN
+F 0 "#PWR010" H 6700 1850 50  0001 C CNN
 F 1 "+3.3V" V 6715 2128 50  0000 L CNN
 F 2 "" H 6700 2000 50  0001 C CNN
@@
 $EndComp
 $Comp
-L power:+5V #PWR?
+L power:+5V #PWR08
 U 1 1 61A491E6
 P 5700 1900
-F 0 "#PWR?" H 5700 1750 50  0001 C CNN
+F 0 "#PWR08" H 5700 1750 50  0001 C CNN
 F 1 "+5V" V 5715 2028 50  0000 L CNN
 F 2 "" H 5700 1900 50  0001 C CNN
@@
 $EndComp
 $Comp
-L power:+3.3V #PWR?
+L power:+3.3V #PWR011
 U 1 1 61A4AB5D
 P 6700 3600
-F 0 "#PWR?" H 6700 3450 50  0001 C CNN
+F 0 "#PWR011" H 6700 3450 50  0001 C CNN
 F 1 "+3.3V" V 6715 3728 50  0000 L CNN
 F 2 "" H 6700 3600 50  0001 C CNN
@@
 $EndComp
 $Comp
-L Power_KiCAD_Project-rescue:L717SDC37P1ACH4F-SamacSys_Parts J?
+L Power_KiCAD_Project-rescue:L717SDC37P1ACH4F-SamacSys_Parts J8
 U 1 1 61D5E9EE
 P 6200 1600
-F 0 "J?" V 6019 1600 50  0000 C CNN
+F 0 "J8" V 6019 1600 50  0000 C CNN
 F 1 "L717SDC37P1ACH4F" V 6110 1600 50  0000 C CNN
 F 2 "SamacSys_Parts:L717SDC37P1ACH4F" H 8450 1900 50  0001 L CNN
@@
 	6850 3700 6700 3700
 $Comp
-L power:+5V #PWR?
+L power:+5V #PWR09
 U 1 1 61A49AB4
 P 5700 3600
-F 0 "#PWR?" H 5700 3450 50  0001 C CNN
+F 0 "#PWR09" H 5700 3450 50  0001 C CNN
 F 1 "+5V" V 5715 3728 50  0000 L CNN
 F 2 "" H 5700 3600 50  0001 C CNN

Commit message: Rearranged LiPo Monitor component sheet
 - Added XT60 connector for external switch connection
 - Updated a few component symbols to be the default ones
 - Replaced label "ground" with the GNDREF symbol
 - LiPo Pack Monitor I2C and Alert Lines still need to be added
Parts:
- renumbered J8 to J12
Changed lines of the file:
@@
 $Descr A4 11693 8268
 encoding utf-8
-Sheet 5 7
+Sheet 5 8
 Title ""
-Date "2021-12-06"
-Rev ""
-Comp "Missouri S&T Rocket Design Team '21 (Jacob King)"
+Date "2021-12-20"
+Rev "v2.0.1"
+Comp "Missouri S&T Rocket Design Team '21 (Jacob King, Thomas Francois)"
 Comment1 ""
 Comment2 ""
@@
 	5300 2400 5700 2400
 $Comp
-L power:+3.3V #PWR010
+L power:+3.3V #PWR015
 U 1 1 61A4A3FB
 P 6700 2000
-F 0 "#PWR010" H 6700 1850 50  0001 C CNN
+F 0 "#PWR015" H 6700 1850 50  0001 C CNN
 F 1 "+3.3V" V 6715 2128 50  0000 L CNN
 F 2 "" H 6700 2000 50  0001 C CNN
@@
 $EndComp
 $Comp
-L power:+5V #PWR08
+L power:+5V #PWR013
 U 1 1 61A491E6
 P 5700 1900
-F 0 "#PWR08" H 5700 1750 50  0001 C CNN
+F 0 "#PWR013" H 5700 1750 50  0001 C CNN
 F 1 "+5V" V 5715 2028 50  0000 L CNN
 F 2 "" H 5700 1900 50  0001 C CNN
@@
 $EndComp
 $Comp
-L power:+3.3V #PWR011
+L power:+3.3V #PWR016
 U 1 1 61A4AB5D
 P 6700 3600
-F 0 "#PWR011" H 6700 3450 50  0001 C CNN
+F 0 "#PWR016" H 6700 3450 50  0001 C CNN
 F 1 "+3.3V" V 6715 3728 50  0000 L CNN
 F 2 "" H 6700 3600 50  0001 C CNN
@@
 $EndComp
 $Comp
-L Power_KiCAD_Project-rescue:L717SDC37P1ACH4F-SamacSys_Parts J8
+L Power_KiCAD_Project-rescue:L717SDC37P1ACH4F-SamacSys_Parts J12
 U 1 1 61D5E9EE
 P 6200 1600
-F 0 "J8" V 6019 1600 50  0000 C CNN
+F 0 "J12" V 6019 1600 50  0000 C CNN
 F 1 "L717SDC37P1ACH4F" V 6110 1600 50  0000 C CNN
 F 2 "SamacSys_Parts:L717SDC37P1ACH4F" H 8450 1900 50  0001 L CNN
@@
 	6850 3700 6700 3700
 $Comp
-L power:+5V #PWR09
+L power:+5V #PWR014
 U 1 1 61A49AB4
 P 5700 3600
-F 0 "#PWR09" H 5700 3450 50  0001 C CNN
+F 0 "#PWR014" H 5700 3450 50  0001 C CNN
 F 1 "+5V" V 5715 3728 50  0000 L CNN
 F 2 "" H 5700 3600 50  0001 C CNN

Commit message: Fixed ground symbols in component sheets, corrected MCU sheet
Connections:
- net labels added: GND
- net labels removed: ground
Changed lines of the file:
@@
 $Descr A4 11693 8268
 encoding utf-8
-Sheet 5 8
+Sheet 4 7
 Title ""
 Date "2021-12-20"
@@
 	0    -1   1    0
 $EndComp
-Text HLabel 6200 1600 2    50   Input ~ 0
-ground
-Text HLabel 6700 1900 2    50   Input ~ 0
-ground
-Text HLabel 6850 3700 2    50   Input ~ 0
-ground
-Text HLabel 6200 4000 3    50   Input ~ 0
-ground
-Text HLabel 5100 2400 0    50   Input ~ 0
-ground
+$Comp
+L power:GND #PWR?
+U 1 1 61CC9506
+P 6850 3700
+AR Path="/61CC9506" Ref="#PWR?"  Part="1"
+AR Path="/61D3585E/61CC9506" Ref="#PWR?"  Part="1"
+F 0 "#PWR?" H 6850 3450 50  0001 C CNN
+F 1 "GND" H 6855 3527 50  0000 C CNN
+F 2 "" H 6850 3700 50  0001 C CNN
+F 3 "" H 6850 3700 50  0001 C CNN
+	1    6850 3700
+	1    0    0    -1
+$EndComp
+$Comp
+L power:GND #PWR?
+U 1 1 61CC95A1
+P 6200 4000
+AR Path="/61CC95A1" Ref="#PWR?"  Part="1"
+AR Path="/61D3585E/61CC95A1" Ref="#PWR?"  Part="1"
+F 0 "#PWR?" H 6200 3750 50  0001 C CNN
+F 1 "GND" H 6205 3827 50  0000 C CNN
+F 2 "" H 6200 4000 50  0001 C CNN
+F 3 "" H 6200 4000 50  0001 C CNN
+	1    6200 4000
+	1    0    0    -1
+$EndComp
+$Comp
+L power:GND #PWR?
+U 1 1 61CC9DA1
+P 6200 1600
+AR Path="/61CC9DA1" Ref="#PWR?"  Part="1"
+AR Path="/61D3585E/61CC9DA1" Ref="#PWR?"  Part="1"
+F 0 "#PWR?" H 6200 1350 50  0001 C CNN
+F 1 "GND" H 6205 1427 50  0000 C CNN
+F 2 "" H 6200 1600 50  0001 C CNN
+F 3 "" H 6200 1600 50  0001 C CNN
+	1    6200 1600
+	-1   0    0    1
+$EndComp
+$Comp
+L power:GND #PWR?
+U 1 1 61CCA122
+P 6700 1900
+AR Path="/61CCA122" Ref="#PWR?"  Part="1"
+AR Path="/61D3585E/61CCA122" Ref="#PWR?"  Part="1"
+F 0 "#PWR?" H 6700 1650 50  0001 C CNN
+F 1 "GND" H 6705 1727 50  0000 C CNN
+F 2 "" H 6700 1900 50  0001 C CNN
+F 3 "" H 6700 1900 50  0001 C CNN
+	1    6700 1900
+	-1   0    0    1
+$EndComp
+$Comp
+L power:GND #PWR?
+U 1 1 61CCA76D
+P 5100 2400
+AR Path="/61CCA76D" Ref="#PWR?"  Part="1"
+AR Path="/61D3585E/61CCA76D" Ref="#PWR?"  Part="1"
+F 0 "#PWR?" H 5100 2150 50  0001 C CNN
+F 1 "GND" H 5105 2227 50  0000 C CNN
+F 2 "" H 5100 2400 50  0001 C CNN
+F 3 "" H 5100 2400 50  0001 C CNN
+	1    5100 2400
+	-1   0    0    1
+$EndComp
 $EndSCHEMATC

Commit message: Updated component footprints, moved to RDT_Custom_Footprints library
Parts:
- C8: footprint Capacitor_SMD:C_0603_1608Metric -> Capacitor_SMD:C_0603_1608Metric_Pad1.08x0.95mm_HandSolder
- J12: footprint SamacSys_Parts:L717SDC37P1ACH4F -> RDT_Custom_Footprints:L717SDC37P1ACH4F
Changed lines of the file:
@@
 $Descr A4 11693 8268
 encoding utf-8
-Sheet 4 7
+Sheet 7 7
 Title ""
 Date "2021-12-20"
@@
 F 0 "C8" H 5292 2446 50  0000 L CNN
 F 1 "100nF" H 5292 2355 50  0000 L CNN
-F 2 "Capacitor_SMD:C_0603_1608Metric" H 5200 2400 50  0001 C CNN
+F 2 "Capacitor_SMD:C_0603_1608Metric_Pad1.08x0.95mm_HandSolder" H 5200 2400 50  0001 C CNN
 F 3 "~" H 5200 2400 50  0001 C CNN
 	1    5200 2400
@@
 F 0 "J12" V 6019 1600 50  0000 C CNN
 F 1 "L717SDC37P1ACH4F" V 6110 1600 50  0000 C CNN
-F 2 "SamacSys_Parts:L717SDC37P1ACH4F" H 8450 1900 50  0001 L CNN
+F 2 "RDT_Custom_Footprints:L717SDC37P1ACH4F" H 8450 1900 50  0001 L CNN
 F 3 "https://cdn.amphenol-icc.com/media/wysiwyg/files/drawing/l717sdxxxp1ach4f.pdf" H 8450 1800 50  0001 L CNN
 F 4 "D-Sub Standard Connectors 37P Sz C Std Density Pin Screwlock 4-40" H 8450 1700 50  0001 L CNN "Description"
@@
 P 6850 3700
 AR Path="/61CC9506" Ref="#PWR?"  Part="1"
-AR Path="/61D3585E/61CC9506" Ref="#PWR?"  Part="1"
-F 0 "#PWR?" H 6850 3450 50  0001 C CNN
+AR Path="/61D3585E/61CC9506" Ref="#PWR0114"  Part="1"
+F 0 "#PWR0114" H 6850 3450 50  0001 C CNN
 F 1 "GND" H 6855 3527 50  0000 C CNN
 F 2 "" H 6850 3700 50  0001 C CNN
@@
 P 6200 4000
 AR Path="/61CC95A1" Ref="#PWR?"  Part="1"
-AR Path="/61D3585E/61CC95A1" Ref="#PWR?"  Part="1"
-F 0 "#PWR?" H 6200 3750 50  0001 C CNN
+AR Path="/61D3585E/61CC95A1" Ref="#PWR0115"  Part="1"
+F 0 "#PWR0115" H 6200 3750 50  0001 C CNN
 F 1 "GND" H 6205 3827 50  0000 C CNN
 F 2 "" H 6200 4000 50  0001 C CNN
@@
 P 6200 1600
 AR Path="/61CC9DA1" Ref="#PWR?"  Part="1"
-AR Path="/61D3585E/61CC9DA1" Ref="#PWR?"  Part="1"
-F 0 "#PWR?" H 6200 1350 50  0001 C CNN
+AR Path="/61D3585E/61CC9DA1" Ref="#PWR0116"  Part="1"
+F 0 "#PWR0116" H 6200 1350 50  0001 C CNN
 F 1 "GND" H 6205 1427 50  0000 C CNN
 F 2 "" H 6200 1600 50  0001 C CNN
@@
 P 6700 1900
 AR Path="/61CCA122" Ref="#PWR?"  Part="1"
-AR Path="/61D3585E/61CCA122" Ref="#PWR?"  Part="1"
-F 0 "#PWR?" H 6700 1650 50  0001 C CNN
+AR Path="/61D3585E/61CCA122" Ref="#PWR0117"  Part="1"
+F 0 "#PWR0117" H 6700 1650 50  0001 C CNN
 F 1 "GND" H 6705 1727 50  0000 C CNN
 F 2 "" H 6700 1900 50  0001 C CNN
@@
 P 5100 2400
 AR Path="/61CCA76D" Ref="#PWR?"  Part="1"
-AR Path="/61D3585E/61CCA76D" Ref="#PWR?"  Part="1"
-F 0 "#PWR?" H 5100 2150 50  0001 C CNN
+AR Path="/61D3585E/61CCA76D" Ref="#PWR0118"  Part="1"
+F 0 "#PWR0118" H 5100 2150 50  0001 C CNN
 F 1 "GND" H 5105 2227 50  0000 C CNN
 F 2 "" H 5100 2400 50  0001 C CNN

Commit message: Reset annotations, changed SPST switch footprint
Parts:
- renumbered C8 to C36, J12 to J8
Changed lines of the file:
@@
 AR Path="/61A55586" Ref="C?"  Part="1"
 AR Path="/61A437B5/61A55586" Ref="C?"  Part="1"
-AR Path="/61D3585E/61A55586" Ref="C8"  Part="1"
-F 0 "C8" H 5292 2446 50  0000 L CNN
+AR Path="/61D3585E/61A55586" Ref="C36"  Part="1"
+F 0 "C36" H 5292 2446 50  0000 L CNN
 F 1 "100nF" H 5292 2355 50  0000 L CNN
 F 2 "Capacitor_SMD:C_0603_1608Metric_Pad1.08x0.95mm_HandSolder" H 5200 2400 50  0001 C CNN
@@
 	5300 2400 5700 2400
 $Comp
-L power:+3.3V #PWR015
+L power:+3.3V #PWR044
 U 1 1 61A4A3FB
 P 6700 2000
-F 0 "#PWR015" H 6700 1850 50  0001 C CNN
+F 0 "#PWR044" H 6700 1850 50  0001 C CNN
 F 1 "+3.3V" V 6715 2128 50  0000 L CNN
 F 2 "" H 6700 2000 50  0001 C CNN
@@
 $EndComp
 $Comp
-L power:+5V #PWR013
+L power:+5V #PWR039
 U 1 1 61A491E6
 P 5700 1900
-F 0 "#PWR013" H 5700 1750 50  0001 C CNN
+F 0 "#PWR039" H 5700 1750 50  0001 C CNN
 F 1 "+5V" V 5715 2028 50  0000 L CNN
 F 2 "" H 5700 1900 50  0001 C CNN
@@
 $EndComp
 $Comp
-L power:+3.3V #PWR016
+L power:+3.3V #PWR045
 U 1 1 61A4AB5D
 P 6700 3600
-F 0 "#PWR016" H 6700 3450 50  0001 C CNN
+F 0 "#PWR045" H 6700 3450 50  0001 C CNN
 F 1 "+3.3V" V 6715 3728 50  0000 L CNN
 F 2 "" H 6700 3600 50  0001 C CNN
@@
 $EndComp
 $Comp
-L Power_KiCAD_Project-rescue:L717SDC37P1ACH4F-SamacSys_Parts J12
+L Power_KiCAD_Project-rescue:L717SDC37P1ACH4F-SamacSys_Parts J8
 U 1 1 61D5E9EE
 P 6200 1600
-F 0 "J12" V 6019 1600 50  0000 C CNN
+F 0 "J8" V 6019 1600 50  0000 C CNN
 F 1 "L717SDC37P1ACH4F" V 6110 1600 50  0000 C CNN
 F 2 "RDT_Custom_Footprints:L717SDC37P1ACH4F" H 8450 1900 50  0001 L CNN
@@
 	6850 3700 6700 3700
 $Comp
-L power:+5V #PWR014
+L power:+5V #PWR040
 U 1 1 61A49AB4
 P 5700 3600
-F 0 "#PWR014" H 5700 3450 50  0001 C CNN
+F 0 "#PWR040" H 5700 3450 50  0001 C CNN
 F 1 "+5V" V 5715 3728 50  0000 L CNN
 F 2 "" H 5700 3600 50  0001 C CNN
@@
 P 6850 3700
 AR Path="/61CC9506" Ref="#PWR?"  Part="1"
-AR Path="/61D3585E/61CC9506" Ref="#PWR0114"  Part="1"
-F 0 "#PWR0114" H 6850 3450 50  0001 C CNN
+AR Path="/61D3585E/61CC9506" Ref="#PWR046"  Part="1"
+F 0 "#PWR046" H 6850 3450 50  0001 C CNN
 F 1 "GND" H 6855 3527 50  0000 C CNN
 F 2 "" H 6850 3700 50  0001 C CNN
@@
 P 6200 4000
 AR Path="/61CC95A1" Ref="#PWR?"  Part="1"
-AR Path="/61D3585E/61CC95A1" Ref="#PWR0115"  Part="1"
-F 0 "#PWR0115" H 6200 3750 50  0001 C CNN
+AR Path="/61D3585E/61CC95A1" Ref="#PWR042"  Part="1"
+F 0 "#PWR042" H 6200 3750 50  0001 C CNN
 F 1 "GND" H 6205 3827 50  0000 C CNN
 F 2 "" H 6200 4000 50  0001 C CNN
@@
 P 6200 1600
 AR Path="/61CC9DA1" Ref="#PWR?"  Part="1"
-AR Path="/61D3585E/61CC9DA1" Ref="#PWR0116"  Part="1"
-F 0 "#PWR0116" H 6200 1350 50  0001 C CNN
+AR Path="/61D3585E/61CC9DA1" Ref="#PWR041"  Part="1"
+F 0 "#PWR041" H 6200 1350 50  0001 C CNN
 F 1 "GND" H 6205 1427 50  0000 C CNN
 F 2 "" H 6200 1600 50  0001 C CNN
@@
 P 6700 1900
 AR Path="/61CCA122" Ref="#PWR?"  Part="1"
-AR Path="/61D3585E/61CCA122" Ref="#PWR0117"  Part="1"
-F 0 "#PWR0117" H 6700 1650 50  0001 C CNN
+AR Path="/61D3585E/61CCA122" Ref="#PWR043"  Part="1"
+F 0 "#PWR043" H 6700 1650 50  0001 C CNN
 F 1 "GND" H 6705 1727 50  0000 C CNN
 F 2 "" H 6700 1900 50  0001 C CNN
@@
 P 5100 2400
 AR Path="/61CCA76D" Ref="#PWR?"  Part="1"
-AR Path="/61D3585E/61CCA76D" Ref="#PWR0118"  Part="1"
-F 0 "#PWR0118" H 5100 2150 50  0001 C CNN
+AR Path="/61D3585E/61CCA76D" Ref="#PWR038"  Part="1"
+F 0 "#PWR038" H 5100 2150 50  0001 C CNN
 F 1 "GND" H 5105 2227 50  0000 C CNN
 F 2 "" H 5100 2400 50  0001 C CNN

Commit message: Routed 3v3 and 5v buck converters
Switched to working on my laptop so some of the component references might be messed up for a bit
Parts:
- J8: symbol Power_KiCAD_Project-rescue:L717SDC37P1ACH4F-SamacSys_Parts -> Power_KiCAD_Project-rescue:L717SDC37P1ACH4F-SamacSys_Parts-Power_KiCAD_Project-rescue
Changed lines of the file:
@@
 $EndComp
 $Comp
-L Power_KiCAD_Project-rescue:L717SDC37P1ACH4F-SamacSys_Parts J8
+L Power_KiCAD_Project-rescue:L717SDC37P1ACH4F-SamacSys_Parts-Power_KiCAD_Project-rescue J8
 U 1 1 61D5E9EE
 P 6200 1600
+AR Path="/61D5E9EE" Ref="J8"  Part="1"
+AR Path="/61D3585E/61D5E9EE" Ref="J8"  Part="1"
 F 0 "J8" V 5900 1600 50  0000 C CNN
 F 1 "L717SDC37P1ACH4F" V 6110 1600 50  0000 C CNN

Commit message: Moved external switch connector to pack+, added missing no connection flags
This change renders the current PCB layout defunct, next commits will be redesigns of the layout.
Connections:
- wire segments 2 -> 4
- no-connect marks 0 -> 20
Other:
- moved on the sheet: C36
Changed lines of the file:
@@
 Text HLabel 5700 2200 0    50   Input ~ 0
 SWCLK
-Text HLabel 5700 2400 0    50   Input ~ 0
+Text HLabel 4950 2400 0    50   Input ~ 0
 NRST
 Text HLabel 6700 2500 2    50   Input ~ 0
@@
 L Device:C_Small C?
 U 1 1 61A55586
-P 5200 2400
+P 5000 2700
 AR Path="/61A55586" Ref="C?"  Part="1"
 AR Path="/61A437B5/61A55586" Ref="C?"  Part="1"
 AR Path="/61D3585E/61A55586" Ref="C36"  Part="1"
-F 0 "C36" H 5292 2446 50  0000 L CNN
-F 1 "100nF" H 5292 2355 50  0000 L CNN
-F 2 "Capacitor_SMD:C_0603_1608Metric_Pad1.08x0.95mm_HandSolder" H 5200 2400 50  0001 C CNN
-F 3 "~" H 5200 2400 50  0001 C CNN
-	1    5200 2400
-	0    1    -1   0
+F 0 "C36" H 5092 2746 50  0000 L CNN
+F 1 "100nF" H 5092 2655 50  0000 L CNN
+F 2 "Capacitor_SMD:C_0603_1608Metric_Pad1.08x0.95mm_HandSolder" H 5000 2700 50  0001 C CNN
+F 3 "~" H 5000 2700 50  0001 C CNN
+	1    5000 2700
+	1    0    0    1
 $EndComp
-Wire Wire Line
-	5300 2400 5700 2400
 $Comp
 L power:+3.3V #PWR044
@@
 L power:GND #PWR?
 U 1 1 61CCA76D
-P 5100 2400
+P 5000 2800
 AR Path="/61CCA76D" Ref="#PWR?"  Part="1"
 AR Path="/61D3585E/61CCA76D" Ref="#PWR038"  Part="1"
-F 0 "#PWR038" H 5100 2150 50  0001 C CNN
-F 1 "GND" H 5105 2227 50  0000 C CNN
-F 2 "" H 5100 2400 50  0001 C CNN
-F 3 "" H 5100 2400 50  0001 C CNN
-	1    5100 2400
-	-1   0    0    1
+F 0 "#PWR038" H 5000 2550 50  0001 C CNN
+F 1 "GND" H 5005 2627 50  0000 C CNN
+F 2 "" H 5000 2800 50  0001 C CNN
+F 3 "" H 5000 2800 50  0001 C CNN
+	1    5000 2800
+	1    0    0    -1
 $EndComp
+NoConn ~ 5700 2600
+NoConn ~ 5700 2700
+NoConn ~ 5700 2800
+NoConn ~ 5700 2900
+NoConn ~ 5700 3000
+NoConn ~ 5700 3100
+NoConn ~ 5700 3200
+NoConn ~ 5700 3300
+NoConn ~ 5700 3400
+NoConn ~ 5700 3500
+NoConn ~ 6700 2600
+NoConn ~ 6700 2700
+NoConn ~ 6700 2800
+NoConn ~ 6700 2900
+NoConn ~ 6700 3000
+NoConn ~ 6700 3100
+NoConn ~ 6700 3200
+NoConn ~ 6700 3300
+NoConn ~ 6700 3400
+NoConn ~ 6700 3500
+Wire Wire Line
+	5000 2600 5000 2400
+Wire Wire Line
+	5000 2400 5700 2400
+Wire Wire Line
+	4950 2400 5000 2400
+Connection ~ 5000 2400
 $EndSCHEMATC
