File: Hardware/COMPONENT_SHEETS/BuckConverters.sch (KiCad schematic (older format))
At the start: 14 parts

Commit message: FIxed board
issues with the board after the merge have been fixed
Parts:
- gave numbers to parts that had none: 14
Connections:
- wire segments 61 -> 62
Changed lines of the file:
@@
 $EndDescr
 $Comp
-L Power_KiCAD_Project-rescue:LM2672M-TO-263-lm2672m-to-263 U?
+L Power_KiCAD_Project-rescue:LM2672M-TO-263-lm2672m-to-263 U4
 U 1 1 61A319C7
 P 4900 5200
-F 0 "U?" H 4900 5667 50  0000 C CNN
+F 0 "U4" H 4900 5667 50  0000 C CNN
 F 1 "LM2678SX-3.3/NOPB" H 4900 5576 50  0000 C CNN
 F 2 "Package_TO_SOT_SMD:TO-263-7_TabPin8" H 4950 4850 50  0001 L CIN
@@
 ground
 $Comp
-L Power_KiCAD_Project-rescue:SBRD10200TR-SBRD10200TR D?
+L Power_KiCAD_Project-rescue:SBRD10200TR-SBRD10200TR D3
 U 1 1 61A8FF3C
 P 6100 3400
-F 0 "D?" H 6276 3441 50  0000 L CNN
+F 0 "D3" H 6276 3441 50  0000 L CNN
 F 1 "SBRD10200TR" H 6276 3350 50  0000 L CNN
 F 2 "SBRD10200TR:DPAK228P1005X240-4N" H 6100 3400 50  0001 L BNN
@@
 $EndComp
 $Comp
-L Power_KiCAD_Project-rescue:SBRD10200TR-SBRD10200TR D?
+L Power_KiCAD_Project-rescue:SBRD10200TR-SBRD10200TR D4
 U 1 1 61A94D59
 P 6200 5600
-F 0 "D?" H 6376 5641 50  0000 L CNN
+F 0 "D4" H 6376 5641 50  0000 L CNN
 F 1 "SBRD10200TR" H 6376 5550 50  0000 L CNN
 F 2 "SBRD10200TR:DPAK228P1005X240-4N" H 6200 5600 50  0001 L BNN
@@
 	6200 3650 7400 3650
 $Comp
-L Power_KiCAD_Project-rescue:CGA4C2C0G1H103J060AA-SamacSys_Parts C?
+L Power_KiCAD_Project-rescue:CGA4C2C0G1H103J060AA-SamacSys_Parts C14
 U 1 1 61BC76DD
 P 5900 5100
-F 0 "C?" V 6104 5228 50  0000 L CNN
+F 0 "C14" V 6104 5228 50  0000 L CNN
 F 1 "CGA4C2C0G1H103J060AA" V 6195 5228 50  0000 L CNN
 F 2 "SamacSys_Parts:CAPC2012X75N" H 6250 5150 50  0001 L CNN
@@
 $EndComp
 $Comp
-L Power_KiCAD_Project-rescue:C0805C104M5RACTU-SamacSys_Parts C?
+L Power_KiCAD_Project-rescue:C0805C104M5RACTU-SamacSys_Parts C12
 U 1 1 61BC89F9
 P 4050 5150
-F 0 "C?" V 4254 5278 50  0000 L CNN
+F 0 "C12" V 4254 5278 50  0000 L CNN
 F 1 "C0805C104M5RACTU" V 4345 5278 50  0000 L CNN
 F 2 "SamacSys_Parts:CAPC2012X88N" H 4400 5200 50  0001 L CNN
@@
 $EndComp
 $Comp
-L Power_KiCAD_Project-rescue:35SVPF82M-35SVPF82M C?
+L Power_KiCAD_Project-rescue:35SVPF82M-35SVPF82M C10
 U 1 1 61BCB4E6
 P 3400 5150
-F 0 "C?" V 3604 5280 50  0000 L CNN
+F 0 "C10" V 3604 5280 50  0000 L CNN
 F 1 "35SVPF82M" V 3695 5280 50  0000 L CNN
 F 2 "SamacSys_Parts:16SVPT560M" H 3750 5200 50  0001 L CNN
@@
 $EndComp
 $Comp
-L Power_KiCAD_Project-rescue:6SVPC330M-6SVPC330M C?
+L Power_KiCAD_Project-rescue:6SVPC330M-6SVPC330M C16
 U 1 1 61BCD9CD
 P 7400 5500
-F 0 "C?" V 7604 5630 50  0000 L CNN
+F 0 "C16" V 7604 5630 50  0000 L CNN
 F 1 "6SVPC330M" V 7695 5630 50  0000 L CNN
 F 2 "SamacSys_Parts:16SVF180M" H 7750 5550 50  0001 L CNN
@@
 $EndComp
 $Comp
-L Power_KiCAD_Project-rescue:35SVPF82M-35SVPF82M C?
+L Power_KiCAD_Project-rescue:35SVPF82M-35SVPF82M C9
 U 1 1 61BCF050
 P 3400 2800
-F 0 "C?" V 3604 2930 50  0000 L CNN
+F 0 "C9" V 3604 2930 50  0000 L CNN
 F 1 "35SVPF82M" V 3695 2930 50  0000 L CNN
 F 2 "SamacSys_Parts:16SVPT560M" H 3750 2850 50  0001 L CNN
@@
 $EndComp
 $Comp
-L Power_KiCAD_Project-rescue:C0805C104M5RACTU-SamacSys_Parts C?
+L Power_KiCAD_Project-rescue:C0805C104M5RACTU-SamacSys_Parts C11
 U 1 1 61BD084E
 P 4050 2800
-F 0 "C?" V 4254 2928 50  0000 L CNN
+F 0 "C11" V 4254 2928 50  0000 L CNN
 F 1 "C0805C104M5RACTU" V 4345 2928 50  0000 L CNN
 F 2 "SamacSys_Parts:CAPC2012X88N" H 4400 2850 50  0001 L CNN
@@
 $EndComp
 $Comp
-L Power_KiCAD_Project-rescue:CGA4C2C0G1H103J060AA-SamacSys_Parts C?
+L Power_KiCAD_Project-rescue:CGA4C2C0G1H103J060AA-SamacSys_Parts C13
 U 1 1 61BD1A0A
 P 5800 2750
-F 0 "C?" V 6004 2878 50  0000 L CNN
+F 0 "C13" V 6004 2878 50  0000 L CNN
 F 1 "CGA4C2C0G1H103J060AA" V 6095 2878 50  0000 L CNN
 F 2 "SamacSys_Parts:CAPC2012X75N" H 6150 2800 50  0001 L CNN
@@
 $EndComp
 $Comp
-L Power_KiCAD_Project-rescue:MSS1210-153MEB-MSS1210-153MEB L?
+L Power_KiCAD_Project-rescue:MSS1210-153MEB-MSS1210-153MEB L2
 U 1 1 61BD4A85
 P 7000 3050
-F 0 "L?" H 7000 3267 50  0000 C CNN
+F 0 "L2" H 7000 3267 50  0000 C CNN
 F 1 "MSS1210-153MEB" H 7000 3176 50  0000 C CNN
 F 2 "MSS1210-153MEB:IND_MSS1210-153MEB" H 7000 3050 50  0001 L BNN
@@
 	5400 5200 5750 5200
 $Comp
-L Power_KiCAD_Project-rescue:LM2672M-TO-263-lm2672m-to-263 U?
+L Power_KiCAD_Project-rescue:LM2672M-TO-263-lm2672m-to-263 U3
 U 1 1 61A7F0DE
 P 4900 2850
-F 0 "U?" H 4900 3317 50  0000 C CNN
+F 0 "U3" H 4900 3317 50  0000 C CNN
 F 1 "LM2678SX-5.0/NOPB" H 4900 3226 50  0000 C CNN
 F 2 "Package_TO_SOT_SMD:TO-263-7_TabPin8" H 4950 2500 50  0001 L CIN
@@
 $EndComp
 $Comp
-L Power_KiCAD_Project-rescue:16SVP330M-16SVP330M C?
+L Power_KiCAD_Project-rescue:16SVP330M-16SVP330M C15
 U 1 1 61BD32A5
 P 7400 3150
-F 0 "C?" V 7604 3280 50  0000 L CNN
+F 0 "C15" V 7604 3280 50  0000 L CNN
 F 1 "16SVP330M" V 7695 3280 50  0000 L CNN
 F 2 "SamacSys_Parts:16SVF1000M" H 7750 3200 50  0001 L CNN
@@
 	0    1    1    0
 $EndComp
-$Comp
-L Power_KiCAD_Project-rescue:SRP1270-8R2M-SamacSys_Parts L?
+Wire Wire Line
+	5400 5000 7400 5000
+Wire Wire Line
+	6000 3610 6000 3650
+Wire Wire Line
+	5950 3650 6000 3650
+Connection ~ 6000 3650
+Wire Wire Line
+	7400 3450 7400 3650
+Wire Wire Line
+	3400 3100 3400 3450
+Wire Wire Line
+	3400 5450 3400 5800
+Wire Wire Line
+	6000 6000 6100 6000
+Connection ~ 6100 6000
+Wire Wire Line
+	6100 6000 6300 6000
+Wire Wire Line
+	6100 5810 6100 6000
+Wire Wire Line
+	7400 5800 7400 6000
+Wire Wire Line
+	5550 3250 5800 3250
+Connection ~ 5800 3250
+Wire Wire Line
+	5800 3250 6100 3250
+Wire Wire Line
+	6100 5400 6200 5400
+$Comp
+L Power_KiCAD_Project-rescue:SRP1270-8R2M-SamacSys_Parts L1
 U 1 1 61D4AE9F
 P 6450 5400
-F 0 "L?" H 6850 5625 50  0000 C CNN
+F 0 "L1" H 6850 5625 50  0000 C CNN
 F 1 "SRP1270-8R2M" H 6850 5534 50  0000 C CNN
 F 2 "SamacSys_Parts:INDPM137129X700N" H 7100 5450 50  0001 L CNN
@@
 $EndComp
 Wire Wire Line
-	5400 5000 7400 5000
-Wire Wire Line
-	5550 3250 6100 3250
-Wire Wire Line
-	5750 5600 6100 5600
-Wire Wire Line
-	7000 5400 7400 5400
-Wire Wire Line
-	6100 5400 6900 5400
-Wire Wire Line
-	6000 3600 6000 3610
-Connection ~ 6000 3610
-Wire Wire Line
-	6000 3610 6000 3650
-Wire Wire Line
-	5950 3650 6000 3650
-Connection ~ 6000 3650
-Wire Wire Line
-	7400 3450 7400 3650
-Wire Wire Line
-	3400 3100 3400 3450
-Wire Wire Line
-	3400 5450 3400 5800
-Wire Wire Line
-	6000 6000 6100 6000
-Wire Wire Line
-	6100 5800 6100 5810
-Connection ~ 6100 6000
-Wire Wire Line
-	6100 6000 6300 6000
-Connection ~ 6100 5810
-Wire Wire Line
-	6100 5810 6100 6000
-Wire Wire Line
-	7400 5800 7400 6000
+	5750 5600 5900 5600
+Wire Wire Line
+	5900 5600 6100 5600
+Connection ~ 5900 5600
+Wire Wire Line
+	6200 5400 6450 5400
+Connection ~ 6200 5400
+Wire Wire Line
+	7400 5400 7250 5400
 $EndSCHEMATC

Commit message: Fixed ground symbols in component sheets, corrected MCU sheet
Connections:
- net labels added: GND
- net labels removed: ground
Changed lines of the file:
@@
 $Descr A4 11693 8268
 encoding utf-8
-Sheet 6 8
+Sheet 5 7
 Title "Buck Converter Supply"
 Date "2021-12-20"
@@
 Text Notes 2950 2150 0    98   ~ 20
 5V Buck Converter
-Text HLabel 4050 3450 3    50   Input ~ 0
-ground
-Text HLabel 5950 3650 0    50   Input ~ 0
-ground
-Text HLabel 6000 6000 0    50   Input ~ 0
-ground
-Text HLabel 4050 5800 3    50   Input ~ 0
-ground
 $Comp
 L Power_KiCAD_Project-rescue:SBRD10200TR-SBRD10200TR D3
@@
 Wire Wire Line
 	7400 5400 7250 5400
+$Comp
+L power:GND #PWR?
+U 1 1 61CCDE7D
+P 4050 3450
+AR Path="/61CCDE7D" Ref="#PWR?"  Part="1"
+AR Path="/61A48488/61CCDE7D" Ref="#PWR?"  Part="1"
+F 0 "#PWR?" H 4050 3200 50  0001 C CNN
+F 1 "GND" H 4055 3277 50  0000 C CNN
+F 2 "" H 4050 3450 50  0001 C CNN
+F 3 "" H 4050 3450 50  0001 C CNN
+	1    4050 3450
+	1    0    0    -1
+$EndComp
+$Comp
+L power:GND #PWR?
+U 1 1 61CCEFCE
+P 5950 3650
+AR Path="/61CCEFCE" Ref="#PWR?"  Part="1"
+AR Path="/61A48488/61CCEFCE" Ref="#PWR?"  Part="1"
+F 0 "#PWR?" H 5950 3400 50  0001 C CNN
+F 1 "GND" H 5955 3477 50  0000 C CNN
+F 2 "" H 5950 3650 50  0001 C CNN
+F 3 "" H 5950 3650 50  0001 C CNN
+	1    5950 3650
+	1    0    0    -1
+$EndComp
+$Comp
+L power:GND #PWR?
+U 1 1 61CD0185
+P 4050 5800
+AR Path="/61CD0185" Ref="#PWR?"  Part="1"
+AR Path="/61A48488/61CD0185" Ref="#PWR?"  Part="1"
+F 0 "#PWR?" H 4050 5550 50  0001 C CNN
+F 1 "GND" H 4055 5627 50  0000 C CNN
+F 2 "" H 4050 5800 50  0001 C CNN
+F 3 "" H 4050 5800 50  0001 C CNN
+	1    4050 5800
+	1    0    0    -1
+$EndComp
+$Comp
+L power:GND #PWR?
+U 1 1 61CD137E
+P 6000 6000
+AR Path="/61CD137E" Ref="#PWR?"  Part="1"
+AR Path="/61A48488/61CD137E" Ref="#PWR?"  Part="1"
+F 0 "#PWR?" H 6000 5750 50  0001 C CNN
+F 1 "GND" H 6005 5827 50  0000 C CNN
+F 2 "" H 6000 6000 50  0001 C CNN
+F 3 "" H 6000 6000 50  0001 C CNN
+	1    6000 6000
+	1    0    0    -1
+$EndComp
 $EndSCHEMATC

Commit message: Updated component footprints, moved to RDT_Custom_Footprints library
Parts:
- C10, C9: footprint SamacSys_Parts:16SVPT560M -> RDT_Custom_Footprints:16SVPT560M
- C11, C12: footprint SamacSys_Parts:CAPC2012X88N -> RDT_Custom_Footprints:CAPC2012X88N
- C13, C14: footprint SamacSys_Parts:CAPC2012X75N -> RDT_Custom_Footprints:CAPC2012X75N
- C15: footprint SamacSys_Parts:16SVF1000M -> RDT_Custom_Footprints:16SVF1000M
- C16: footprint SamacSys_Parts:16SVF180M -> RDT_Custom_Footprints:16SVF180M
- D3, D4: footprint SBRD10200TR:DPAK228P1005X240-4N -> RDT_Custom_Footprints:DPAK228P1005X240-4N
- L1: footprint SamacSys_Parts:INDPM137129X700N -> RDT_Custom_Footprints:INDPM137129X700N
- L2: footprint MSS1210-153MEB:IND_MSS1210-153MEB -> RDT_Custom_Footprints:IND_MSS1210-153MEB
Changed lines of the file:
@@
 $Descr A4 11693 8268
 encoding utf-8
-Sheet 5 7
+Sheet 4 7
 Title "Buck Converter Supply"
 Date "2021-12-20"
@@
 F 0 "D3" H 6276 3441 50  0000 L CNN
 F 1 "SBRD10200TR" H 6276 3350 50  0000 L CNN
-F 2 "SBRD10200TR:DPAK228P1005X240-4N" H 6100 3400 50  0001 L BNN
+F 2 "RDT_Custom_Footprints:DPAK228P1005X240-4N" H 6100 3400 50  0001 L BNN
 F 3 "" H 6100 3400 50  0001 L BNN
 F 4 "SBRD10200TR" H 6100 3400 50  0001 L BNN "MP"
@@
 F 0 "D4" H 6376 5641 50  0000 L CNN
 F 1 "SBRD10200TR" H 6376 5550 50  0000 L CNN
-F 2 "SBRD10200TR:DPAK228P1005X240-4N" H 6200 5600 50  0001 L BNN
+F 2 "RDT_Custom_Footprints:DPAK228P1005X240-4N" H 6200 5600 50  0001 L BNN
 F 3 "" H 6200 5600 50  0001 L BNN
 F 4 "SBRD10200TR" H 6200 5600 50  0001 L BNN "MP"
@@
 F 0 "C14" V 6104 5228 50  0000 L CNN
 F 1 "CGA4C2C0G1H103J060AA" V 6195 5228 50  0000 L CNN
-F 2 "SamacSys_Parts:CAPC2012X75N" H 6250 5150 50  0001 L CNN
+F 2 "RDT_Custom_Footprints:CAPC2012X75N" H 6250 5150 50  0001 L CNN
 F 3 "https://datasheet.datasheetarchive.com/originals/distributors/Datasheets-DGA20/25667.pdf" H 6250 5050 50  0001 L CNN
 F 4 "TDK 2012 CGA 10nF Ceramic Multilayer Capacitor, 50 V dc, +125C, C0G Dielectric, +/-5%" H 6250 4950 50  0001 L CNN "Description"
@@
 F 0 "C12" V 4254 5278 50  0000 L CNN
 F 1 "C0805C104M5RACTU" V 4345 5278 50  0000 L CNN
-F 2 "SamacSys_Parts:CAPC2012X88N" H 4400 5200 50  0001 L CNN
+F 2 "RDT_Custom_Footprints:CAPC2012X88N" H 4400 5200 50  0001 L CNN
 F 3 "https://datasheet.datasheetarchive.com/originals/distributors/Datasheets-DGA10/2409909.pdf" H 4400 5100 50  0001 L CNN
 F 4 "Multilayer Ceramic Chip Capacitors" H 4400 5000 50  0001 L CNN "Description"
@@
 F 0 "C10" V 3604 5280 50  0000 L CNN
 F 1 "35SVPF82M" V 3695 5280 50  0000 L CNN
-F 2 "SamacSys_Parts:16SVPT560M" H 3750 5200 50  0001 L CNN
+F 2 "RDT_Custom_Footprints:16SVPT560M" H 3750 5200 50  0001 L CNN
 F 3 "http://industrial.panasonic.com/cdbs/www-data/pdf/AAB8000/AAB8000C177.pdf" H 3750 5100 50  0001 L CNN
 F 4 "Panasonic 82uF 35 V dc Polymer Aluminium Electrolytic Capacitor E12, OS-CON Series 5000h 8 x 11.9mm" H 3750 5000 50  0001 L CNN "Description"
@@
 F 0 "C16" V 7604 5630 50  0000 L CNN
 F 1 "6SVPC330M" V 7695 5630 50  0000 L CNN
-F 2 "SamacSys_Parts:16SVF180M" H 7750 5550 50  0001 L CNN
+F 2 "RDT_Custom_Footprints:16SVF180M" H 7750 5550 50  0001 L CNN
 F 3 "http://industrial.panasonic.com/cdbs/www-data/pdf/AAB8000/AAB8000C256.pdf" H 7750 5450 50  0001 L CNN
 F 4 "Panasonic 330uF Polymer Capacitor 6.3V dc, Surface Mount - 6SVPC330M" H 7750 5350 50  0001 L CNN "Description"
@@
 F 0 "C9" V 3604 2930 50  0000 L CNN
 F 1 "35SVPF82M" V 3695 2930 50  0000 L CNN
-F 2 "SamacSys_Parts:16SVPT560M" H 3750 2850 50  0001 L CNN
+F 2 "RDT_Custom_Footprints:16SVPT560M" H 3750 2850 50  0001 L CNN
 F 3 "http://industrial.panasonic.com/cdbs/www-data/pdf/AAB8000/AAB8000C177.pdf" H 3750 2750 50  0001 L CNN
 F 4 "Panasonic 82uF 35 V dc Polymer Aluminium Electrolytic Capacitor E12, OS-CON Series 5000h 8 x 11.9mm" H 3750 2650 50  0001 L CNN "Description"
@@
 F 0 "C11" V 4254 2928 50  0000 L CNN
 F 1 "C0805C104M5RACTU" V 4345 2928 50  0000 L CNN
-F 2 "SamacSys_Parts:CAPC2012X88N" H 4400 2850 50  0001 L CNN
+F 2 "RDT_Custom_Footprints:CAPC2012X88N" H 4400 2850 50  0001 L CNN
 F 3 "https://datasheet.datasheetarchive.com/originals/distributors/Datasheets-DGA10/2409909.pdf" H 4400 2750 50  0001 L CNN
 F 4 "Multilayer Ceramic Chip Capacitors" H 4400 2650 50  0001 L CNN "Description"
@@
 F 0 "C13" V 6004 2878 50  0000 L CNN
 F 1 "CGA4C2C0G1H103J060AA" V 6095 2878 50  0000 L CNN
-F 2 "SamacSys_Parts:CAPC2012X75N" H 6150 2800 50  0001 L CNN
+F 2 "RDT_Custom_Footprints:CAPC2012X75N" H 6150 2800 50  0001 L CNN
 F 3 "https://datasheet.datasheetarchive.com/originals/distributors/Datasheets-DGA20/25667.pdf" H 6150 2700 50  0001 L CNN
 F 4 "TDK 2012 CGA 10nF Ceramic Multilayer Capacitor, 50 V dc, +125C, C0G Dielectric, +/-5%" H 6150 2600 50  0001 L CNN "Description"
@@
 F 0 "L2" H 7000 3267 50  0000 C CNN
 F 1 "MSS1210-153MEB" H 7000 3176 50  0000 C CNN
-F 2 "MSS1210-153MEB:IND_MSS1210-153MEB" H 7000 3050 50  0001 L BNN
+F 2 "RDT_Custom_Footprints:IND_MSS1210-153MEB" H 7000 3050 50  0001 L BNN
 F 3 "" H 7000 3050 50  0001 L BNN
 F 4 "In Stock" H 7000 3050 50  0001 L BNN "Availability"
@@
 F 0 "C15" V 7604 3280 50  0000 L CNN
 F 1 "16SVP330M" V 7695 3280 50  0000 L CNN
-F 2 "SamacSys_Parts:16SVF1000M" H 7750 3200 50  0001 L CNN
+F 2 "RDT_Custom_Footprints:16SVF1000M" H 7750 3200 50  0001 L CNN
 F 3 "http://industrial.panasonic.com/cdbs/www-data/pdf/AAB8000/AAB8000C193.pdf" H 7750 3100 50  0001 L CNN
 F 4 "Capacitor SMD SVP series 16V 330uF Panasonic 330uF 16 V Polymer Aluminium Electrolytic Capacitor F12, OS-CON Series 2000h 10 x 12.6mm" H 7750 3000 50  0001 L CNN "Description"
@@
 F 0 "L1" H 6850 5625 50  0000 C CNN
 F 1 "SRP1270-8R2M" H 6850 5534 50  0000 C CNN
-F 2 "SamacSys_Parts:INDPM137129X700N" H 7100 5450 50  0001 L CNN
+F 2 "RDT_Custom_Footprints:INDPM137129X700N" H 7100 5450 50  0001 L CNN
 F 3 "https://datasheet.datasheetarchive.com/originals/distributors/SFDatasheet-7/sf-000140448.pdf" H 7100 5350 50  0001 L CNN
 F 4 "Bourns, SRP1270, 1270 Shielded Wire-wound SMD Inductor with a Iron Core, 8.2 uH +/-20% Wire-Wound 17A Idc" H 7100 5250 50  0001 L CNN "Description"
@@
 P 4050 3450
 AR Path="/61CCDE7D" Ref="#PWR?"  Part="1"
-AR Path="/61A48488/61CCDE7D" Ref="#PWR?"  Part="1"
-F 0 "#PWR?" H 4050 3200 50  0001 C CNN
+AR Path="/61A48488/61CCDE7D" Ref="#PWR0106"  Part="1"
+F 0 "#PWR0106" H 4050 3200 50  0001 C CNN
 F 1 "GND" H 4055 3277 50  0000 C CNN
 F 2 "" H 4050 3450 50  0001 C CNN
@@
 P 5950 3650
 AR Path="/61CCEFCE" Ref="#PWR?"  Part="1"
-AR Path="/61A48488/61CCEFCE" Ref="#PWR?"  Part="1"
-F 0 "#PWR?" H 5950 3400 50  0001 C CNN
+AR Path="/61A48488/61CCEFCE" Ref="#PWR0107"  Part="1"
+F 0 "#PWR0107" H 5950 3400 50  0001 C CNN
 F 1 "GND" H 5955 3477 50  0000 C CNN
 F 2 "" H 5950 3650 50  0001 C CNN
@@
 P 4050 5800
 AR Path="/61CD0185" Ref="#PWR?"  Part="1"
-AR Path="/61A48488/61CD0185" Ref="#PWR?"  Part="1"
-F 0 "#PWR?" H 4050 5550 50  0001 C CNN
+AR Path="/61A48488/61CD0185" Ref="#PWR0108"  Part="1"
+F 0 "#PWR0108" H 4050 5550 50  0001 C CNN
 F 1 "GND" H 4055 5627 50  0000 C CNN
 F 2 "" H 4050 5800 50  0001 C CNN
@@
 P 6000 6000
 AR Path="/61CD137E" Ref="#PWR?"  Part="1"
-AR Path="/61A48488/61CD137E" Ref="#PWR?"  Part="1"
-F 0 "#PWR?" H 6000 5750 50  0001 C CNN
+AR Path="/61A48488/61CD137E" Ref="#PWR0109"  Part="1"
+F 0 "#PWR0109" H 6000 5750 50  0001 C CNN
 F 1 "GND" H 6005 5827 50  0000 C CNN
 F 2 "" H 6000 6000 50  0001 C CNN

Commit message: Updated Buck Converter component sheet
Parts:
- removed C10, C9: 35SVPF82M, RDT_Custom_Footprints:16SVPT560M, symbol Power_KiCAD_Project-rescue:35SVPF82M-35SVPF82M
- removed C11, C12: C0805C104M5RACTU, RDT_Custom_Footprints:CAPC2012X88N, symbol Power_KiCAD_Project-rescue:C0805C104M5RACTU-SamacSys_Parts
- removed C13, C14: CGA4C2C0G1H103J060AA, RDT_Custom_Footprints:CAPC2012X75N, symbol Power_KiCAD_Project-rescue:CGA4C2C0G1H103J060AA-SamacSys_Parts
- removed C15: 16SVP330M, RDT_Custom_Footprints:16SVF1000M, symbol Power_KiCAD_Project-rescue:16SVP330M-16SVP330M
- removed L1: SRP1270-8R2M, RDT_Custom_Footprints:INDPM137129X700N, symbol Power_KiCAD_Project-rescue:SRP1270-8R2M-SamacSys_Parts
- removed L2: MSS1210-153MEB, RDT_Custom_Footprints:IND_MSS1210-153MEB, symbol Power_KiCAD_Project-rescue:MSS1210-153MEB-MSS1210-153MEB
- added C10, C9: 35SVPF82M, RDT_Custom_Footprints:16SVPT560M, symbol Device:CP
- added C11, C12: C0805C104M5RACTU, RDT_Custom_Footprints:CAPC2012X88N, symbol Device:C
- added C14, C?: CGA4C2C0G1H103J060AA, RDT_Custom_Footprints:CAPC2012X75N, symbol Device:C
- added C?: 16SVP330M, RDT_Custom_Footprints:16SVF1000M, symbol Device:CP
- added L1: SRP1270-8R2M, RDT_Custom_Footprints:INDPM137129X700N, symbol Device:L
- added L2: MSS1210-153MEB, RDT_Custom_Footprints:IND_MSS1210-153MEB, symbol Device:L
Connections:
- wire segments 62 -> 67

Commit message: Reset annotations, changed SPST switch footprint
Parts:
- gave numbers to parts that had none: 2
- renumbered C9 to C3, C10 to C4, C11 to C5, C12 to C6, C14 to C8, C16 to C9, D3 to D1, D4 to D2, L2 to L1, L1 to L2
Changed lines of the file:
@@
 5V Buck Converter
 $Comp
-L Power_KiCAD_Project-rescue:SBRD10200TR-SBRD10200TR D3
+L Power_KiCAD_Project-rescue:SBRD10200TR-SBRD10200TR D1
 U 1 1 61A8FF3C
 P 6400 3400
-F 0 "D3" H 6576 3441 50  0000 L CNN
+F 0 "D1" H 6576 3441 50  0000 L CNN
 F 1 "SBRD10200TR" H 6576 3350 50  0000 L CNN
 F 2 "RDT_Custom_Footprints:DPAK228P1005X240-4N" H 6400 3400 50  0001 L BNN
@@
 $EndComp
 $Comp
-L Power_KiCAD_Project-rescue:SBRD10200TR-SBRD10200TR D4
+L Power_KiCAD_Project-rescue:SBRD10200TR-SBRD10200TR D2
 U 1 1 61A94D59
 P 6400 5600
-F 0 "D4" H 6576 5641 50  0000 L CNN
+F 0 "D2" H 6576 5641 50  0000 L CNN
 F 1 "SBRD10200TR" H 6576 5550 50  0000 L CNN
 F 2 "RDT_Custom_Footprints:DPAK228P1005X240-4N" H 6400 5600 50  0001 L BNN
@@
 	6500 3650 7700 3650
 $Comp
-L Power_KiCAD_Project-rescue:6SVPC330M-6SVPC330M C16
+L Power_KiCAD_Project-rescue:6SVPC330M-6SVPC330M C9
 U 1 1 61BCD9CD
 P 7600 5500
-F 0 "C16" V 7804 5630 50  0000 L CNN
+F 0 "C9" V 7804 5630 50  0000 L CNN
 F 1 "6SVPC330M" V 7895 5630 50  0000 L CNN
 F 2 "RDT_Custom_Footprints:16SVF180M" H 7950 5550 50  0001 L CNN
@@
 P 3400 3450
 AR Path="/61CCDE7D" Ref="#PWR?"  Part="1"
-AR Path="/61A48488/61CCDE7D" Ref="#PWR0106"  Part="1"
-F 0 "#PWR0106" H 3400 3200 50  0001 C CNN
+AR Path="/61A48488/61CCDE7D" Ref="#PWR013"  Part="1"
+F 0 "#PWR013" H 3400 3200 50  0001 C CNN
 F 1 "GND" H 3405 3277 50  0000 C CNN
 F 2 "" H 3400 3450 50  0001 C CNN
@@
 P 6250 3650
 AR Path="/61CCEFCE" Ref="#PWR?"  Part="1"
-AR Path="/61A48488/61CCEFCE" Ref="#PWR0107"  Part="1"
-F 0 "#PWR0107" H 6250 3400 50  0001 C CNN
+AR Path="/61A48488/61CCEFCE" Ref="#PWR016"  Part="1"
+F 0 "#PWR016" H 6250 3400 50  0001 C CNN
 F 1 "GND" H 6255 3477 50  0000 C CNN
 F 2 "" H 6250 3650 50  0001 C CNN
@@
 P 3400 5800
 AR Path="/61CD0185" Ref="#PWR?"  Part="1"
-AR Path="/61A48488/61CD0185" Ref="#PWR0108"  Part="1"
-F 0 "#PWR0108" H 3400 5550 50  0001 C CNN
+AR Path="/61A48488/61CD0185" Ref="#PWR014"  Part="1"
+F 0 "#PWR014" H 3400 5550 50  0001 C CNN
 F 1 "GND" H 3405 5627 50  0000 C CNN
 F 2 "" H 3400 5800 50  0001 C CNN
@@
 P 6200 6000
 AR Path="/61CD137E" Ref="#PWR?"  Part="1"
-AR Path="/61A48488/61CD137E" Ref="#PWR0109"  Part="1"
-F 0 "#PWR0109" H 6200 5750 50  0001 C CNN
+AR Path="/61A48488/61CD137E" Ref="#PWR015"  Part="1"
+F 0 "#PWR015" H 6200 5750 50  0001 C CNN
 F 1 "GND" H 6205 5827 50  0000 C CNN
 F 2 "" H 6200 6000 50  0001 C CNN
@@
 $EndComp
 $Comp
-L Device:CP C9
+L Device:CP C3
 U 1 1 61C4FD95
 P 2750 3000
-F 0 "C9" H 2868 3046 50  0000 L CNN
+F 0 "C3" H 2868 3046 50  0000 L CNN
 F 1 "35SVPF82M" H 2868 2955 50  0000 L CNN
 F 2 "RDT_Custom_Footprints:16SVPT560M" H 3100 3050 50  0001 L CNN
@@
 $EndComp
 $Comp
-L Device:C C11
+L Device:C C5
 U 1 1 61C536F2
 P 3400 3000
-F 0 "C11" H 3515 3046 50  0000 L CNN
+F 0 "C5" H 3515 3046 50  0000 L CNN
 F 1 "C0805C104M5RACTU" H 3515 2955 50  0000 L CNN
 F 2 "RDT_Custom_Footprints:CAPC2012X88N" H 3750 3050 50  0001 L CNN
@@
 	5550 3250 5800 3250
 $Comp
-L Device:C C?
+L Device:C C7
 U 1 1 61C620DC
 P 5800 2950
-F 0 "C?" H 5915 2996 50  0000 L CNN
+F 0 "C7" H 5915 2996 50  0000 L CNN
 F 1 "CGA4C2C0G1H103J060AA" H 5915 2905 50  0000 L CNN
 F 2 "RDT_Custom_Footprints:CAPC2012X75N" H 6150 3000 50  0001 L CNN
@@
 	5800 3250 6400 3250
 $Comp
-L Device:L L2
+L Device:L L1
 U 1 1 61C65BE9
 P 7300 3050
-F 0 "L2" V 7490 3050 50  0000 C CNN
+F 0 "L1" V 7490 3050 50  0000 C CNN
 F 1 "MSS1210-153MEB" V 7400 3050 50  0000 C CNN
 F 2 "RDT_Custom_Footprints:IND_MSS1210-153MEB" H 7300 3050 50  0001 L BNN
@@
 	7450 3050 7700 3050
 $Comp
-L Device:CP C?
+L Device:CP C10
 U 1 1 61C6A85B
 P 7700 3300
-F 0 "C?" H 7818 3346 50  0000 L CNN
+F 0 "C10" H 7818 3346 50  0000 L CNN
 F 1 "16SVP330M" H 7818 3255 50  0000 L CNN
 F 2 "RDT_Custom_Footprints:16SVF1000M" H 8050 3350 50  0001 L CNN
@@
 $EndComp
 $Comp
-L Device:CP C10
+L Device:CP C4
 U 1 1 61C6E1A8
 P 2750 5400
-F 0 "C10" H 2868 5446 50  0000 L CNN
+F 0 "C4" H 2868 5446 50  0000 L CNN
 F 1 "35SVPF82M" H 2868 5355 50  0000 L CNN
 F 2 "RDT_Custom_Footprints:16SVPT560M" H 3100 5450 50  0001 L CNN
@@
 $EndComp
 $Comp
-L Device:C C12
+L Device:C C6
 U 1 1 61C6FB03
 P 3400 5400
-F 0 "C12" H 3515 5446 50  0000 L CNN
+F 0 "C6" H 3515 5446 50  0000 L CNN
 F 1 "C0805C104M5RACTU" H 3515 5355 50  0000 L CNN
 F 2 "RDT_Custom_Footprints:CAPC2012X88N" H 3750 5450 50  0001 L CNN
@@
 	2750 5550 2750 5800
 $Comp
-L Device:C C14
+L Device:C C8
 U 1 1 61C7B39E
 P 5900 5300
-F 0 "C14" H 6015 5346 50  0000 L CNN
+F 0 "C8" H 6015 5346 50  0000 L CNN
 F 1 "CGA4C2C0G1H103J060AA" H 6015 5255 50  0000 L CNN
 F 2 "RDT_Custom_Footprints:CAPC2012X75N" H 6250 5350 50  0001 L CNN
@@
 	5400 5000 7600 5000
 $Comp
-L Device:L L1
+L Device:L L2
 U 1 1 61C836B3
 P 7300 5400
-F 0 "L1" H 7700 5625 50  0000 C CNN
+F 0 "L2" H 7700 5625 50  0000 C CNN
 F 1 "SRP1270-8R2M" H 7700 5534 50  0000 C CNN
 F 2 "RDT_Custom_Footprints:INDPM137129X700N" H 7950 5450 50  0001 L CNN
