File: Hardware/COMPONENT_SHEETS/MCU_L562VE.sch (KiCad schematic (older format))
At the start: 16 parts, among them U6 STM32L562VET, Y2 32MHz

Commit message: Fixed ground symbols in component sheets, corrected MCU sheet
Parts:
- added D?: RED, LED_SMD:LED_0603_1608Metric, symbol Device:LED
- added D?: GREEN, LED_SMD:LED_0603_1608Metric, symbol Device:LED
- added R? (x2): 1k5Ω, Resistor_SMD:R_0603_1608Metric, symbol Device:R
Connections:
- net labels added: EXT_INT1, EXT_INT2, EXT_INT3, I2C2_SCL, I2C2_SDA
- net labels removed: GNDREF, SPI1_MISO, SPI1_MOSI, SPI1_SCK, SPI2_EXT_INT, SPI2_MISO, SPI2_MOSI, SPI2_RST, SPI2_SCK, SPI3_EXT_INT, SPI3_MISO, SPI3_MOSI, SPI3_RST, SPI3_SCK, USB_DM, USB_DP, ~SPI1_NSS, ~SPI2_NSS, ~SPI3_NSS
- wire segments 81 -> 87
- no-connect marks 58 -> 69
Changed lines of the file:
@@
 $Descr A4 11693 8268
 encoding utf-8
-Sheet 8 8
+Sheet 7 7
 Title ""
 Date "2021-12-20"
@@
 Wire Notes Line
 	6450 1050 11050 1050
-Text HLabel 3850 4200 2    50   Input ~ 0
-I2C1_SDA
-Text HLabel 3850 4100 2    50   Input ~ 0
-I2C1_SCL
-Text HLabel 3850 3900 2    50   Input ~ 0
-I2C1_EN
 Text HLabel 3850 3000 2    50   Input ~ 0
 DEBUG_SWCLK
-Text HLabel 2050 5000 0    50   Input ~ 0
-~SPI2_NSS
-Text HLabel 3850 6200 2    50   Input ~ 0
-SPI3_MOSI
-Text HLabel 3850 6100 2    50   Input ~ 0
-SPI3_MISO
-Text HLabel 3850 6000 2    50   Input ~ 0
-SPI3_SCK
 Text HLabel 3850 2900 2    50   Input ~ 0
 DEBUG_SWDIO
-Text HLabel 3850 2800 2    50   Input ~ 0
-USB_DP
-Text HLabel 3850 2700 2    50   Input ~ 0
-USB_DM
-Text HLabel 3850 4600 2    50   Input ~ 0
-SPI2_SCK
-Text HLabel 3850 4700 2    50   Input ~ 0
-SPI2_MISO
-Text HLabel 3850 4800 2    50   Input ~ 0
-SPI2_MOSI
-Text HLabel 3850 2000 2    50   Input ~ 0
-~SPI3_NSS
-Text HLabel 3850 2100 2    50   Input ~ 0
-SPI1_SCK
-Text HLabel 3850 2200 2    50   Input ~ 0
-SPI1_MISO
-Text HLabel 3850 2300 2    50   Input ~ 0
-SPI1_MOSI
-Text HLabel 3850 3300 2    50   Input ~ 0
-~SPI1_NSS
 Text Notes 650  4200 0    50   ~ 0
 CL = 2 * (Cload - Cstray)\nCstray ≈ 20pF, Cstray ≈ 5pF\nCL = 2 * (Cload - 5pF)\nCL = 30pF
@@
 NoConn ~ 3850 2500
 NoConn ~ 3850 2600
-NoConn ~ 3850 5700
 NoConn ~ 2050 5300
 NoConn ~ 2050 5400
@@
 NoConn ~ 3850 3400
 NoConn ~ 3850 3500
-NoConn ~ 3850 3600
-NoConn ~ 3850 3700
-NoConn ~ 3850 3800
-NoConn ~ 3850 4300
-NoConn ~ 3850 4400
 NoConn ~ 3850 5000
 NoConn ~ 3850 5100
@@
 NoConn ~ 3850 5800
 NoConn ~ 3850 5900
-NoConn ~ 2050 6000
-NoConn ~ 2050 6100
 NoConn ~ 2050 6200
 NoConn ~ 2050 6300
@@
 NoConn ~ 3850 6400
 NoConn ~ 3850 6500
-NoConn ~ 3850 4000
-Text HLabel 2050 5800 0    50   Input ~ 0
-SPI2_RST
-Text HLabel 3850 3100 2    50   Input ~ 0
-SPI3_RST
-NoConn ~ 3850 5600
-Text HLabel 2050 5100 0    50   Input ~ 0
-SPI3_EXT_INT
 NoConn ~ 2050 5200
-Text HLabel 2050 5900 0    50   Input ~ 0
-SPI2_EXT_INT
 NoConn ~ 2050 2300
-$Comp
-L power:GNDREF #PWR029
-U 1 1 61C9D008
+Wire Wire Line
+	4700 5700 4700 5850
+Wire Wire Line
+	5050 5850 5050 5600
+Wire Wire Line
+	4700 6250 4700 6150
+Wire Wire Line
+	5050 6250 5050 6150
+$Comp
+L Device:R R?
+U 1 1 61C2F110
+P 5050 6400
+AR Path="/61C2F110" Ref="R?"  Part="1"
+AR Path="/6160DF75/61C2F110" Ref="R?"  Part="1"
+AR Path="/61C99968/61C2F110" Ref="R?"  Part="1"
+F 0 "R?" H 5120 6446 50  0000 L CNN
+F 1 "1k5Ω" H 5120 6355 50  0000 L CNN
+F 2 "Resistor_SMD:R_0603_1608Metric" V 4980 6400 50  0001 C CNN
+F 3 "~" H 5050 6400 50  0001 C CNN
+	1    5050 6400
+	-1   0    0    -1
+$EndComp
+$Comp
+L Device:LED D?
+U 1 1 61C2F116
+P 5050 6000
+AR Path="/61C2F116" Ref="D?"  Part="1"
+AR Path="/6160DF75/61C2F116" Ref="D?"  Part="1"
+AR Path="/61C99968/61C2F116" Ref="D?"  Part="1"
+F 0 "D?" V 5089 5882 50  0000 R CNN
+F 1 "RED" V 4998 5882 50  0000 R CNN
+F 2 "LED_SMD:LED_0603_1608Metric" H 5050 6000 50  0001 C CNN
+F 3 "~" H 5050 6000 50  0001 C CNN
+	1    5050 6000
+	0    1    -1   0
+$EndComp
+$Comp
+L Device:LED D?
+U 1 1 61C2F11C
+P 4700 6000
+AR Path="/61C2F11C" Ref="D?"  Part="1"
+AR Path="/6160DF75/61C2F11C" Ref="D?"  Part="1"
+AR Path="/61C99968/61C2F11C" Ref="D?"  Part="1"
+F 0 "D?" V 4739 5882 50  0000 R CNN
+F 1 "GREEN" V 4648 5882 50  0000 R CNN
+F 2 "LED_SMD:LED_0603_1608Metric" H 4700 6000 50  0001 C CNN
+F 3 "~" H 4700 6000 50  0001 C CNN
+	1    4700 6000
+	0    1    -1   0
+$EndComp
+$Comp
+L Device:R R?
+U 1 1 61C2F122
+P 4700 6400
+AR Path="/61C2F122" Ref="R?"  Part="1"
+AR Path="/6160DF75/61C2F122" Ref="R?"  Part="1"
+AR Path="/61C99968/61C2F122" Ref="R?"  Part="1"
+F 0 "R?" H 4770 6446 50  0000 L CNN
+F 1 "1k5Ω" H 4770 6355 50  0000 L CNN
+F 2 "Resistor_SMD:R_0603_1608Metric" V 4630 6400 50  0001 C CNN
+F 3 "~" H 4700 6400 50  0001 C CNN
+	1    4700 6400
+	-1   0    0    -1
+$EndComp
+Wire Wire Line
+	3850 5700 4700 5700
+Wire Wire Line
+	3850 5600 5050 5600
+NoConn ~ 3850 6100
+NoConn ~ 3850 6000
+NoConn ~ 3850 6200
+NoConn ~ 3850 4100
+NoConn ~ 3850 4600
+NoConn ~ 3850 4700
+NoConn ~ 3850 4800
+$Comp
+L power:GND #PWR?
+U 1 1 61C575EE
+P 4700 6550
+F 0 "#PWR?" H 4700 6300 50  0001 C CNN
+F 1 "GND" H 4705 6377 50  0000 C CNN
+F 2 "" H 4700 6550 50  0001 C CNN
+F 3 "" H 4700 6550 50  0001 C CNN
+	1    4700 6550
+	1    0    0    -1
+$EndComp
+$Comp
+L power:GND #PWR?
+U 1 1 61C598CA
+P 5050 6550
+F 0 "#PWR?" H 5050 6300 50  0001 C CNN
+F 1 "GND" H 5055 6377 50  0000 C CNN
+F 2 "" H 5050 6550 50  0001 C CNN
+F 3 "" H 5050 6550 50  0001 C CNN
+	1    5050 6550
+	1    0    0    -1
+$EndComp
+$Comp
+L power:GND #PWR?
+U 1 1 61C5BB8E
 P 1150 3550
-F 0 "#PWR029" H 1150 3300 50  0001 C CNN
-F 1 "GNDREF" H 1155 3377 50  0000 C CNN
+F 0 "#PWR?" H 1150 3300 50  0001 C CNN
+F 1 "GND" H 1155 3377 50  0000 C CNN
 F 2 "" H 1150 3550 50  0001 C CNN
 F 3 "" H 1150 3550 50  0001 C CNN
@@
 $EndComp
 $Comp
-L power:GNDREF #PWR030
-U 1 1 61C9D81F
+L power:GND #PWR?
+U 1 1 61C5DEA1
 P 1550 3550
-F 0 "#PWR030" H 1550 3300 50  0001 C CNN
-F 1 "GNDREF" H 1555 3377 50  0000 C CNN
+F 0 "#PWR?" H 1550 3300 50  0001 C CNN
+F 1 "GND" H 1555 3377 50  0000 C CNN
 F 2 "" H 1550 3550 50  0001 C CNN
 F 3 "" H 1550 3550 50  0001 C CNN
@@
 	1    0    0    -1
 $EndComp
+Text HLabel 3850 4400 2    50   Input ~ 0
+I2C2_SDA
+Text HLabel 3850 4300 2    50   Input ~ 0
+I2C2_SCL
+Text HLabel 3850 3800 2    50   Input ~ 0
+I2C1_EN
+Text HLabel 3850 3900 2    50   Input ~ 0
+I2C1_SCL
+Text HLabel 3850 4000 2    50   Input ~ 0
+I2C1_SDA
+NoConn ~ 3850 4200
+NoConn ~ 3850 3100
+NoConn ~ 2050 5000
+NoConn ~ 2050 5100
+NoConn ~ 2050 5800
+NoConn ~ 3850 3300
+NoConn ~ 3850 2300
+NoConn ~ 3850 2200
+NoConn ~ 3850 2100
+NoConn ~ 3850 2000
+NoConn ~ 3850 2700
+NoConn ~ 3850 2800
+Text HLabel 2050 6100 0    50   Input ~ 0
+EXT_INT1
+Text HLabel 2050 6000 0    50   Input ~ 0
+EXT_INT2
+Text HLabel 2050 5900 0    50   Input ~ 0
+EXT_INT3
+NoConn ~ 3850 3600
+NoConn ~ 3850 3700
 $EndSCHEMATC

Commit message: Updated component footprints, moved to RDT_Custom_Footprints library
Parts:
- R1, R2: renamed from R?; footprint Resistor_SMD:R_0603_1608Metric -> Resistor_SMD:R_0603_1608Metric_Pad1.05x0.95mm_HandSolder
- gave numbers to parts that had none: 2
Changed lines of the file:
@@
 $Descr A4 11693 8268
 encoding utf-8
-Sheet 7 7
+Sheet 6 7
 Title ""
 Date "2021-12-20"
@@
 AR Path="/61C2F110" Ref="R?"  Part="1"
 AR Path="/6160DF75/61C2F110" Ref="R?"  Part="1"
-AR Path="/61C99968/61C2F110" Ref="R?"  Part="1"
-F 0 "R?" H 5120 6446 50  0000 L CNN
+AR Path="/61C99968/61C2F110" Ref="R2"  Part="1"
+F 0 "R2" H 5120 6446 50  0000 L CNN
 F 1 "1k5Ω" H 5120 6355 50  0000 L CNN
-F 2 "Resistor_SMD:R_0603_1608Metric" V 4980 6400 50  0001 C CNN
+F 2 "Resistor_SMD:R_0603_1608Metric_Pad1.05x0.95mm_HandSolder" V 4980 6400 50  0001 C CNN
 F 3 "~" H 5050 6400 50  0001 C CNN
 	1    5050 6400
@@
 AR Path="/61C2F116" Ref="D?"  Part="1"
 AR Path="/6160DF75/61C2F116" Ref="D?"  Part="1"
-AR Path="/61C99968/61C2F116" Ref="D?"  Part="1"
-F 0 "D?" V 5089 5882 50  0000 R CNN
+AR Path="/61C99968/61C2F116" Ref="D2"  Part="1"
+F 0 "D2" V 5089 5882 50  0000 R CNN
 F 1 "RED" V 4998 5882 50  0000 R CNN
 F 2 "LED_SMD:LED_0603_1608Metric" H 5050 6000 50  0001 C CNN
@@
 AR Path="/61C2F11C" Ref="D?"  Part="1"
 AR Path="/6160DF75/61C2F11C" Ref="D?"  Part="1"
-AR Path="/61C99968/61C2F11C" Ref="D?"  Part="1"
-F 0 "D?" V 4739 5882 50  0000 R CNN
+AR Path="/61C99968/61C2F11C" Ref="D1"  Part="1"
+F 0 "D1" V 4739 5882 50  0000 R CNN
 F 1 "GREEN" V 4648 5882 50  0000 R CNN
 F 2 "LED_SMD:LED_0603_1608Metric" H 4700 6000 50  0001 C CNN
@@
 AR Path="/61C2F122" Ref="R?"  Part="1"
 AR Path="/6160DF75/61C2F122" Ref="R?"  Part="1"
-AR Path="/61C99968/61C2F122" Ref="R?"  Part="1"
-F 0 "R?" H 4770 6446 50  0000 L CNN
+AR Path="/61C99968/61C2F122" Ref="R1"  Part="1"
+F 0 "R1" H 4770 6446 50  0000 L CNN
 F 1 "1k5Ω" H 4770 6355 50  0000 L CNN
-F 2 "Resistor_SMD:R_0603_1608Metric" V 4630 6400 50  0001 C CNN
+F 2 "Resistor_SMD:R_0603_1608Metric_Pad1.05x0.95mm_HandSolder" V 4630 6400 50  0001 C CNN
 F 3 "~" H 4700 6400 50  0001 C CNN
 	1    4700 6400
@@
 NoConn ~ 3850 4800
 $Comp
-L power:GND #PWR?
+L power:GND #PWR0110
 U 1 1 61C575EE
 P 4700 6550
-F 0 "#PWR?" H 4700 6300 50  0001 C CNN
+F 0 "#PWR0110" H 4700 6300 50  0001 C CNN
 F 1 "GND" H 4705 6377 50  0000 C CNN
 F 2 "" H 4700 6550 50  0001 C CNN
@@
 $EndComp
 $Comp
-L power:GND #PWR?
+L power:GND #PWR0111
 U 1 1 61C598CA
 P 5050 6550
-F 0 "#PWR?" H 5050 6300 50  0001 C CNN
+F 0 "#PWR0111" H 5050 6300 50  0001 C CNN
 F 1 "GND" H 5055 6377 50  0000 C CNN
 F 2 "" H 5050 6550 50  0001 C CNN
@@
 $EndComp
 $Comp
-L power:GND #PWR?
+L power:GND #PWR0112
 U 1 1 61C5BB8E
 P 1150 3550
-F 0 "#PWR?" H 1150 3300 50  0001 C CNN
+F 0 "#PWR0112" H 1150 3300 50  0001 C CNN
 F 1 "GND" H 1155 3377 50  0000 C CNN
 F 2 "" H 1150 3550 50  0001 C CNN
@@
 $EndComp
 $Comp
-L power:GND #PWR?
+L power:GND #PWR0113
 U 1 1 61C5DEA1
 P 1550 3550
-F 0 "#PWR?" H 1550 3300 50  0001 C CNN
+F 0 "#PWR0113" H 1550 3300 50  0001 C CNN
 F 1 "GND" H 1555 3377 50  0000 C CNN
 F 2 "" H 1550 3550 50  0001 C CNN

Commit message: Reset annotations, changed SPST switch footprint
Parts:
- renumbered C30 to C24, C31 to C25, C32 to C26, C33 to C27, C34 to C28, C35 to C29, C36 to C30, C37 to C31, C38 to C32, C39 to C33, C40 to C34, C41 to C35, D1 to D5, D2 to D6, R1 to R16, R2 to R17, Y2 to Y1
Changed lines of the file:
@@
 AR Path="/619FB6DF/61A17DD9" Ref="#PWR?"  Part="1"
 AR Path="/61A107A5/61A17DD9" Ref="#PWR?"  Part="1"
-AR Path="/61C99968/61A17DD9" Ref="#PWR033"  Part="1"
-F 0 "#PWR033" H 6600 1150 50  0001 C CNN
+AR Path="/61C99968/61A17DD9" Ref="#PWR035"  Part="1"
+F 0 "#PWR035" H 6600 1150 50  0001 C CNN
 F 1 "+3.3V" H 6615 1473 50  0000 C CNN
 F 2 "" H 6600 1300 50  0001 C CNN
@@
 AR Path="/619FB6DF/61A17DDF" Ref="C?"  Part="1"
 AR Path="/61A107A5/61A17DDF" Ref="C?"  Part="1"
-AR Path="/61C99968/61A17DDF" Ref="C32"  Part="1"
-F 0 "C32" H 6692 1546 50  0000 L CNN
+AR Path="/61C99968/61A17DDF" Ref="C26"  Part="1"
+F 0 "C26" H 6692 1546 50  0000 L CNN
 F 1 "1uF" H 6692 1455 50  0000 L CNN
 F 2 "Capacitor_SMD:C_0603_1608Metric_Pad1.08x0.95mm_HandSolder" H 6600 1500 50  0001 C CNN
@@
 AR Path="/619FB6DF/61A17DE5" Ref="C?"  Part="1"
 AR Path="/61A107A5/61A17DE5" Ref="C?"  Part="1"
-AR Path="/61C99968/61A17DE5" Ref="C33"  Part="1"
-F 0 "C33" H 7092 1546 50  0000 L CNN
+AR Path="/61C99968/61A17DE5" Ref="C27"  Part="1"
+F 0 "C27" H 7092 1546 50  0000 L CNN
 F 1 "100nF" H 7092 1455 50  0000 L CNN
 F 2 "Capacitor_SMD:C_0603_1608Metric_Pad1.08x0.95mm_HandSolder" H 7000 1500 50  0001 C CNN
@@
 AR Path="/619FB6DF/61A17DEB" Ref="C?"  Part="1"
 AR Path="/61A107A5/61A17DEB" Ref="C?"  Part="1"
-AR Path="/61C99968/61A17DEB" Ref="C34"  Part="1"
-F 0 "C34" H 7542 1546 50  0000 L CNN
+AR Path="/61C99968/61A17DEB" Ref="C28"  Part="1"
+F 0 "C28" H 7542 1546 50  0000 L CNN
 F 1 "100nF" H 7542 1455 50  0000 L CNN
 F 2 "Capacitor_SMD:C_0603_1608Metric_Pad1.08x0.95mm_HandSolder" H 7450 1500 50  0001 C CNN
@@
 AR Path="/619FB6DF/61A17DF1" Ref="C?"  Part="1"
 AR Path="/61A107A5/61A17DF1" Ref="C?"  Part="1"
-AR Path="/61C99968/61A17DF1" Ref="C37"  Part="1"
-F 0 "C37" H 8892 1546 50  0000 L CNN
+AR Path="/61C99968/61A17DF1" Ref="C31"  Part="1"
+F 0 "C31" H 8892 1546 50  0000 L CNN
 F 1 "100nF" H 8892 1455 50  0000 L CNN
 F 2 "Capacitor_SMD:C_0603_1608Metric_Pad1.08x0.95mm_HandSolder" H 8800 1500 50  0001 C CNN
@@
 AR Path="/619FB6DF/61A17DF7" Ref="C?"  Part="1"
 AR Path="/61A107A5/61A17DF7" Ref="C?"  Part="1"
-AR Path="/61C99968/61A17DF7" Ref="C41"  Part="1"
-F 0 "C41" H 10692 1546 50  0000 L CNN
+AR Path="/61C99968/61A17DF7" Ref="C35"  Part="1"
+F 0 "C35" H 10692 1546 50  0000 L CNN
 F 1 "100nF" H 10692 1455 50  0000 L CNN
 F 2 "Capacitor_SMD:C_0603_1608Metric_Pad1.08x0.95mm_HandSolder" H 10600 1500 50  0001 C CNN
@@
 AR Path="/619FB6DF/61A17DFD" Ref="#PWR?"  Part="1"
 AR Path="/61A107A5/61A17DFD" Ref="#PWR?"  Part="1"
-AR Path="/61C99968/61A17DFD" Ref="#PWR034"  Part="1"
-F 0 "#PWR034" H 6600 1450 50  0001 C CNN
+AR Path="/61C99968/61A17DFD" Ref="#PWR036"  Part="1"
+F 0 "#PWR036" H 6600 1450 50  0001 C CNN
 F 1 "GND" H 6605 1527 50  0000 C CNN
 F 2 "" H 6600 1700 50  0001 C CNN
@@
 AR Path="/619FB6DF/61A17E24" Ref="#PWR?"  Part="1"
 AR Path="/61A107A5/61A17E24" Ref="#PWR?"  Part="1"
-AR Path="/61C99968/61A17E24" Ref="#PWR035"  Part="1"
-F 0 "#PWR035" H 7400 3100 50  0001 C CNN
+AR Path="/61C99968/61A17E24" Ref="#PWR037"  Part="1"
+F 0 "#PWR037" H 7400 3100 50  0001 C CNN
 F 1 "+3.3V" H 7415 3423 50  0000 C CNN
 F 2 "" H 7400 3250 50  0001 C CNN
@@
 AR Path="/619FB6DF/61A89EEB" Ref="C?"  Part="1"
 AR Path="/61A107A5/61A89EEB" Ref="C?"  Part="1"
-AR Path="/61C99968/61A89EEB" Ref="C35"  Part="1"
-F 0 "C35" H 7992 1546 50  0000 L CNN
+AR Path="/61C99968/61A89EEB" Ref="C29"  Part="1"
+F 0 "C29" H 7992 1546 50  0000 L CNN
 F 1 "100nF" H 7992 1455 50  0000 L CNN
 F 2 "Capacitor_SMD:C_0603_1608Metric_Pad1.08x0.95mm_HandSolder" H 7900 1500 50  0001 C CNN
@@
 AR Path="/619FB6DF/61A89EF1" Ref="C?"  Part="1"
 AR Path="/61A107A5/61A89EF1" Ref="C?"  Part="1"
-AR Path="/61C99968/61A89EF1" Ref="C36"  Part="1"
-F 0 "C36" H 8442 1546 50  0000 L CNN
+AR Path="/61C99968/61A89EF1" Ref="C30"  Part="1"
+F 0 "C30" H 8442 1546 50  0000 L CNN
 F 1 "100nF" H 8442 1455 50  0000 L CNN
 F 2 "Capacitor_SMD:C_0603_1608Metric_Pad1.08x0.95mm_HandSolder" H 8350 1500 50  0001 C CNN
@@
 AR Path="/619FB6DF/61AA18EF" Ref="C?"  Part="1"
 AR Path="/61A107A5/61AA18EF" Ref="C?"  Part="1"
-AR Path="/61C99968/61AA18EF" Ref="C38"  Part="1"
-F 0 "C38" H 9342 1546 50  0000 L CNN
+AR Path="/61C99968/61AA18EF" Ref="C32"  Part="1"
+F 0 "C32" H 9342 1546 50  0000 L CNN
 F 1 "100nF" H 9342 1455 50  0000 L CNN
 F 2 "Capacitor_SMD:C_0603_1608Metric_Pad1.08x0.95mm_HandSolder" H 9250 1500 50  0001 C CNN
@@
 AR Path="/619FB6DF/61AA2382" Ref="C?"  Part="1"
 AR Path="/61A107A5/61AA2382" Ref="C?"  Part="1"
-AR Path="/61C99968/61AA2382" Ref="C39"  Part="1"
-F 0 "C39" H 9792 1546 50  0000 L CNN
+AR Path="/61C99968/61AA2382" Ref="C33"  Part="1"
+F 0 "C33" H 9792 1546 50  0000 L CNN
 F 1 "100nF" H 9792 1455 50  0000 L CNN
 F 2 "Capacitor_SMD:C_0603_1608Metric_Pad1.08x0.95mm_HandSolder" H 9700 1500 50  0001 C CNN
@@
 AR Path="/619FB6DF/61AA2953" Ref="C?"  Part="1"
 AR Path="/61A107A5/61AA2953" Ref="C?"  Part="1"
-AR Path="/61C99968/61AA2953" Ref="C40"  Part="1"
-F 0 "C40" H 10242 1546 50  0000 L CNN
+AR Path="/61C99968/61AA2953" Ref="C34"  Part="1"
+F 0 "C34" H 10242 1546 50  0000 L CNN
 F 1 "100nF" H 10242 1455 50  0000 L CNN
 F 2 "Capacitor_SMD:C_0603_1608Metric_Pad1.08x0.95mm_HandSolder" H 10150 1500 50  0001 C CNN
@@
 AR Path="/619FB6DF/61ADFE6A" Ref="C?"  Part="1"
 AR Path="/61A107A5/61ADFE6A" Ref="C?"  Part="1"
-AR Path="/61C99968/61ADFE6A" Ref="C30"  Part="1"
-F 0 "C30" H 1242 3496 50  0000 L CNN
+AR Path="/61C99968/61ADFE6A" Ref="C24"  Part="1"
+F 0 "C24" H 1242 3496 50  0000 L CNN
 F 1 "30pF" H 1242 3405 50  0000 L CNN
 F 2 "Capacitor_SMD:C_0603_1608Metric_Pad1.08x0.95mm_HandSolder" H 1150 3450 50  0001 C CNN
@@
 AR Path="/619FB6DF/61ADFE7C" Ref="C?"  Part="1"
 AR Path="/61A107A5/61ADFE7C" Ref="C?"  Part="1"
-AR Path="/61C99968/61ADFE7C" Ref="C31"  Part="1"
-F 0 "C31" H 1642 3496 50  0000 L CNN
+AR Path="/61C99968/61ADFE7C" Ref="C25"  Part="1"
+F 0 "C25" H 1642 3496 50  0000 L CNN
 F 1 "30pF" H 1642 3405 50  0000 L CNN
 F 2 "Capacitor_SMD:C_0603_1608Metric_Pad1.08x0.95mm_HandSolder" H 1550 3450 50  0001 C CNN
@@
 AR Path="/619FB6DF/61ADFE82" Ref="Y?"  Part="1"
 AR Path="/61A107A5/61ADFE82" Ref="Y?"  Part="1"
-AR Path="/61C99968/61ADFE82" Ref="Y2"  Part="1"
-F 0 "Y2" H 1350 3475 50  0000 C CNN
+AR Path="/61C99968/61ADFE82" Ref="Y1"  Part="1"
+F 0 "Y1" H 1350 3475 50  0000 C CNN
 F 1 "32MHz" H 1350 3384 50  0000 C CNN
 F 2 "Crystal:Crystal_SMD_2012-2Pin_2.0x1.2mm_HandSoldering" H 1350 3250 50  0001 C CNN
@@
 AR Path="/61C2F110" Ref="R?"  Part="1"
 AR Path="/6160DF75/61C2F110" Ref="R?"  Part="1"
-AR Path="/61C99968/61C2F110" Ref="R2"  Part="1"
-F 0 "R2" H 5120 6446 50  0000 L CNN
+AR Path="/61C99968/61C2F110" Ref="R17"  Part="1"
+F 0 "R17" H 5120 6446 50  0000 L CNN
 F 1 "1k5Ω" H 5120 6355 50  0000 L CNN
 F 2 "Resistor_SMD:R_0603_1608Metric_Pad1.05x0.95mm_HandSolder" V 4980 6400 50  0001 C CNN
@@
 AR Path="/61C2F116" Ref="D?"  Part="1"
 AR Path="/6160DF75/61C2F116" Ref="D?"  Part="1"
-AR Path="/61C99968/61C2F116" Ref="D2"  Part="1"
-F 0 "D2" V 5089 5882 50  0000 R CNN
+AR Path="/61C99968/61C2F116" Ref="D6"  Part="1"
+F 0 "D6" V 5089 5882 50  0000 R CNN
 F 1 "RED" V 4998 5882 50  0000 R CNN
 F 2 "LED_SMD:LED_0603_1608Metric" H 5050 6000 50  0001 C CNN
@@
 AR Path="/61C2F11C" Ref="D?"  Part="1"
 AR Path="/6160DF75/61C2F11C" Ref="D?"  Part="1"
-AR Path="/61C99968/61C2F11C" Ref="D1"  Part="1"
-F 0 "D1" V 4739 5882 50  0000 R CNN
+AR Path="/61C99968/61C2F11C" Ref="D5"  Part="1"
+F 0 "D5" V 4739 5882 50  0000 R CNN
 F 1 "GREEN" V 4648 5882 50  0000 R CNN
 F 2 "LED_SMD:LED_0603_1608Metric" H 4700 6000 50  0001 C CNN
@@
 AR Path="/61C2F122" Ref="R?"  Part="1"
 AR Path="/6160DF75/61C2F122" Ref="R?"  Part="1"
-AR Path="/61C99968/61C2F122" Ref="R1"  Part="1"
-F 0 "R1" H 4770 6446 50  0000 L CNN
+AR Path="/61C99968/61C2F122" Ref="R16"  Part="1"
+F 0 "R16" H 4770 6446 50  0000 L CNN
 F 1 "1k5Ω" H 4770 6355 50  0000 L CNN
 F 2 "Resistor_SMD:R_0603_1608Metric_Pad1.05x0.95mm_HandSolder" V 4630 6400 50  0001 C CNN
@@
 NoConn ~ 3850 4800
 $Comp
-L power:GND #PWR0110
+L power:GND #PWR033
 U 1 1 61C575EE
 P 4700 6550
-F 0 "#PWR0110" H 4700 6300 50  0001 C CNN
+F 0 "#PWR033" H 4700 6300 50  0001 C CNN
 F 1 "GND" H 4705 6377 50  0000 C CNN
 F 2 "" H 4700 6550 50  0001 C CNN
@@
 $EndComp
 $Comp
-L power:GND #PWR0111
+L power:GND #PWR034
 U 1 1 61C598CA
 P 5050 6550
-F 0 "#PWR0111" H 5050 6300 50  0001 C CNN
+F 0 "#PWR034" H 5050 6300 50  0001 C CNN
 F 1 "GND" H 5055 6377 50  0000 C CNN
 F 2 "" H 5050 6550 50  0001 C CNN
@@
 $EndComp
 $Comp
-L power:GND #PWR0112
+L power:GND #PWR029
 U 1 1 61C5BB8E
 P 1150 3550
-F 0 "#PWR0112" H 1150 3300 50  0001 C CNN
+F 0 "#PWR029" H 1150 3300 50  0001 C CNN
 F 1 "GND" H 1155 3377 50  0000 C CNN
 F 2 "" H 1150 3550 50  0001 C CNN
@@
 $EndComp
 $Comp
-L power:GND #PWR0113
+L power:GND #PWR030
 U 1 1 61C5DEA1
 P 1550 3550
-F 0 "#PWR0113" H 1550 3300 50  0001 C CNN
+F 0 "#PWR030" H 1550 3300 50  0001 C CNN
 F 1 "GND" H 1555 3377 50  0000 C CNN
 F 2 "" H 1550 3550 50  0001 C CNN

Commit message: Routed I2C lines between temp sensors, lipo monitor, and mcu
Connections:
- no-connect marks 69 -> 68
Changed lines of the file:
@@
 Text HLabel 3850 2900 2    50   Input ~ 0
 DEBUG_SWDIO
-Text Notes 650  4200 0    50   ~ 0
+Text Notes 600  2850 0    50   ~ 0
 CL = 2 * (Cload - Cstray)\nCstray ≈ 20pF, Cstray ≈ 5pF\nCL = 2 * (Cload - 5pF)\nCL = 30pF
 Wire Wire Line
@@
 NoConn ~ 2050 3800
 NoConn ~ 2050 3900
-NoConn ~ 2050 4000
-NoConn ~ 2050 4100
-NoConn ~ 2050 4200
 NoConn ~ 2050 4300
 NoConn ~ 2050 4400
@@
 NoConn ~ 3850 2700
 NoConn ~ 3850 2800
-Text HLabel 2050 6100 0    50   Input ~ 0
+Text HLabel 2050 4100 0    50   Input ~ 0
 EXT_INT1
-Text HLabel 2050 6000 0    50   Input ~ 0
+Text HLabel 2050 4200 0    50   Input ~ 0
 EXT_INT2
-Text HLabel 2050 5900 0    50   Input ~ 0
+Text HLabel 2050 4000 0    50   Input ~ 0
 EXT_INT3
 NoConn ~ 3850 3600
 NoConn ~ 3850 3700
+NoConn ~ 2050 6000
+NoConn ~ 2050 6100
 $EndSCHEMATC
