File: Hardware/COMPONENT_SHEETS/MCU_L562VE.sch (KiCad schematic (older format))
At the start: 20 parts, among them U6 STM32L562VET, Y1 32MHz

Commit message: Routed data busses from MCU to DB37
Changed lines of the file:
@@
 NoConn ~ 2050 3800
 NoConn ~ 2050 3900
-NoConn ~ 2050 4300
-NoConn ~ 2050 4400
 NoConn ~ 2050 4500
 NoConn ~ 2050 4600
@@
 NoConn ~ 2050 2300
 Wire Wire Line
-	4700 5700 4700 5850
+	1050 5200 1050 5100
 Wire Wire Line
-	5050 5850 5050 5600
-Wire Wire Line
-	4700 6250 4700 6150
-Wire Wire Line
-	5050 6250 5050 6150
+	1400 5200 1400 5100
 $Comp
 L Device:R R?
 U 1 1 61C2F110
-P 5050 6400
+P 1400 5350
 AR Path="/61C2F110" Ref="R?"  Part="1"
 AR Path="/6160DF75/61C2F110" Ref="R?"  Part="1"
 AR Path="/61C99968/61C2F110" Ref="R17"  Part="1"
-F 0 "R17" H 5120 6446 50  0000 L CNN
-F 1 "1k5Ω" H 5120 6355 50  0000 L CNN
-F 2 "Resistor_SMD:R_0603_1608Metric_Pad1.05x0.95mm_HandSolder" V 4980 6400 50  0001 C CNN
-F 3 "~" H 5050 6400 50  0001 C CNN
-	1    5050 6400
+F 0 "R17" H 1470 5396 50  0000 L CNN
+F 1 "1k5Ω" H 1470 5305 50  0000 L CNN
+F 2 "Resistor_SMD:R_0603_1608Metric_Pad1.05x0.95mm_HandSolder" V 1330 5350 50  0001 C CNN
+F 3 "~" H 1400 5350 50  0001 C CNN
+	1    1400 5350
 	-1   0    0    -1
 $EndComp
@@
 L Device:LED D?
 U 1 1 61C2F116
-P 5050 6000
+P 1400 4950
 AR Path="/61C2F116" Ref="D?"  Part="1"
 AR Path="/6160DF75/61C2F116" Ref="D?"  Part="1"
 AR Path="/61C99968/61C2F116" Ref="D6"  Part="1"
-F 0 "D6" V 5089 5882 50  0000 R CNN
-F 1 "RED" V 4998 5882 50  0000 R CNN
-F 2 "LED_SMD:LED_0603_1608Metric" H 5050 6000 50  0001 C CNN
-F 3 "~" H 5050 6000 50  0001 C CNN
-	1    5050 6000
+F 0 "D6" V 1439 4832 50  0000 R CNN
+F 1 "RED" V 1348 4832 50  0000 R CNN
+F 2 "LED_SMD:LED_0603_1608Metric" H 1400 4950 50  0001 C CNN
+F 3 "~" H 1400 4950 50  0001 C CNN
+	1    1400 4950
 	0    1    -1   0
 $EndComp
@@
 L Device:LED D?
 U 1 1 61C2F11C
-P 4700 6000
+P 1050 4950
 AR Path="/61C2F11C" Ref="D?"  Part="1"
 AR Path="/6160DF75/61C2F11C" Ref="D?"  Part="1"
 AR Path="/61C99968/61C2F11C" Ref="D5"  Part="1"
-F 0 "D5" V 4739 5882 50  0000 R CNN
-F 1 "GREEN" V 4648 5882 50  0000 R CNN
-F 2 "LED_SMD:LED_0603_1608Metric" H 4700 6000 50  0001 C CNN
-F 3 "~" H 4700 6000 50  0001 C CNN
-	1    4700 6000
+F 0 "D5" V 1089 4832 50  0000 R CNN
+F 1 "GREEN" V 998 4832 50  0000 R CNN
+F 2 "LED_SMD:LED_0603_1608Metric" H 1050 4950 50  0001 C CNN
+F 3 "~" H 1050 4950 50  0001 C CNN
+	1    1050 4950
 	0    1    -1   0
 $EndComp
@@
 L Device:R R?
 U 1 1 61C2F122
-P 4700 6400
+P 1050 5350
 AR Path="/61C2F122" Ref="R?"  Part="1"
 AR Path="/6160DF75/61C2F122" Ref="R?"  Part="1"
 AR Path="/61C99968/61C2F122" Ref="R16"  Part="1"
-F 0 "R16" H 4770 6446 50  0000 L CNN
-F 1 "1k5Ω" H 4770 6355 50  0000 L CNN
-F 2 "Resistor_SMD:R_0603_1608Metric_Pad1.05x0.95mm_HandSolder" V 4630 6400 50  0001 C CNN
-F 3 "~" H 4700 6400 50  0001 C CNN
-	1    4700 6400
+F 0 "R16" H 1120 5396 50  0000 L CNN
+F 1 "1k5Ω" H 1120 5305 50  0000 L CNN
+F 2 "Resistor_SMD:R_0603_1608Metric_Pad1.05x0.95mm_HandSolder" V 980 5350 50  0001 C CNN
+F 3 "~" H 1050 5350 50  0001 C CNN
+	1    1050 5350
 	-1   0    0    -1
 $EndComp
-Wire Wire Line
-	3850 5700 4700 5700
-Wire Wire Line
-	3850 5600 5050 5600
 NoConn ~ 3850 6100
 NoConn ~ 3850 6000
@@
 L power:GND #PWR033
 U 1 1 61C575EE
-P 4700 6550
-F 0 "#PWR033" H 4700 6300 50  0001 C CNN
-F 1 "GND" H 4705 6377 50  0000 C CNN
-F 2 "" H 4700 6550 50  0001 C CNN
-F 3 "" H 4700 6550 50  0001 C CNN
-	1    4700 6550
+P 1050 5500
+F 0 "#PWR033" H 1050 5250 50  0001 C CNN
+F 1 "GND" H 1055 5327 50  0000 C CNN
+F 2 "" H 1050 5500 50  0001 C CNN
+F 3 "" H 1050 5500 50  0001 C CNN
+	1    1050 5500
 	1    0    0    -1
 $EndComp
@@
 L power:GND #PWR034
 U 1 1 61C598CA
-P 5050 6550
-F 0 "#PWR034" H 5050 6300 50  0001 C CNN
-F 1 "GND" H 5055 6377 50  0000 C CNN
-F 2 "" H 5050 6550 50  0001 C CNN
-F 3 "" H 5050 6550 50  0001 C CNN
-	1    5050 6550
+P 1400 5500
+F 0 "#PWR034" H 1400 5250 50  0001 C CNN
+F 1 "GND" H 1405 5327 50  0000 C CNN
+F 2 "" H 1400 5500 50  0001 C CNN
+F 3 "" H 1400 5500 50  0001 C CNN
+	1    1400 5500
 	1    0    0    -1
 $EndComp
@@
 NoConn ~ 2050 6000
 NoConn ~ 2050 6100
+Wire Wire Line
+	1400 4400 2050 4400
+Wire Wire Line
+	1400 4400 1400 4800
+Wire Wire Line
+	2050 4300 1050 4300
+Wire Wire Line
+	1050 4300 1050 4800
+NoConn ~ 3850 5600
+NoConn ~ 3850 5700
 $EndSCHEMATC

Commit message: Moved external switch connector to pack+, added missing no connection flags
This change renders the current PCB layout defunct, next commits will be redesigns of the layout.
Connections:
- no-connect marks 68 -> 69
Changed lines of the file:
@@
 NoConn ~ 3850 5600
 NoConn ~ 3850 5700
+NoConn ~ 2050 5900
 $EndSCHEMATC

Commit message: Routed all connections and placed all components
MCU crystal still needs a ground peninsula
Connections:
- net labels added: I2C2_EN
- no-connect marks 69 -> 68
Changed lines of the file:
@@
 Wire Wire Line
 	2050 2900 1150 2900
-Text HLabel 2050 4700 0    50   Input ~ 0
-ABORT_1
-Text HLabel 2050 4800 0    50   Input ~ 0
-ABORT_2
 Text HLabel 2050 1600 0    50   Input ~ 0
 NRST
@@
 NoConn ~ 2050 3800
 NoConn ~ 2050 3900
-NoConn ~ 2050 4500
-NoConn ~ 2050 4600
 NoConn ~ 3850 2500
 NoConn ~ 3850 2600
@@
 NoConn ~ 3850 1900
 NoConn ~ 3850 2400
-NoConn ~ 3850 3400
-NoConn ~ 3850 3500
 NoConn ~ 3850 5000
 NoConn ~ 3850 5100
@@
 NoConn ~ 2050 2300
 Wire Wire Line
-	1050 5200 1050 5100
-Wire Wire Line
-	1400 5200 1400 5100
+	4950 3100 4950 3000
+Wire Wire Line
+	5300 3100 5300 3000
 $Comp
 L Device:R R?
 U 1 1 61C2F110
-P 1400 5350
+P 5300 3250
 AR Path="/61C2F110" Ref="R?"  Part="1"
 AR Path="/6160DF75/61C2F110" Ref="R?"  Part="1"
 AR Path="/61C99968/61C2F110" Ref="R17"  Part="1"
-F 0 "R17" H 1470 5396 50  0000 L CNN
-F 1 "1k5Ω" H 1470 5305 50  0000 L CNN
-F 2 "Resistor_SMD:R_0603_1608Metric_Pad1.05x0.95mm_HandSolder" V 1330 5350 50  0001 C CNN
-F 3 "~" H 1400 5350 50  0001 C CNN
-	1    1400 5350
+F 0 "R17" H 5370 3296 50  0000 L CNN
+F 1 "1k5Ω" H 5370 3205 50  0000 L CNN
+F 2 "Resistor_SMD:R_0603_1608Metric_Pad1.05x0.95mm_HandSolder" V 5230 3250 50  0001 C CNN
+F 3 "~" H 5300 3250 50  0001 C CNN
+	1    5300 3250
 	-1   0    0    -1
 $EndComp
@@
 L Device:LED D?
 U 1 1 61C2F116
-P 1400 4950
+P 5300 2850
 AR Path="/61C2F116" Ref="D?"  Part="1"
 AR Path="/6160DF75/61C2F116" Ref="D?"  Part="1"
 AR Path="/61C99968/61C2F116" Ref="D6"  Part="1"
-F 0 "D6" V 1439 4832 50  0000 R CNN
-F 1 "RED" V 1348 4832 50  0000 R CNN
-F 2 "LED_SMD:LED_0603_1608Metric" H 1400 4950 50  0001 C CNN
-F 3 "~" H 1400 4950 50  0001 C CNN
-	1    1400 4950
+F 0 "D6" V 5339 2732 50  0000 R CNN
+F 1 "RED" V 5248 2732 50  0000 R CNN
+F 2 "LED_SMD:LED_0603_1608Metric" H 5300 2850 50  0001 C CNN
+F 3 "~" H 5300 2850 50  0001 C CNN
+	1    5300 2850
 	0    1    -1   0
 $EndComp
@@
 L Device:LED D?
 U 1 1 61C2F11C
-P 1050 4950
+P 4950 2850
 AR Path="/61C2F11C" Ref="D?"  Part="1"
 AR Path="/6160DF75/61C2F11C" Ref="D?"  Part="1"
 AR Path="/61C99968/61C2F11C" Ref="D5"  Part="1"
-F 0 "D5" V 1089 4832 50  0000 R CNN
-F 1 "GREEN" V 998 4832 50  0000 R CNN
-F 2 "LED_SMD:LED_0603_1608Metric" H 1050 4950 50  0001 C CNN
-F 3 "~" H 1050 4950 50  0001 C CNN
-	1    1050 4950
+F 0 "D5" V 4989 2732 50  0000 R CNN
+F 1 "GREEN" V 4898 2732 50  0000 R CNN
+F 2 "LED_SMD:LED_0603_1608Metric" H 4950 2850 50  0001 C CNN
+F 3 "~" H 4950 2850 50  0001 C CNN
+	1    4950 2850
 	0    1    -1   0
 $EndComp
@@
 L Device:R R?
 U 1 1 61C2F122
-P 1050 5350
+P 4950 3250
 AR Path="/61C2F122" Ref="R?"  Part="1"
 AR Path="/6160DF75/61C2F122" Ref="R?"  Part="1"
 AR Path="/61C99968/61C2F122" Ref="R16"  Part="1"
-F 0 "R16" H 1120 5396 50  0000 L CNN
-F 1 "1k5Ω" H 1120 5305 50  0000 L CNN
-F 2 "Resistor_SMD:R_0603_1608Metric_Pad1.05x0.95mm_HandSolder" V 980 5350 50  0001 C CNN
-F 3 "~" H 1050 5350 50  0001 C CNN
-	1    1050 5350
+F 0 "R16" H 5020 3296 50  0000 L CNN
+F 1 "1k5Ω" H 5020 3205 50  0000 L CNN
+F 2 "Resistor_SMD:R_0603_1608Metric_Pad1.05x0.95mm_HandSolder" V 4880 3250 50  0001 C CNN
+F 3 "~" H 4950 3250 50  0001 C CNN
+	1    4950 3250
 	-1   0    0    -1
 $EndComp
@@
 NoConn ~ 3850 6200
 NoConn ~ 3850 4100
-NoConn ~ 3850 4600
 NoConn ~ 3850 4700
 NoConn ~ 3850 4800
@@
 L power:GND #PWR033
 U 1 1 61C575EE
-P 1050 5500
-F 0 "#PWR033" H 1050 5250 50  0001 C CNN
-F 1 "GND" H 1055 5327 50  0000 C CNN
-F 2 "" H 1050 5500 50  0001 C CNN
-F 3 "" H 1050 5500 50  0001 C CNN
-	1    1050 5500
+P 4950 3400
+F 0 "#PWR033" H 4950 3150 50  0001 C CNN
+F 1 "GND" H 4955 3227 50  0000 C CNN
+F 2 "" H 4950 3400 50  0001 C CNN
+F 3 "" H 4950 3400 50  0001 C CNN
+	1    4950 3400
 	1    0    0    -1
 $EndComp
@@
 L power:GND #PWR034
 U 1 1 61C598CA
-P 1400 5500
-F 0 "#PWR034" H 1400 5250 50  0001 C CNN
-F 1 "GND" H 1405 5327 50  0000 C CNN
-F 2 "" H 1400 5500 50  0001 C CNN
-F 3 "" H 1400 5500 50  0001 C CNN
-	1    1400 5500
+P 5300 3400
+F 0 "#PWR034" H 5300 3150 50  0001 C CNN
+F 1 "GND" H 5305 3227 50  0000 C CNN
+F 2 "" H 5300 3400 50  0001 C CNN
+F 3 "" H 5300 3400 50  0001 C CNN
+	1    5300 3400
 	1    0    0    -1
 $EndComp
@@
 NoConn ~ 2050 5100
 NoConn ~ 2050 5800
-NoConn ~ 3850 3300
-NoConn ~ 3850 2300
-NoConn ~ 3850 2200
 NoConn ~ 3850 2100
 NoConn ~ 3850 2000
 NoConn ~ 3850 2700
 NoConn ~ 3850 2800
-Text HLabel 2050 4100 0    50   Input ~ 0
+Text HLabel 3850 3300 2    50   Input ~ 0
 EXT_INT1
-Text HLabel 2050 4200 0    50   Input ~ 0
+Text HLabel 2050 4300 0    50   Input ~ 0
 EXT_INT2
-Text HLabel 2050 4000 0    50   Input ~ 0
+Text HLabel 3850 3500 2    50   Input ~ 0
 EXT_INT3
 NoConn ~ 3850 3600
@@
 NoConn ~ 2050 6000
 NoConn ~ 2050 6100
-Wire Wire Line
-	1400 4400 2050 4400
-Wire Wire Line
-	1400 4400 1400 4800
-Wire Wire Line
-	2050 4300 1050 4300
-Wire Wire Line
-	1050 4300 1050 4800
 NoConn ~ 3850 5600
 NoConn ~ 3850 5700
 NoConn ~ 2050 5900
+NoConn ~ 2050 4700
+Wire Wire Line
+	5300 2700 5300 2200
+Wire Wire Line
+	4950 2300 4950 2700
+Wire Wire Line
+	3850 2300 4950 2300
+Wire Wire Line
+	3850 2200 5300 2200
+NoConn ~ 2050 4000
+NoConn ~ 2050 4600
+Text HLabel 2050 4500 0    50   Input ~ 0
+ABORT_2
+Text HLabel 2050 4200 0    50   Input ~ 0
+ABORT_1
+NoConn ~ 2050 4400
+NoConn ~ 2050 4100
+Text HLabel 3850 4600 2    50   Input ~ 0
+I2C2_EN
+NoConn ~ 2050 4800
+NoConn ~ 3850 3400
 $EndSCHEMATC
