File: Hardware/COMPONENT_SHEETS/DSUB-slot.kicad_sch (KiCad schematic)
At the start: 2 parts, among them J8 L717SDC37P1ACH4F

Commit message: Added bootloader pins, adjusted lipo monitor and mcu buttons
Parts:
- removed C36: 100nF, Capacitor_SMD:C_0603_1608Metric_Pad1.08x0.95mm_HandSolder, symbol Device:C_Small
Changed lines of the file:
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@@
     (company "Missouri S&T Rocket Design Team '21 (Jacob King, Thomas Francois)")
-  )
-  (junction (at 127 60.96) (diameter 0) (color 0 0 0 0)
   )
   (no_connect (at 170.18 78.74))
@@
   (no_connect (at 144.78 76.2))
   (no_connect (at 170.18 81.28))
-  (wire (pts (xy 127 66.04) (xy 127 60.96))
-    (stroke (width 0) (type default) (color 0 0 0 0))
-  )
-  (wire (pts (xy 127 60.96) (xy 144.78 60.96))
-    (stroke (width 0) (type default) (color 0 0 0 0))
-  )
   (wire (pts (xy 173.99 93.98) (xy 170.18 93.98))
-    (stroke (width 0) (type default) (color 0 0 0 0))
-  )
-  (wire (pts (xy 125.73 60.96) (xy 127 60.96))
     (stroke (width 0) (type default) (color 0 0 0 0))
   )
@@
     (effects (font (size 1.27 1.27)) (justify left))
   )
-  (hierarchical_label "NRST" (shape input) (at 125.73 60.96 180)
+  (hierarchical_label "NRST" (shape input) (at 144.78 60.96 180)
     (effects (font (size 1.27 1.27)) (justify right))
   )
@@
     (pin "1")
   )
-  (symbol (lib_id "Device:C_Small") (at 127 68.58 0) (mirror x) (unit 1)
-    (in_bom yes) (on_board yes)
-    (property "Reference" "C36" (id 0) (at 129.3368 69.7484 0)
-      (effects (font (size 1.27 1.27)) (justify left))
-    )
-    (property "Value" "100nF" (id 1) (at 129.3368 67.437 0)
-      (effects (font (size 1.27 1.27)) (justify left))
-    )
-    (property "Footprint" "Capacitor_SMD:C_0603_1608Metric_Pad1.08x0.95mm_HandSolder" (id 2) (at 127 68.58 0)
-      (effects (font (size 1.27 1.27)) hide)
-    )
-    (property "Datasheet" "~" (id 3) (at 127 68.58 0)
-      (effects (font (size 1.27 1.27)) hide)
-    )
-    (pin "1")
-    (pin "2")
-  )
   (symbol (lib_id "power:GND") (at 173.99 93.98 0) (unit 1)
     (in_bom yes) (on_board yes)
@@
       (effects (font (size 1.27 1.27)) hide)
     )
-    (pin "1")
-  )
-  (symbol (lib_id "power:GND") (at 127 71.12 0) (unit 1)
-    (in_bom yes) (on_board yes)
-    (property "Reference" "#PWR038" (id 0) (at 127 77.47 0)
-      (effects (font (size 1.27 1.27)) hide)
-    )
-    (property "Value" "GND" (id 1) (at 127.127 75.5142 0))
-    (property "Footprint" "" (id 2) (at 127 71.12 0)
-      (effects (font (size 1.27 1.27)) hide)
-    )
-    (property "Datasheet" "" (id 3) (at 127 71.12 0)
-      (effects (font (size 1.27 1.27)) hide)
-    )
