File: Hardware/COMPONENT_SHEETS/LiPo_Pack_Monitor.kicad_sch (KiCad schematic)
At the start: 36 parts, among them IC1 TL3301NF260QG, Q1 PSMN2R6-40YS, Q2 BSS84PH6327XTSA2, Q3 PSMN2R6-40YS, U5 BQ76920PW

Commit message: Progress 1 to small board
Changed components around,deleted xt60s
Parts:
- removed C12, C14: 1μF, Capacitor_SMD:C_1206_3216Metric_Pad1.42x1.75mm_HandSolder, symbol Device:C_Small
Connections:
- net VC2 is gone; now on net VC1: C13.2, R4.2, U5.15 (VC2)
- net VC4 is gone; now on net VC3: C11.2, R2.2, U5.13 (VC4)
Other:
- note removed: "Cell 2"
- note removed: "Cell 4"
Changed lines of the file:
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@@
-    (stroke (width 0) (type default) (color 0 0 0 0))
-  )
-  (polyline (pts (xy 38.1 100.33) (xy 46.99 100.33))
     (stroke (width 0) (type default) (color 0 0 0 0))
   )
@@
     (stroke (width 0) (type default) (color 0 0 0 0))
   )
-  (polyline (pts (xy 46.99 100.33) (xy 46.99 107.95))
-    (stroke (width 0) (type default) (color 0 0 0 0))
-  )
   (wire (pts (xy 242.57 146.05) (xy 242.57 144.78))
     (stroke (width 0) (type default) (color 0 0 0 0))
@@
     (stroke (width 0) (type default) (color 0 0 0 0))
   )
-  (wire (pts (xy 74.93 78.74) (xy 74.93 81.28))
-    (stroke (width 0) (type default) (color 0 0 0 0))
-  )
   (bus (pts (xy 87.63 93.98) (xy 120.65 93.98))
     (stroke (width 0) (type default) (color 0 0 0 0))
   )
-  (polyline (pts (xy 46.99 80.01) (xy 46.99 87.63))
-    (stroke (width 0) (type default) (color 0 0 0 0))
-  )
   (wire (pts (xy 74.93 99.06) (xy 85.09 99.06))
     (stroke (width 0) (type default) (color 0 0 0 0))
@@
     (stroke (width 0) (type default) (color 0 0 0 0))
   )
-  (wire (pts (xy 74.93 106.68) (xy 74.93 109.22))
-    (stroke (width 0) (type default) (color 0 0 0 0))
-  )
   (wire (pts (xy 191.77 146.05) (xy 187.96 146.05))
     (stroke (width 0) (type default) (color 0 0 0 0))
@@
     (stroke (width 0) (type default) (color 0 0 0 0))
   )
-  (polyline (pts (xy 38.1 107.95) (xy 38.1 100.33))
-    (stroke (width 0) (type default) (color 0 0 0 0))
-  )
   (polyline (pts (xy 43.18 69.85) (xy 43.18 68.58))
     (stroke (width 0) (type default) (color 0 0 0 0))
@@
     (stroke (width 0) (type default) (color 0 0 0 0))
   )
-  (polyline (pts (xy 38.1 80.01) (xy 46.99 80.01))
-    (stroke (width 0) (type default) (color 0 0 0 0))
-  )
   (wire (pts (xy 229.87 133.35) (xy 233.68 133.35))
     (stroke (width 0) (type default) (color 0 0 0 0))
@@
     (stroke (width 0) (type default) (color 0 0 0 0))
   )
-  (wire (pts (xy 74.93 101.6) (xy 74.93 99.06))
+  (wire (pts (xy 74.93 99.06) (xy 74.93 109.22))
     (stroke (width 0) (type default) (color 0 0 0 0))
   )
@@
     (stroke (width 0) (type default) (color 0 0 0 0))
   )
-  (wire (pts (xy 74.93 88.9) (xy 74.93 86.36))
+  (wire (pts (xy 74.93 78.74) (xy 74.93 88.9))
     (stroke (width 0) (type default) (color 0 0 0 0))
   )
@@
     (stroke (width 0) (type default) (color 0 0 0 0))
   )
-  (polyline (pts (xy 46.99 87.63) (xy 38.1 87.63))
-    (stroke (width 0) (type default) (color 0 0 0 0))
-  )
   (wire (pts (xy 148.59 91.44) (xy 143.51 91.44))
     (stroke (width 0) (type default) (color 0 0 0 0))
@@
     (stroke (width 0) (type default) (color 0 0 0 0))
   )
-  (polyline (pts (xy 38.1 87.63) (xy 38.1 80.01))
-    (stroke (width 0) (type default) (color 0 0 0 0))
-  )
   (bus (pts (xy 142.24 83.82) (xy 142.24 86.36))
     (stroke (width 0) (type default) (color 0 0 0 0))
@@
     (stroke (width 0) (type default) (color 0 0 0 0))
   )
-  (polyline (pts (xy 46.99 107.95) (xy 38.1 107.95))
-    (stroke (width 0) (type default) (color 0 0 0 0))
-  )
   (wire (pts (xy 74.93 118.11) (xy 74.93 116.84))
     (stroke (width 0) (type default) (color 0 0 0 0))
@@
     (stroke (width 0) (type default) (color 0 0 0 0))
   )
-  (text "-" (at 41.91 107.95 0)
-    (effects (font (size 1.27 1.27)) (justify left bottom))
-  )
-  (text "Cell 4" (at 39.37 85.09 0)
-    (effects (font (size 1.27 1.27)) (justify left bottom))
-  )
   (text "Cell 1" (at 39.37 118.11 0)
     (effects (font (size 1.27 1.27)) (justify left bottom))
   )
-  (text "Cell 2" (at 39.37 105.41 0)
-    (effects (font (size 1.27 1.27)) (justify left bottom))
-  )
   (text "-" (at 41.91 120.65 0)
     (effects (font (size 1.27 1.27)) (justify left bottom))
@@
     (effects (font (size 1.27 1.27)) (justify left bottom))
   )
-  (text "+" (at 41.91 82.55 0)
-    (effects (font (size 1.27 1.27)) (justify left bottom))
-  )
   (text "+" (at 41.91 72.39 0)
     (effects (font (size 1.27 1.27)) (justify left bottom))
@@
   )
   (text "+" (at 41.91 115.57 0)
-    (effects (font (size 1.27 1.27)) (justify left bottom))
-  )
-  (text "-" (at 41.91 87.63 0)
-    (effects (font (size 1.27 1.27)) (justify left bottom))
-  )
-  (text "+" (at 41.91 102.87 0)
     (effects (font (size 1.27 1.27)) (justify left bottom))
   )
@@
     (pin "2")
   )
-  (symbol (lib_id "Device:C_Small") (at 74.93 83.82 0) (unit 1)
-    (in_bom yes) (on_board yes)
-    (property "Reference" "C12" (id 0) (at 77.2668 82.6516 0)
-      (effects (font (size 1.27 1.27)) (justify left))
-    )
-    (property "Value" "1μF" (id 1) (at 77.2668 84.963 0)
-      (effects (font (size 1.27 1.27)) (justify left))
-    )
-    (property "Footprint" "Capacitor_SMD:C_1206_3216Metric_Pad1.42x1.75mm_HandSolder" (id 2) (at 74.93 83.82 0)
-      (effects (font (size 1.27 1.27)) hide)
-    )
-    (property "Datasheet" "~" (id 3) (at 74.93 83.82 0)
-      (effects (font (size 1.27 1.27)) hide)
-    )
-    (pin "1")
-    (pin "2")
-  )
   (symbol (lib_id "Device:C_Small") (at 74.93 93.98 0) (unit 1)
     (in_bom yes) (on_board yes)
@@
       (effects (font (size 1.27 1.27)) hide)
     )
-    (pin "1")
-    (pin "2")
-  )
-  (symbol (lib_id "Device:C_Small") (at 74.93 104.14 0) (unit 1)
-    (in_bom yes) (on_board yes)
-    (property "Reference" "C14" (id 0) (at 77.2668 102.9716 0)
-      (effects (font (size 1.27 1.27)) (justify left))
-    )
-    (property "Value" "1μF" (id 1) (at 77.2668 105.283 0)
-      (effects (font (size 1.27 1.27)) (justify left))
-    )
-    (property "Footprint" "Capacitor_SMD:C_1206_3216Metric_Pad1.42x1.75mm_HandSolder" (id 2) (at 74.93 104.14 0)
-      (effects (font (size 1.27 1.27)) hide)
-    )
-    (property "Datasheet" "~" (id 3) (at 74.93 104.14 0)
-      (effects (font (size 1.27 1.27)) hide)
-    )
