File: Hardware/COMPONENT_SHEETS/TEMPSENSOR_MCP9808.kicad_sch (KiCad schematic)
At the start: 2 parts, among them U2 MIC184YMM-TR

Commit message: Test
Parts:
- renumbered C1 to C2, U2 to U1
Changed lines of the file:
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@@
     (effects (font (size 1.27 1.27)) (justify left))
   )
-  (symbol (lib_id "power:+3.3V") (at 143.51 46.99 0)
+  (symbol (lib_id "power:+3.3V") (at 143.51 46.99 0) (unit 1)
     (in_bom yes) (on_board yes)
-    (property "Reference" "#PWR08" (id 0) (at 143.51 50.8 0)
+    (property "Reference" "#PWR011" (id 0) (at 143.51 50.8 0)
       (effects (font (size 1.27 1.27)) hide)
     )
@@
     (pin "1")
   )
-  (symbol (lib_id "Device:C") (at 124.46 62.23 0)
+  (symbol (lib_id "Device:C") (at 124.46 62.23 0) (unit 1)
     (in_bom yes) (on_board yes)
-    (property "Reference" "C1" (id 0) (at 127.381 61.0616 0)
+    (property "Reference" "C2" (id 0) (at 127.381 61.0616 0)
       (effects (font (size 1.27 1.27)) (justify left))
     )
@@
     (pin "2")
   )
-  (symbol (lib_id "power:GND") (at 124.46 66.04 0)
+  (symbol (lib_id "power:GND") (at 124.46 66.04 0) (unit 1)
     (in_bom yes) (on_board yes)
-    (property "Reference" "#PWR09" (id 0) (at 124.46 72.39 0)
+    (property "Reference" "#PWR012" (id 0) (at 124.46 72.39 0)
       (effects (font (size 1.27 1.27)) hide)
     )
@@
     (pin "1")
   )
-  (symbol (lib_id "power:GND") (at 140.97 110.49 0)
+  (symbol (lib_id "power:GND") (at 140.97 110.49 0) (unit 1)
     (in_bom yes) (on_board yes)
-    (property "Reference" "#PWR07" (id 0) (at 140.97 116.84 0)
+    (property "Reference" "#PWR010" (id 0) (at 140.97 116.84 0)
       (effects (font (size 1.27 1.27)) hide)
     )
@@
     (pin "1")
   )
-  (symbol (lib_id "RDT_Custom_Symbols:MIC184YMM-TR") (at 138.43 107.95 90)
+  (symbol (lib_id "RDT_Custom_Symbols:MIC184YMM-TR") (at 138.43 107.95 90) (unit 1)
     (in_bom yes) (on_board yes) (fields_autoplaced)
-    (property "Reference" "U2" (id 0) (at 154.4066 75.6306 90)
+    (property "Reference" "U1" (id 0) (at 154.4066 75.6306 90)
       (effects (font (size 1.524 1.524)) (justify right))
     )
